File: 8086proj/28F010.kicad_sch (KiCad schematic)
At the start: 3 parts, among them U4 28F010, U5 28F010

Commit message: power added
Parts:
- added C? (x3): .1uF, symbol Device:C
Connections:
- net GND: now also C?.1, C?.1, C?.2
- net +5V renamed VIN
- net VIN: now also C?.1, C?.2, C?.2
Changed lines of the file:
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@@
 (kicad_sch (version 20211123) (generator eeschema)
   (paper "A4")
+  (junction (at 199.39 35.56) (diameter 0) (color 0 0 0 0)
+  )
+  (junction (at 195.58 93.98) (diameter 0) (color 0 0 0 0)
+  )
+  (junction (at 68.58 17.78) (diameter 0) (color 0 0 0 0)
+  )
+  (junction (at 210.82 35.56) (diameter 0) (color 0 0 0 0)
+  )
+  (junction (at 68.58 33.02) (diameter 0) (color 0 0 0 0)
+  )
+  (junction (at 210.82 93.98) (diameter 0) (color 0 0 0 0)
+  )
   (no_connect (at 133.35 35.56))
   (no_connect (at 129.54 93.98))
@@
     (stroke (width 0) (type default) (color 0 0 0 0))
   )
+  (wire (pts (xy 189.23 35.56) (xy 199.39 35.56))
+    (stroke (width 0) (type default) (color 0 0 0 0))
+  )
   (wire (pts (xy 125.73 58.42) (xy 133.35 58.42))
     (stroke (width 0) (type default) (color 0 0 0 0))
@@
     (stroke (width 0) (type default) (color 0 0 0 0))
   )
+  (wire (pts (xy 68.58 17.78) (xy 68.58 33.02))
+    (stroke (width 0) (type default) (color 0 0 0 0))
+  )
   (wire (pts (xy 125.73 63.5) (xy 133.35 63.5))
     (stroke (width 0) (type default) (color 0 0 0 0))
@@
     (stroke (width 0) (type default) (color 0 0 0 0))
   )
+  (wire (pts (xy 58.42 17.78) (xy 68.58 17.78))
+    (stroke (width 0) (type default) (color 0 0 0 0))
+  )
   (wire (pts (xy 125.73 50.8) (xy 133.35 50.8))
     (stroke (width 0) (type default) (color 0 0 0 0))
@@
     (stroke (width 0) (type default) (color 0 0 0 0))
   )
+  (wire (pts (xy 210.82 35.56) (xy 210.82 93.98))
+    (stroke (width 0) (type default) (color 0 0 0 0))
+  )
   (bus (pts (xy 27.94 24.13) (xy 27.94 96.52))
     (stroke (width 0) (type default) (color 0 0 0 0))
@@
     (stroke (width 0) (type default) (color 0 0 0 0))
   )
-  (bus (pts (xy 199.39 24.13) (xy 27.94 24.13))
-    (stroke (width 0) (type default) (color 0 0 0 0))
-  )
   (wire (pts (xy 121.92 96.52) (xy 129.54 96.52))
     (stroke (width 0) (type default) (color 0 0 0 0))
@@
     (stroke (width 0) (type default) (color 0 0 0 0))
   )
+  (wire (pts (xy 210.82 93.98) (xy 210.82 100.33))
+    (stroke (width 0) (type default) (color 0 0 0 0))
+  )
   (wire (pts (xy 125.73 60.96) (xy 133.35 60.96))
     (stroke (width 0) (type default) (color 0 0 0 0))
   )
+  (wire (pts (xy 68.58 17.78) (xy 210.82 17.78))
+    (stroke (width 0) (type default) (color 0 0 0 0))
+  )
+  (wire (pts (xy 195.58 93.98) (xy 210.82 93.98))
+    (stroke (width 0) (type default) (color 0 0 0 0))
+  )
   (wire (pts (xy 185.42 104.14) (xy 191.77 104.14))
     (stroke (width 0) (type default) (color 0 0 0 0))
@@
     (stroke (width 0) (type default) (color 0 0 0 0))
   )
+  (wire (pts (xy 185.42 93.98) (xy 195.58 93.98))
+    (stroke (width 0) (type default) (color 0 0 0 0))
+  )
+  (wire (pts (xy 210.82 17.78) (xy 210.82 35.56))
+    (stroke (width 0) (type default) (color 0 0 0 0))
+  )
   (wire (pts (xy 189.23 68.58) (xy 191.77 68.58))
     (stroke (width 0) (type default) (color 0 0 0 0))
@@
     (stroke (width 0) (type default) (color 0 0 0 0))
   )
+  (wire (pts (xy 68.58 33.02) (xy 68.58 38.1))
+    (stroke (width 0) (type default) (color 0 0 0 0))
+  )
   (wire (pts (xy 48.26 50.8) (xy 55.88 50.8))
+    (stroke (width 0) (type default) (color 0 0 0 0))
+  )
+  (wire (pts (xy 199.39 35.56) (xy 210.82 35.56))
     (stroke (width 0) (type default) (color 0 0 0 0))
   )
@@
     (effects (font (size 1.27 1.27)) (justify left))
   )
+  (hierarchical_label "VIN" (shape input) (at 58.42 17.78 180)
+    (effects (font (size 1.27 1.27)) (justify right))
+  )
   (hierarchical_label "DATA" (shape bidirectional) (at 27.94 130.81 0)
     (effects (font (size 1.27 1.27)) (justify left))
@@
   (hierarchical_label "OE" (shape input) (at 195.58 55.88 0)
     (effects (font (size 1.27 1.27)) (justify left))
+  )
+  (symbol (lib_id "Device:C") (at 72.39 33.02 270) (unit 1)
+    (in_bom yes) (on_board yes) (fields_autoplaced)
+    (property "Reference" "C?" (id 0) (at 72.39 25.4 90))
+    (property "Value" ".1uF" (id 1) (at 72.39 27.94 90))
+    (property "Footprint" "" (id 2) (at 68.58 33.9852 0)
+      (effects (font (size 1.27 1.27)) hide)
+    )
+    (property "Datasheet" "~" (id 3) (at 72.39 33.02 0)
+      (effects (font (size 1.27 1.27)) hide)
+    )
+    (pin "1")
+    (pin "2")
   )
   (symbol (lib_id "Logic_Programmable:PAL16L8") (at 68.58 55.88 0) (unit 1)
@@
     (pin "8")
     (pin "9")
+  )
+  (symbol (lib_id "power:GND") (at 199.39 27.94 180) (unit 1)
+    (in_bom yes) (on_board yes) (fields_autoplaced)
+    (property "Reference" "#PWR?" (id 0) (at 199.39 21.59 0)
+      (effects (font (size 1.27 1.27)) hide)
+    )
+    (property "Value" "" (id 1) (at 199.39 22.86 0))
+    (property "Footprint" "" (id 2) (at 199.39 27.94 0)
+      (effects (font (size 1.27 1.27)) hide)
+    )
+    (property "Datasheet" "" (id 3) (at 199.39 27.94 0)
+      (effects (font (size 1.27 1.27)) hide)
+    )
+    (pin "1")
+  )
+  (symbol (lib_id "power:GND") (at 195.58 86.36 90) (unit 1)
+    (in_bom yes) (on_board yes) (fields_autoplaced)
+    (property "Reference" "#PWR?" (id 0) (at 201.93 86.36 0)
+      (effects (font (size 1.27 1.27)) hide)
+    )
+    (property "Value" "" (id 1) (at 199.39 86.3599 90)
+      (effects (font (size 1.27 1.27)) (justify right))
+    )
+    (property "Footprint" "" (id 2) (at 195.58 86.36 0)
+      (effects (font (size 1.27 1.27)) hide)
+    )
+    (property "Datasheet" "" (id 3) (at 195.58 86.36 0)
+      (effects (font (size 1.27 1.27)) hide)
+    )
+    (pin "1")
   )
   (symbol (lib_id "power:GND") (at 68.58 71.12 0) (unit 1)
@@
     (pin "9")
   )
-  (symbol (lib_id "power:+5V") (at 185.42 93.98 0) (unit 1)
-    (in_bom yes) (on_board yes)
-    (property "Reference" "#PWR?" (id 0) (at 185.42 97.79 0)
-      (effects (font (size 1.27 1.27)) hide)
-    )
-    (property "Value" "+5V" (id 1) (at 185.42 88.9 0))
-    (property "Footprint" "" (id 2) (at 185.42 93.98 0)
-      (effects (font (size 1.27 1.27)) hide)
-    )
-    (property "Datasheet" "" (id 3) (at 185.42 93.98 0)
-      (effects (font (size 1.27 1.27)) hide)
-    )
-    (pin "1")
+  (symbol (lib_id "Device:C") (at 195.58 90.17 0) (unit 1)
+    (in_bom yes) (on_board yes) (fields_autoplaced)
+    (property "Reference" "C?" (id 0) (at 199.39 88.8999 0)
+      (effects (font (size 1.27 1.27)) (justify left))
+    )
+    (property "Value" ".1uF" (id 1) (at 199.39 91.4399 0)
+      (effects (font (size 1.27 1.27)) (justify left))
+    )
+    (property "Footprint" "" (id 2) (at 196.5452 93.98 0)
+      (effects (font (size 1.27 1.27)) hide)
+    )
+    (property "Datasheet" "~" (id 3) (at 195.58 90.17 0)
+      (effects (font (size 1.27 1.27)) hide)
+    )
+    (pin "1")
+    (pin "2")
   )
   (symbol (lib_id "power:GND") (at 133.35 73.66 0) (unit 1)
@@
     (pin "1")
   )
-  (symbol (lib_id "power:+5V") (at 68.58 38.1 0) (unit 1)
-    (in_bom yes) (on_board yes) (fields_autoplaced)
-    (property "Reference" "#PWR?" (id 0) (at 68.58 41.91 0)
-      (effects (font (size 1.27 1.27)) hide)
-    )
-    (property "Value" "+5V" (id 1) (at 68.58 33.02 0))
-    (property "Footprint" "" (id 2) (at 68.58 38.1 0)
-      (effects (font (size 1.27 1.27)) hide)
-    )
-    (property "Datasheet" "" (id 3) (at 68.58 38.1 0)
+  (symbol (lib_id "power:GND") (at 76.2 33.02 0) (unit 1)
+    (in_bom yes) (on_board yes) (fields_autoplaced)
+    (property "Reference" "#PWR?" (id 0) (at 76.2 39.37 0)
+      (effects (font (size 1.27 1.27)) hide)
+    )
+    (property "Value" "" (id 1) (at 76.2 38.1 0))
+    (property "Footprint" "" (id 2) (at 76.2 33.02 0)
+      (effects (font (size 1.27 1.27)) hide)
+    )
+    (property "Datasheet" "" (id 3) (at 76.2 33.02 0)
       (effects (font (size 1.27 1.27)) hide)
     )
@@
     (pin "1")
   )
-  (symbol (lib_id "power:+5V") (at 189.23 35.56 0) (unit 1)
-    (in_bom yes) (on_board yes) (fields_autoplaced)
-    (property "Reference" "#PWR?" (id 0) (at 189.23 39.37 0)
-      (effects (font (size 1.27 1.27)) hide)
-    )
-    (property "Value" "+5V" (id 1) (at 189.23 30.48 0))
-    (property "Footprint" "" (id 2) (at 189.23 35.56 0)
-      (effects (font (size 1.27 1.27)) hide)
-    )
-    (property "Datasheet" "" (id 3) (at 189.23 35.56 0)
-      (effects (font (size 1.27 1.27)) hide)
-    )
-    (pin "1")
+  (symbol (lib_id "Device:C") (at 199.39 31.75 180) (unit 1)
+    (in_bom yes) (on_board yes) (fields_autoplaced)
+    (property "Reference" "C?" (id 0) (at 203.2 30.4799 0)
+      (effects (font (size 1.27 1.27)) (justify right))
+    )
+    (property "Value" ".1uF" (id 1) (at 203.2 33.0199 0)
+      (effects (font (size 1.27 1.27)) (justify right))
+    )
+    (property "Footprint" "" (id 2) (at 198.4248 27.94 0)
+      (effects (font (size 1.27 1.27)) hide)
+    )
+    (property "Datasheet" "~" (id 3) (at 199.39 31.75 0)
+      (effects (font (size 1.27 1.27)) hide)
+    )
+    (pin "1")
+    (pin "2")
   )
   (symbol (lib_id "28F010:28F010") (at 129.54 93.98 0) (unit 1)

Commit message: power added
Parts:
- removed C?: .1uF, symbol Device:C
Changed lines of the file:
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@@
   (junction (at 210.82 35.56) (diameter 0) (color 0 0 0 0)
-  )
-  (junction (at 68.58 33.02) (diameter 0) (color 0 0 0 0)
   )
   (junction (at 210.82 93.98) (diameter 0) (color 0 0 0 0)
@@
     (stroke (width 0) (type default) (color 0 0 0 0))
   )
-  (wire (pts (xy 68.58 17.78) (xy 68.58 33.02))
+  (wire (pts (xy 68.58 17.78) (xy 68.58 38.1))
     (stroke (width 0) (type default) (color 0 0 0 0))
   )
@@
   )
   (wire (pts (xy 125.73 38.1) (xy 133.35 38.1))
-    (stroke (width 0) (type default) (color 0 0 0 0))
-  )
-  (wire (pts (xy 68.58 33.02) (xy 68.58 38.1))
     (stroke (width 0) (type default) (color 0 0 0 0))
   )
@@
   (hierarchical_label "OE" (shape input) (at 195.58 55.88 0)
     (effects (font (size 1.27 1.27)) (justify left))
-  )
-  (symbol (lib_id "Device:C") (at 72.39 33.02 270) (unit 1)
-    (in_bom yes) (on_board yes) (fields_autoplaced)
-    (property "Reference" "C?" (id 0) (at 72.39 25.4 90))
-    (property "Value" ".1uF" (id 1) (at 72.39 27.94 90))
-    (property "Footprint" "" (id 2) (at 68.58 33.9852 0)
-      (effects (font (size 1.27 1.27)) hide)
-    )
-    (property "Datasheet" "~" (id 3) (at 72.39 33.02 0)
-      (effects (font (size 1.27 1.27)) hide)
-    )
-    (pin "1")
-    (pin "2")
   )
   (symbol (lib_id "Logic_Programmable:PAL16L8") (at 68.58 55.88 0) (unit 1)
@@
       (effects (font (size 1.27 1.27)) hide)
     )
-    (pin "1")
-  )
-  (symbol (lib_id "power:GND") (at 76.2 33.02 0) (unit 1)
-    (in_bom yes) (on_board yes) (fields_autoplaced)
-    (property "Reference" "#PWR?" (id 0) (at 76.2 39.37 0)
-      (effects (font (size 1.27 1.27)) hide)
-    )
-    (property "Value" "" (id 1) (at 76.2 38.1 0))
-    (property "Footprint" "" (id 2) (at 76.2 33.02 0)
-      (effects (font (size 1.27 1.27)) hide)
-    )
-    (property "Datasheet" "" (id 3) (at 76.2 33.02 0)
-      (effects (font (size 1.27 1.27)) hide)
-    )

Commit message: 8259
Changed lines of the file:
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@@
       (effects (font (size 1.27 1.27)) hide)
     )
-    (property "Value" "" (id 1) (at 199.39 22.86 0))
+    (property "Value" "GND" (id 1) (at 199.39 22.86 0))
     (property "Footprint" "" (id 2) (at 199.39 27.94 0)
       (effects (font (size 1.27 1.27)) hide)
@@
       (effects (font (size 1.27 1.27)) hide)
     )
-    (property "Value" "" (id 1) (at 199.39 86.3599 90)
+    (property "Value" "GND" (id 1) (at 199.39 86.3599 90)
       (effects (font (size 1.27 1.27)) (justify right))
     )

Commit message: fixes
Connections:
- net M/_IO: now reaches U?.5 (I5)
- no-connect marks 16 -> 15
Changed lines of the file:
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@@
   (no_connect (at 133.35 35.56))
   (no_connect (at 129.54 93.98))
-  (no_connect (at 55.88 53.34))
   (no_connect (at 55.88 55.88))
   (no_connect (at 55.88 58.42))
@@
     (stroke (width 0) (type default) (color 0 0 0 0))
   )
+  (wire (pts (xy 48.26 53.34) (xy 55.88 53.34))
+    (stroke (width 0) (type default) (color 0 0 0 0))
+  )
   (wire (pts (xy 185.42 127) (xy 193.04 127))
     (stroke (width 0) (type default) (color 0 0 0 0))
@@
     (effects (font (size 1.27 1.27)) (justify left))
   )
+  (hierarchical_label "M{slash}_IO" (shape input) (at 48.26 53.34 180)
+    (effects (font (size 1.27 1.27)) (justify right))
+  )
   (symbol (lib_id "Logic_Programmable:PAL16L8") (at 68.58 55.88 0) (unit 1)
