File: 8086proj/28F010.kicad_sch (KiCad schematic)
At the start: 5 parts, among them U4 28F010, U5 28F010

Commit message: final look
Parts:
- gave numbers to parts that had none: 3
- renumbered U4 to U402, U5 to U403
Changed lines of the file:
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@@
   (symbol (lib_id "Logic_Programmable:PAL16L8") (at 68.58 55.88 0) (unit 1)
     (in_bom yes) (on_board yes) (fields_autoplaced)
-    (property "Reference" "U?" (id 0) (at 70.5994 36.83 0)
+    (property "Reference" "U401" (id 0) (at 70.5994 36.83 0)
       (effects (font (size 1.27 1.27)) (justify left))
     )
@@
   (symbol (lib_id "power:GND") (at 199.39 27.94 180) (unit 1)
     (in_bom yes) (on_board yes) (fields_autoplaced)
-    (property "Reference" "#PWR0113" (id 0) (at 199.39 21.59 0)
+    (property "Reference" "#PWR0405" (id 0) (at 199.39 21.59 0)
       (effects (font (size 1.27 1.27)) hide)
     )
@@
   (symbol (lib_id "power:GND") (at 195.58 86.36 90) (unit 1)
     (in_bom yes) (on_board yes) (fields_autoplaced)
-    (property "Reference" "#PWR0112" (id 0) (at 201.93 86.36 0)
+    (property "Reference" "#PWR0404" (id 0) (at 201.93 86.36 0)
       (effects (font (size 1.27 1.27)) hide)
     )
@@
   (symbol (lib_id "power:GND") (at 68.58 71.12 0) (unit 1)
     (in_bom yes) (on_board yes) (fields_autoplaced)
-    (property "Reference" "#PWR0115" (id 0) (at 68.58 77.47 0)
+    (property "Reference" "#PWR0401" (id 0) (at 68.58 77.47 0)
       (effects (font (size 1.27 1.27)) hide)
     )
@@
   (symbol (lib_id "28F010:28F010") (at 133.35 35.56 0) (unit 1)
     (in_bom yes) (on_board yes) (fields_autoplaced)
-    (property "Reference" "U5" (id 0) (at 161.29 24.13 0)
+    (property "Reference" "U403" (id 0) (at 161.29 24.13 0)
       (effects (font (size 1.524 1.524)))
     )
@@
   (symbol (lib_id "Device:C") (at 195.58 90.17 0) (unit 1)
     (in_bom yes) (on_board yes) (fields_autoplaced)
-    (property "Reference" "C?" (id 0) (at 199.39 88.8999 0)
+    (property "Reference" "C401" (id 0) (at 199.39 88.8999 0)
       (effects (font (size 1.27 1.27)) (justify left))
     )
@@
   (symbol (lib_id "power:GND") (at 133.35 73.66 0) (unit 1)
     (in_bom yes) (on_board yes) (fields_autoplaced)
-    (property "Reference" "#PWR0111" (id 0) (at 133.35 80.01 0)
+    (property "Reference" "#PWR0403" (id 0) (at 133.35 80.01 0)
       (effects (font (size 1.27 1.27)) hide)
     )
@@
   (symbol (lib_id "power:GND") (at 129.54 132.08 0) (unit 1)
     (in_bom yes) (on_board yes) (fields_autoplaced)
-    (property "Reference" "#PWR0114" (id 0) (at 129.54 138.43 0)
+    (property "Reference" "#PWR0402" (id 0) (at 129.54 138.43 0)
       (effects (font (size 1.27 1.27)) hide)
     )
@@
   (symbol (lib_id "Device:C") (at 199.39 31.75 180) (unit 1)
     (in_bom yes) (on_board yes) (fields_autoplaced)
-    (property "Reference" "C?" (id 0) (at 203.2 30.4799 0)
+    (property "Reference" "C402" (id 0) (at 203.2 30.4799 0)
       (effects (font (size 1.27 1.27)) (justify right))
     )
@@
   (symbol (lib_id "28F010:28F010") (at 129.54 93.98 0) (unit 1)
     (in_bom yes) (on_board yes)
-    (property "Reference" "U4" (id 0) (at 157.48 82.55 0)
+    (property "Reference" "U402" (id 0) (at 157.48 82.55 0)
       (effects (font (size 1.524 1.524)))
     )

Commit message: footprints
Parts:
- C401, C402: footprint (none) -> Capacitor_SMD:CP_Elec_3x5.3
Changed lines of the file:
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@@
       (effects (font (size 1.27 1.27)) (justify left))
     )
-    (property "Footprint" "" (id 2) (at 196.5452 93.98 0)
+    (property "Footprint" "Capacitor_SMD:CP_Elec_3x5.3" (id 2) (at 196.5452 93.98 0)
       (effects (font (size 1.27 1.27)) hide)
     )
@@
       (effects (font (size 1.27 1.27)) (justify right))
     )
-    (property "Footprint" "" (id 2) (at 198.4248 27.94 0)
+    (property "Footprint" "Capacitor_SMD:CP_Elec_3x5.3" (id 2) (at 198.4248 27.94 0)
       (effects (font (size 1.27 1.27)) hide)
     )

Commit message: pcb
Parts:
- U401: footprint (none) -> Package_DIP:DIP-20_W7.62mm
- U402, U403: footprint 28F010 -> Package_DIP:DIP-32_W15.24mm
Changed lines of the file:
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@@
       (effects (font (size 1.27 1.27)) (justify left))
     )
-    (property "Footprint" "" (id 2) (at 68.58 55.88 0)
+    (property "Footprint" "Package_DIP:DIP-20_W7.62mm" (id 2) (at 68.58 55.88 0)
       (effects (font (size 1.27 1.27)) hide)
     )
@@
       (effects (font (size 1.524 1.524)))
     )
-    (property "Footprint" "28F010" (id 2) (at 161.29 29.464 0)
+    (property "Footprint" "Package_DIP:DIP-32_W15.24mm" (id 2) (at 161.29 29.464 0)
       (effects (font (size 1.524 1.524)) hide)
     )
@@
       (effects (font (size 1.524 1.524)))
     )
-    (property "Footprint" "28F010" (id 2) (at 157.48 87.884 0)
+    (property "Footprint" "Package_DIP:DIP-32_W15.24mm" (id 2) (at 157.48 87.884 0)
       (effects (font (size 1.524 1.524)) hide)
     )
