File: 8086proj/FinalProj.kicad_sch (KiCad schematic)
At the start: 0 parts

Commit message: latch added
Other:
- sheet 28F010 ports: added DATA; removed A high
- sheet 8086 ports: added ADR, DATA; removed A16-19, ALE, A/D BUS
Changed lines of the file:
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@@
   (junction (at 143.51 59.69) (diameter 0) (color 0 0 0 0)
   )
-  (junction (at 146.05 53.34) (diameter 0) (color 0 0 0 0)
-  )
-  (junction (at 144.78 55.88) (diameter 0) (color 0 0 0 0)
+  (bus (pts (xy 133.35 49.53) (xy 133.35 53.34))
+    (stroke (width 0) (type default) (color 0 0 0 0))
   )
   (wire (pts (xy 148.59 59.69) (xy 143.51 59.69))
     (stroke (width 0) (type default) (color 0 0 0 0))
   )
-  (bus (pts (xy 144.78 55.88) (xy 144.78 86.36))
-    (stroke (width 0) (type default) (color 0 0 0 0))
-  )
   (wire (pts (xy 76.2 25.4) (xy 85.09 25.4))
     (stroke (width 0) (type default) (color 0 0 0 0))
@@
     (stroke (width 0) (type default) (color 0 0 0 0))
   )
-  (bus (pts (xy 96.52 66.04) (xy 91.44 66.04))
-    (stroke (width 0) (type default) (color 0 0 0 0))
-  )
-  (bus (pts (xy 144.78 55.88) (xy 96.52 55.88))
-    (stroke (width 0) (type default) (color 0 0 0 0))
-  )
-  (bus (pts (xy 146.05 83.82) (xy 148.59 83.82))
-    (stroke (width 0) (type default) (color 0 0 0 0))
-  )
   (wire (pts (xy 72.39 22.86) (xy 72.39 46.99))
     (stroke (width 0) (type default) (color 0 0 0 0))
   )
-  (bus (pts (xy 146.05 53.34) (xy 146.05 83.82))
-    (stroke (width 0) (type default) (color 0 0 0 0))
-  )
   (wire (pts (xy 143.51 59.69) (xy 97.79 59.69))
     (stroke (width 0) (type default) (color 0 0 0 0))
@@
     (stroke (width 0) (type default) (color 0 0 0 0))
   )
-  (bus (pts (xy 144.78 86.36) (xy 148.59 86.36))
-    (stroke (width 0) (type default) (color 0 0 0 0))
-  )
-  (bus (pts (xy 96.52 55.88) (xy 96.52 66.04))
+  (bus (pts (xy 148.59 57.15) (xy 96.52 57.15))
+    (stroke (width 0) (type default) (color 0 0 0 0))
+  )
+  (bus (pts (xy 91.44 49.53) (xy 133.35 49.53))
     (stroke (width 0) (type default) (color 0 0 0 0))
   )
@@
     (stroke (width 0) (type default) (color 0 0 0 0))
   )
-  (bus (pts (xy 148.59 53.34) (xy 146.05 53.34))
-    (stroke (width 0) (type default) (color 0 0 0 0))
-  )
   (wire (pts (xy 91.44 73.66) (xy 99.06 73.66))
     (stroke (width 0) (type default) (color 0 0 0 0))
   )
-  (bus (pts (xy 96.52 53.34) (xy 96.52 50.8))
-    (stroke (width 0) (type default) (color 0 0 0 0))
-  )
-  (bus (pts (xy 148.59 55.88) (xy 144.78 55.88))
+  (bus (pts (xy 133.35 53.34) (xy 148.59 53.34))
     (stroke (width 0) (type default) (color 0 0 0 0))
   )
@@
     (stroke (width 0) (type default) (color 0 0 0 0))
   )
+  (bus (pts (xy 96.52 52.07) (xy 91.44 52.07))
+    (stroke (width 0) (type default) (color 0 0 0 0))
+  )
   (wire (pts (xy 142.24 91.44) (xy 148.59 91.44))
     (stroke (width 0) (type default) (color 0 0 0 0))
@@
     (stroke (width 0) (type default) (color 0 0 0 0))
   )
-  (bus (pts (xy 146.05 53.34) (xy 96.52 53.34))
-    (stroke (width 0) (type default) (color 0 0 0 0))
-  )
   (wire (pts (xy 97.79 78.74) (xy 91.44 78.74))
     (stroke (width 0) (type default) (color 0 0 0 0))
@@
     (stroke (width 0) (type default) (color 0 0 0 0))
   )
-  (bus (pts (xy 96.52 50.8) (xy 91.44 50.8))
+  (bus (pts (xy 96.52 57.15) (xy 96.52 52.07))
     (stroke (width 0) (type default) (color 0 0 0 0))
   )
@@
       (effects (font (size 1.27 1.27)) (justify left))
     )
-    (pin "A high" input (at 148.59 55.88 180)
-      (effects (font (size 1.27 1.27)) (justify left))
-    )
     (pin "AIN" bidirectional (at 148.59 53.34 180)
+      (effects (font (size 1.27 1.27)) (justify left))
+    )
+    (pin "DATA" bidirectional (at 148.59 57.15 180)
       (effects (font (size 1.27 1.27)) (justify left))
     )
@@
       (effects (font (size 1.27 1.27)) (justify right))
     )
-    (pin "A{slash}D BUS" bidirectional (at 91.44 50.8 0)
-      (effects (font (size 1.27 1.27)) (justify right))
-    )
-    (pin "ALE" output (at 66.04 46.99 90)
-      (effects (font (size 1.27 1.27)) (justify right))
-    )
     (pin "DR{slash}_R" output (at 68.58 46.99 90)
       (effects (font (size 1.27 1.27)) (justify right))
@@
       (effects (font (size 1.27 1.27)) (justify right))
     )
-    (pin "A16-19" output (at 91.44 66.04 0)
-      (effects (font (size 1.27 1.27)) (justify right))
-    )
     (pin "MIN{slash}_MAX" input (at 48.26 86.36 270)
       (effects (font (size 1.27 1.27)) (justify left))
+    )
+    (pin "ADR" output (at 91.44 49.53 0)
+      (effects (font (size 1.27 1.27)) (justify right))
+    )
+    (pin "DATA" bidirectional (at 91.44 52.07 0)
+      (effects (font (size 1.27 1.27)) (justify right))
     )
   )
@@
       (reference "#PWR?") (unit 1) (value "GND") (footprint "")
     )
+    (path "/33150f27-98b3-4b2a-92cc-16b50b335e66/68baa8d0-f185-49b1-a0de-efe65cf5e226"
+      (reference "#PWR?") (unit 1) (value "GND") (footprint "")
+    )
     (path "/13edf85d-e5b3-408c-9ca0-37b4fd7394a6/7533e456-82d6-4314-a558-1c0c4fd0b94e"
       (reference "#PWR?") (unit 1) (value "+5V") (footprint "")
     )
+    (path "/33150f27-98b3-4b2a-92cc-16b50b335e66/835398a9-a3e0-415f-b1f5-e468129ca980"
+      (reference "#PWR?") (unit 1) (value "GND") (footprint "")
+    )
     (path "/13edf85d-e5b3-408c-9ca0-37b4fd7394a6/8841ec03-9d7b-4fff-9c78-98d20a533ddf"
       (reference "#PWR?") (unit 1) (value "GND") (footprint "")
@@
       (reference "#PWR?") (unit 1) (value "+5V") (footprint "")
     )
+    (path "/33150f27-98b3-4b2a-92cc-16b50b335e66/bf9bd0ab-b178-4669-8c72-648e62946057"
+      (reference "#PWR?") (unit 1) (value "GND") (footprint "")
+    )
+    (path "/33150f27-98b3-4b2a-92cc-16b50b335e66/c142b3fb-78a7-4021-abfc-c01694965616"
+      (reference "#PWR?") (unit 1) (value "GND") (footprint "")
+    )
     (path "/13edf85d-e5b3-408c-9ca0-37b4fd7394a6/c480bd84-d1e3-42a6-a63d-95f2d2ca225a"
+      (reference "#PWR?") (unit 1) (value "GND") (footprint "")
+    )
+    (path "/33150f27-98b3-4b2a-92cc-16b50b335e66/c6328b88-b461-4428-ab62-9075960cf66f"
+      (reference "#PWR?") (unit 1) (value "GND") (footprint "")
+    )
+    (path "/33150f27-98b3-4b2a-92cc-16b50b335e66/c7b879f7-9404-47f2-80ad-e55ebbd9c561"
       (reference "#PWR?") (unit 1) (value "GND") (footprint "")
     )
@@
       (reference "U?") (unit 1) (value "PAL16L8") (footprint "")
     )
+    (path "/33150f27-98b3-4b2a-92cc-16b50b335e66/5d641701-ae71-47e2-b2b5-1195fb39dac2"
+      (reference "U?") (unit 1) (value "74AHC373") (footprint "")
+    )
+    (path "/33150f27-98b3-4b2a-92cc-16b50b335e66/9373769f-8ce9-4bcb-9b72-e5e308bd5605"
+      (reference "U?") (unit 1) (value "74AHC373") (footprint "")
+    )
+    (path "/33150f27-98b3-4b2a-92cc-16b50b335e66/9ca45473-66a2-4ee7-956f-2c5c24210e95"
+      (reference "U?") (unit 1) (value "74AHC373") (footprint "")
+    )
     (path "/ca0389f4-f711-40c0-919a-1246dc815a6c/edadb144-4be9-4c46-b55a-67edd1499a7a"

Commit message: power added
Other:
- added sheet 8255 (8255.kicad_sch)
- added sheet power (power.kicad_sch)
- sheet 28F010 ports: added VIN; removed none
- sheet 8086 ports: added VIN; removed none
- sheet ClockFinal ports: added VIN; removed none

Commit message: 8255
Other:
- sheet 8255 ports: added AIN, DATA, RESET, VIN, _RD, _WR; removed none

Commit message: 8259
Other:
- added sheet 8259 (8259.kicad_sch)
- sheet CY7C199 ports: added DOUT, VIN; removed A high

Commit message: fixes
Other:
- sheet 28F010 ports: added M/_IO; removed none
- sheet 8255 ports: added INT, M/_IO, _INTA; removed none
Changed lines of the file:
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@@
   (junction (at 118.11 49.53) (diameter 0) (color 0 0 0 0)
   )
+  (junction (at 93.98 88.9) (diameter 0) (color 0 0 0 0)
+  )
   (junction (at 194.31 24.13) (diameter 0) (color 0 0 0 0)
   )
@@
   (junction (at 144.78 86.36) (diameter 0) (color 0 0 0 0)
   )
+  (junction (at 60.96 95.25) (diameter 0) (color 0 0 0 0)
+  )
   (junction (at 143.51 59.69) (diameter 0) (color 0 0 0 0)
   )
   (junction (at 72.39 40.64) (diameter 0) (color 0 0 0 0)
   )
+  (junction (at 127 95.25) (diameter 0) (color 0 0 0 0)
+  )
   (junction (at 104.14 64.77) (diameter 0) (color 0 0 0 0)
   )
+  (junction (at 53.34 97.79) (diameter 0) (color 0 0 0 0)
+  )
   (bus (pts (xy 133.35 49.53) (xy 133.35 53.34))
     (stroke (width 0) (type default) (color 0 0 0 0))
@@
     (stroke (width 0) (type default) (color 0 0 0 0))
   )
+  (wire (pts (xy 53.34 97.79) (xy 53.34 102.87))
+    (stroke (width 0) (type default) (color 0 0 0 0))
+  )
   (bus (pts (xy 144.78 86.36) (xy 144.78 128.27))
     (stroke (width 0) (type default) (color 0 0 0 0))
@@
     (stroke (width 0) (type default) (color 0 0 0 0))
   )
+  (wire (pts (xy 127 95.25) (xy 127 67.31))
+    (stroke (width 0) (type default) (color 0 0 0 0))
+  )
   (wire (pts (xy 97.79 59.69) (xy 142.24 59.69))
     (stroke (width 0) (type default) (color 0 0 0 0))
@@
     (stroke (width 0) (type default) (color 0 0 0 0))
   )
+  (wire (pts (xy 127 95.25) (xy 153.67 95.25))
+    (stroke (width 0) (type default) (color 0 0 0 0))
+  )
   (wire (pts (xy 80.01 27.94) (xy 80.01 46.99))
     (stroke (width 0) (type default) (color 0 0 0 0))
@@
     (stroke (width 0) (type default) (color 0 0 0 0))
   )
+  (wire (pts (xy 93.98 88.9) (xy 67.31 88.9))
+    (stroke (width 0) (type default) (color 0 0 0 0))
+  )
   (bus (pts (xy 146.05 53.34) (xy 201.93 53.34))
     (stroke (width 0) (type default) (color 0 0 0 0))
@@
     (stroke (width 0) (type default) (color 0 0 0 0))
   )
+  (wire (pts (xy 93.98 88.9) (xy 93.98 96.52))
+    (stroke (width 0) (type default) (color 0 0 0 0))
+  )
+  (wire (pts (xy 67.31 88.9) (xy 67.31 102.87))
+    (stroke (width 0) (type default) (color 0 0 0 0))
+  )
   (wire (pts (xy 143.51 59.69) (xy 142.24 59.69))
     (stroke (width 0) (type default) (color 0 0 0 0))
@@
     (stroke (width 0) (type default) (color 0 0 0 0))
   )
+  (wire (pts (xy 127 67.31) (xy 201.93 67.31))
+    (stroke (width 0) (type default) (color 0 0 0 0))
+  )
   (bus (pts (xy 146.05 83.82) (xy 146.05 125.73))
     (stroke (width 0) (type default) (color 0 0 0 0))
@@
     (stroke (width 0) (type default) (color 0 0 0 0))
   )
-  (wire (pts (xy 41.91 95.25) (xy 153.67 95.25))
+  (wire (pts (xy 41.91 95.25) (xy 60.96 95.25))
     (stroke (width 0) (type default) (color 0 0 0 0))
   )
@@
     (stroke (width 0) (type default) (color 0 0 0 0))
   )
+  (wire (pts (xy 60.96 95.25) (xy 60.96 102.87))
+    (stroke (width 0) (type default) (color 0 0 0 0))
+  )
   (wire (pts (xy 130.81 93.98) (xy 157.48 93.98))
     (stroke (width 0) (type default) (color 0 0 0 0))
@@
     (stroke (width 0) (type default) (color 0 0 0 0))
   )
-  (wire (pts (xy 93.98 54.61) (xy 93.98 96.52))
+  (wire (pts (xy 93.98 54.61) (xy 93.98 88.9))
     (stroke (width 0) (type default) (color 0 0 0 0))
   )
@@
   )
   (wire (pts (xy 99.06 64.77) (xy 104.14 64.77))
+    (stroke (width 0) (type default) (color 0 0 0 0))
+  )
+  (wire (pts (xy 60.96 95.25) (xy 127 95.25))
     (stroke (width 0) (type default) (color 0 0 0 0))
   )
@@
       (effects (font (size 1.27 1.27)) (justify right))
     )
+    (pin "M{slash}_IO" input (at 201.93 67.31 180)
+      (effects (font (size 1.27 1.27)) (justify left))
+    )
   )
   (sheet (at 43.18 46.99) (size 48.26 39.37) (fields_autoplaced)
@@
       (effects (font (size 1.27 1.27)) (justify left))
     )
-    (pin "VIN" output (at 193.04 121.92 0)
+    (pin "VIN" input (at 193.04 121.92 0)
       (effects (font (size 1.27 1.27)) (justify right))
     )
@@
     )
     (pin "VIN" input (at 71.12 102.87 90)
+      (effects (font (size 1.27 1.27)) (justify right))
+    )
+    (pin "M{slash}_IO" input (at 60.96 102.87 90)
+      (effects (font (size 1.27 1.27)) (justify right))
+    )
+    (pin "INT" output (at 67.31 102.87 90)
+      (effects (font (size 1.27 1.27)) (justify right))
+    )
+    (pin "_INTA" input (at 53.34 102.87 90)
       (effects (font (size 1.27 1.27)) (justify right))
     )
@@
       (reference "SW1") (unit 1) (value "SW_DIP_x01") (footprint "")
     )
+    (path "/db110dd7-866f-4182-8c0a-892c963cb565/c6656dd3-c24e-4fce-812a-91bfb890aed5"
+      (reference "SW?") (unit 1) (value "SW_DIP_x08") (footprint "")
+    )
     (path "/c8186690-a67f-40cd-87ed-969498418dbb/6c9bbb6e-7d6d-4b3d-9a04-a28153eebc60"
       (reference "U0") (unit 1) (value "PAL16L8") (footprint "")
@@
       (reference "U?") (unit 1) (value "74AHC373") (footprint "")
     )
+    (path "/db110dd7-866f-4182-8c0a-892c963cb565/79a99526-da32-4c8f-8cda-1db7e38c6e8d"
+      (reference "U?") (unit 1) (value "74AUC2G32") (footprint "")
+    )
     (path "/db110dd7-866f-4182-8c0a-892c963cb565/91b99f18-5963-4619-add5-19923b675a26"
       (reference "U?") (unit 1) (value "PAL16L8") (footprint "")
@@
       (reference "U?") (unit 1) (value "74AHC373") (footprint "")
     )
+    (path "/db110dd7-866f-4182-8c0a-892c963cb565/a83a8be9-be31-45aa-9824-294382c6de56"
+      (reference "U?") (unit 1) (value "74AHCT04") (footprint "")
+    )
     (path "/db110dd7-866f-4182-8c0a-892c963cb565/b704e957-926b-497a-b469-1f01911cc579"
       (reference "U?") (unit 1) (value "8255") (footprint "Package_DIP:DIP-40_W15.24mm")
     )
+    (path "/db110dd7-866f-4182-8c0a-892c963cb565/c6ed3ed7-6647-437a-a7b6-6172f7793d84"
+      (reference "U?") (unit 1) (value "4011") (footprint "")
+    )
+    (path "/db110dd7-866f-4182-8c0a-892c963cb565/dbcbe67d-354a-472f-a7be-296f387299e2"
+      (reference "U?") (unit 1) (value "74LVC1G332") (footprint "")
+    )
     (path "/db110dd7-866f-4182-8c0a-892c963cb565/e17e2dcf-c8e6-4a75-9281-58df50c2fb38"
       (reference "U?") (unit 1) (value "8255") (footprint "Package_DIP:DIP-40_W15.24mm")
@@
       (reference "U?") (unit 2) (value "74LS21") (footprint "")
     )
+    (path "/db110dd7-866f-4182-8c0a-892c963cb565/2e4e3494-5151-4cd5-b479-ce36e9747643"
+      (reference "U?") (unit 2) (value "74AUC2G32") (footprint "")
+    )
+    (path "/db110dd7-866f-4182-8c0a-892c963cb565/8bcb48db-661f-46cb-b1c0-30e57d444c26"
+      (reference "U?") (unit 2) (value "74AUC2G32") (footprint "")
+    )
     (path "/c8186690-a67f-40cd-87ed-969498418dbb/8c713461-21ec-4448-baa7-43fd1d99a058"

Commit message: 16550
Other:
- added sheet 16550 (16550.kicad_sch)
