File: 8086proj/FinalProj.kicad_sch (KiCad schematic)
At the start: 0 parts

Commit message: 16550
Changed lines of the file:
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@@
   (junction (at 140.97 64.77) (diameter 0) (color 0 0 0 0)
   )
-  (junction (at 85.09 99.06) (diameter 0) (color 0 0 0 0)
-  )
-  (junction (at 97.79 110.49) (diameter 0) (color 0 0 0 0)
-  )
   (junction (at 106.68 57.15) (diameter 0) (color 0 0 0 0)
   )
-  (junction (at 93.98 114.3) (diameter 0) (color 0 0 0 0)
-  )
   (junction (at 146.05 83.82) (diameter 0) (color 0 0 0 0)
   )
@@
   (junction (at 213.36 24.13) (diameter 0) (color 0 0 0 0)
   )
-  (junction (at 86.36 118.11) (diameter 0) (color 0 0 0 0)
-  )
   (junction (at 130.81 41.91) (diameter 0) (color 0 0 0 0)
   )
@@
     (stroke (width 0) (type default) (color 0 0 0 0))
   )
-  (wire (pts (xy 115.57 149.86) (xy 200.66 138.43))
-    (stroke (width 0) (type default) (color 0 0 0 0))
-  )
-  (wire (pts (xy 78.74 147.32) (xy 85.09 135.89))
-    (stroke (width 0) (type default) (color 0 0 0 0))
-  )
-  (wire (pts (xy 200.66 138.43) (xy 200.66 113.03))
-    (stroke (width 0) (type default) (color 0 0 0 0))
-  )
   (bus (pts (xy 144.78 86.36) (xy 144.78 128.27))
     (stroke (width 0) (type default) (color 0 0 0 0))
   )
-  (wire (pts (xy 76.2 138.43) (xy 115.57 138.43))
-    (stroke (width 0) (type default) (color 0 0 0 0))
-  )
   (wire (pts (xy 93.98 96.52) (xy 156.21 96.52))
     (stroke (width 0) (type default) (color 0 0 0 0))
@@
     (stroke (width 0) (type default) (color 0 0 0 0))
   )
-  (wire (pts (xy 130.81 99.06) (xy 85.09 99.06))
+  (wire (pts (xy 130.81 99.06) (xy 71.12 99.06))
     (stroke (width 0) (type default) (color 0 0 0 0))
   )
@@
     (stroke (width 0) (type default) (color 0 0 0 0))
   )
-  (bus (pts (xy 66.04 123.19) (xy 66.04 138.43))
-    (stroke (width 0) (type default) (color 0 0 0 0))
-  )
   (bus (pts (xy 146.05 53.34) (xy 201.93 53.34))
     (stroke (width 0) (type default) (color 0 0 0 0))
@@
     (stroke (width 0) (type default) (color 0 0 0 0))
   )
-  (wire (pts (xy 85.09 99.06) (xy 71.12 99.06))
-    (stroke (width 0) (type default) (color 0 0 0 0))
-  )
   (wire (pts (xy 36.83 96.52) (xy 36.83 124.46))
     (stroke (width 0) (type default) (color 0 0 0 0))
   )
-  (wire (pts (xy 62.23 125.73) (xy 62.23 138.43))
+  (wire (pts (xy 62.23 125.73) (xy 62.23 127))
     (stroke (width 0) (type default) (color 0 0 0 0))
   )
@@
     (stroke (width 0) (type default) (color 0 0 0 0))
   )
-  (wire (pts (xy 93.98 114.3) (xy 78.74 114.3))
-    (stroke (width 0) (type default) (color 0 0 0 0))
-  )
   (wire (pts (xy 140.97 64.77) (xy 140.97 118.11))
     (stroke (width 0) (type default) (color 0 0 0 0))
@@
     (stroke (width 0) (type default) (color 0 0 0 0))
   )
-  (wire (pts (xy 115.57 138.43) (xy 115.57 149.86))
-    (stroke (width 0) (type default) (color 0 0 0 0))
-  )
-  (wire (pts (xy 85.09 135.89) (xy 85.09 99.06))
-    (stroke (width 0) (type default) (color 0 0 0 0))
-  )
   (wire (pts (xy 143.51 59.69) (xy 143.51 88.9))
     (stroke (width 0) (type default) (color 0 0 0 0))
@@
     (stroke (width 0) (type default) (color 0 0 0 0))
   )
-  (wire (pts (xy 55.88 124.46) (xy 55.88 138.43))
+  (wire (pts (xy 55.88 124.46) (xy 55.88 127))
     (stroke (width 0) (type default) (color 0 0 0 0))
   )
@@
     (stroke (width 0) (type default) (color 0 0 0 0))
   )
-  (bus (pts (xy 97.79 121.92) (xy 69.85 121.92))
-    (stroke (width 0) (type default) (color 0 0 0 0))
-  )
   (wire (pts (xy 91.44 54.61) (xy 93.98 54.61))
     (stroke (width 0) (type default) (color 0 0 0 0))
   )
-  (wire (pts (xy 93.98 114.3) (xy 93.98 120.65))
-    (stroke (width 0) (type default) (color 0 0 0 0))
-  )
-  (bus (pts (xy 106.68 110.49) (xy 97.79 110.49))
+  (bus (pts (xy 106.68 110.49) (xy 78.74 110.49))
     (stroke (width 0) (type default) (color 0 0 0 0))
   )
@@
     (stroke (width 0) (type default) (color 0 0 0 0))
   )
-  (bus (pts (xy 97.79 110.49) (xy 97.79 121.92))
-    (stroke (width 0) (type default) (color 0 0 0 0))
-  )
   (wire (pts (xy 53.34 97.79) (xy 154.94 97.79))
     (stroke (width 0) (type default) (color 0 0 0 0))
@@
     (stroke (width 0) (type default) (color 0 0 0 0))
   )
-  (wire (pts (xy 72.39 120.65) (xy 72.39 138.43))
-    (stroke (width 0) (type default) (color 0 0 0 0))
-  )
   (wire (pts (xy 142.24 120.65) (xy 157.48 120.65))
     (stroke (width 0) (type default) (color 0 0 0 0))
@@
     (stroke (width 0) (type default) (color 0 0 0 0))
   )
-  (wire (pts (xy 93.98 120.65) (xy 72.39 120.65))
-    (stroke (width 0) (type default) (color 0 0 0 0))
-  )
-  (wire (pts (xy 59.69 124.46) (xy 59.69 138.43))
+  (wire (pts (xy 59.69 124.46) (xy 59.69 127))
     (stroke (width 0) (type default) (color 0 0 0 0))
   )
@@
     (stroke (width 0) (type default) (color 0 0 0 0))
   )
-  (bus (pts (xy 97.79 110.49) (xy 78.74 110.49))
-    (stroke (width 0) (type default) (color 0 0 0 0))
-  )
   (wire (pts (xy 95.25 78.74) (xy 95.25 105.41))
     (stroke (width 0) (type default) (color 0 0 0 0))
@@
     (stroke (width 0) (type default) (color 0 0 0 0))
   )
-  (bus (pts (xy 86.36 118.11) (xy 86.36 123.19))
-    (stroke (width 0) (type default) (color 0 0 0 0))
-  )
-  (bus (pts (xy 86.36 123.19) (xy 66.04 123.19))
-    (stroke (width 0) (type default) (color 0 0 0 0))
-  )
   (wire (pts (xy 90.17 125.73) (xy 62.23 125.73))
     (stroke (width 0) (type default) (color 0 0 0 0))
@@
     (stroke (width 0) (type default) (color 0 0 0 0))
   )
-  (bus (pts (xy 118.11 118.11) (xy 86.36 118.11))
+  (bus (pts (xy 118.11 118.11) (xy 78.74 118.11))
     (stroke (width 0) (type default) (color 0 0 0 0))
   )
@@
     (stroke (width 0) (type default) (color 0 0 0 0))
   )
-  (wire (pts (xy 200.66 113.03) (xy 193.04 113.03))
-    (stroke (width 0) (type default) (color 0 0 0 0))
-  )
   (wire (pts (xy 154.94 97.79) (xy 154.94 115.57))
     (stroke (width 0) (type default) (color 0 0 0 0))
   )
-  (bus (pts (xy 86.36 118.11) (xy 78.74 118.11))
-    (stroke (width 0) (type default) (color 0 0 0 0))
-  )
   (wire (pts (xy 50.8 96.52) (xy 50.8 102.87))
     (stroke (width 0) (type default) (color 0 0 0 0))
   )
-  (bus (pts (xy 69.85 121.92) (xy 69.85 138.43))
-    (stroke (width 0) (type default) (color 0 0 0 0))
-  )
   (wire (pts (xy 130.81 41.91) (xy 83.82 41.91))
     (stroke (width 0) (type default) (color 0 0 0 0))
@@
     (stroke (width 0) (type default) (color 0 0 0 0))
   )
-  (wire (pts (xy 104.14 114.3) (xy 93.98 114.3))
+  (wire (pts (xy 104.14 114.3) (xy 78.74 114.3))
     (stroke (width 0) (type default) (color 0 0 0 0))
   )
@@
     )
   )
-  (sheet (at 46.99 138.43) (size 31.75 15.24) (fields_autoplaced)
+  (sheet (at 46.99 127) (size 31.75 15.24) (fields_autoplaced)
     (stroke (width 0.1524) (type solid) (color 0 0 0 0))
     (fill (color 0 0 0 0.0000))
-    (property "Sheet name" "16550" (id 0) (at 46.2784 153.67 90)
+    (property "Sheet name" "16550" (id 0) (at 46.2784 142.24 90)
       (effects (font (size 1.27 1.27)) (justify left bottom))
     )
-    (property "Sheet file" "16550.kicad_sch" (id 1) (at 79.3246 153.67 90)
+    (property "Sheet file" "16550.kicad_sch" (id 1) (at 79.3246 142.24 90)
       (effects (font (size 1.27 1.27)) (justify left top))
     )
-    (pin "AIN" input (at 66.04 138.43 90)
-      (effects (font (size 1.27 1.27)) (justify right))
-    )
-    (pin "DATA" bidirectional (at 69.85 138.43 90)
-      (effects (font (size 1.27 1.27)) (justify right))
-    )
-    (pin "M{slash}_IO" input (at 62.23 138.43 90)
-      (effects (font (size 1.27 1.27)) (justify right))
-    )
-    (pin "_WR" input (at 72.39 138.43 90)
-      (effects (font (size 1.27 1.27)) (justify right))
-    )
-    (pin "INTR" output (at 76.2 138.43 90)
-      (effects (font (size 1.27 1.27)) (justify right))
-    )
-    (pin "_RD" input (at 59.69 138.43 90)
-      (effects (font (size 1.27 1.27)) (justify right))
-    )
-    (pin "MR" input (at 55.88 138.43 90)
-      (effects (font (size 1.27 1.27)) (justify right))
-    )
-    (pin "VIN" input (at 78.74 147.32 0)
+    (pin "AIN" input (at 66.04 127 90)
+      (effects (font (size 1.27 1.27)) (justify right))
+    )
+    (pin "DATA" bidirectional (at 69.85 127 90)
+      (effects (font (size 1.27 1.27)) (justify right))
+    )
+    (pin "M{slash}_IO" input (at 62.23 127 90)
+      (effects (font (size 1.27 1.27)) (justify right))
+    )
+    (pin "_WR" input (at 72.39 127 90)
+      (effects (font (size 1.27 1.27)) (justify right))
+    )
+    (pin "INTR" output (at 76.2 127 90)
+      (effects (font (size 1.27 1.27)) (justify right))
+    )
+    (pin "_RD" input (at 59.69 127 90)
+      (effects (font (size 1.27 1.27)) (justify right))
+    )
+    (pin "MR" input (at 55.88 127 90)
+      (effects (font (size 1.27 1.27)) (justify right))
+    )
+    (pin "VIN" input (at 78.74 135.89 0)
       (effects (font (size 1.27 1.27)) (justify right))
     )
@@
       (reference "#PWR0134") (unit 1) (value "GND") (footprint "")
     )
-    (path "/be3f0182-1888-4a47-ad24-125d3a138d53/16e489eb-844e-4b76-9f36-0689e71ac525"
+    (path "/be3f0182-1888-4a47-ad24-125d3a138d53/3afd0546-0cbc-4692-b2c9-b49fb88ee908"
       (reference "#PWR?") (unit 1) (value "GND") (footprint "")
     )
@@
       (reference "#PWR?") (unit 1) (value "GND") (footprint "")
     )
+    (path "/be3f0182-1888-4a47-ad24-125d3a138d53/8a2ca719-efac-4c53-bb04-d2caeaf41dc3"
+      (reference "#PWR?") (unit 1) (value "GND") (footprint "")
+    )
     (path "/be3f0182-1888-4a47-ad24-125d3a138d53/9ee42518-ab21-4367-b4e7-d2f79c9f576b"
       (reference "#PWR?") (unit 1) (value "GND") (footprint "")
     )
-    (path "/be3f0182-1888-4a47-ad24-125d3a138d53/b48586e2-5a37-471d-a2d3-40539d2bffa4"
+    (path "/be3f0182-1888-4a47-ad24-125d3a138d53/beed13cc-723b-482d-9b68-ed77d6b867bd"
       (reference "#PWR?") (unit 1) (value "GND") (footprint "")
     )
