File: 8086proj/FinalProj.kicad_sch (KiCad schematic)
At the start: 0 parts

Commit message: LCD
Other:
- added sheet LCD (LCD.kicad_sch)

Commit message: 7seg
Other:
- added sheet 7seg (7seg.kicad_sch)

Commit message: 74244
Other:
- added sheet 74374 (74374.kicad_sch)
- sheet CY7C199 ports: added M/_IO; removed none

Commit message: fixes
Other:
- sheet 8086 ports: added none; removed DR/_R, HLDA, MIN/_MAX, _BHE/S7, _DEN
- sheet 8254 ports: added none; removed CLK
- sheet 8259 ports: added none; removed IR0
- sheet 8279 ports: added 8279 IRG; removed IR0
