File: 8086proj/8086_sch.kicad_sch (KiCad schematic)
At the start: 1 part

Commit message: 28F010.kicad_sch
Parts:
- gave numbers to parts that had none: 1
Changed lines of the file:
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@@
     (stroke (width 0) (type default) (color 0 0 0 0))
+  )
+  (label "A[16..19]" (at 119.38 109.22 0)
+    (effects (font (size 1.27 1.27)) (justify left bottom))
+  )
+  (label "A[0..15]" (at 119.38 78.74 0)
+    (effects (font (size 1.27 1.27)) (justify left bottom))
   )
   (hierarchical_label "_DEN" (shape output) (at 125.73 49.53 0)
@@
   (symbol (lib_id "power:+5V") (at 95.25 31.75 180) (unit 1)
     (in_bom yes) (on_board yes) (fields_autoplaced)
-    (property "Reference" "#PWR?" (id 0) (at 95.25 27.94 0)
+    (property "Reference" "#PWR0101" (id 0) (at 95.25 27.94 0)
       (effects (font (size 1.27 1.27)) hide)
     )
@@
   (symbol (lib_id "MCU_Intel:8086_Min_Mode") (at 95.25 85.09 0) (unit 1)
     (in_bom yes) (on_board yes) (fields_autoplaced)
-    (property "Reference" "U?" (id 0) (at 97.2694 38.1 0)
+    (property "Reference" "U1" (id 0) (at 97.2694 38.1 0)
       (effects (font (size 1.27 1.27)) (justify left))
     )
@@
   (symbol (lib_id "power:GND") (at 95.25 134.62 0) (unit 1)
     (in_bom yes) (on_board yes) (fields_autoplaced)
-    (property "Reference" "#PWR?" (id 0) (at 95.25 140.97 0)
+    (property "Reference" "#PWR0102" (id 0) (at 95.25 140.97 0)
       (effects (font (size 1.27 1.27)) hide)
     )

Commit message: latch added
Parts:
- added U? (x2): 74AHC373, symbol 74xx:74AHC373
- added U?: (no value), symbol 74xx:74AHC373
Connections:
- net GND: now also U?.1 (OE), U?.1 (OE), U?.1 (OE), U?.10 (GND), U?.10 (GND), U?.10 (GND)
- net at U1.35 (A19/S6): now also U?.8 (D3)
- net at U1.36 (A18/S5): now also U?.7 (D2)
- net at U1.37 (A17/S4): now also U?.4 (D1)
- net at U1.38 (A16/S3): now also U?.3 (D0)
- net ALE: no longer names the net of U1.25 (ALE)
- net ALE: now also U?.11 (LE), U?.11 (LE), U?.11 (LE)
- new net D0: U?.3 (D0)
- new net D1: U?.4 (D1)
- new net D10: U?.7 (D2)
- new net D11: U?.8 (D3)
- new net D12: U?.13 (D4)
- new net D13: U?.14 (D5)
- new net D14: U?.17 (D6)
- new net D15: U?.18 (D7)
- new net D2: U?.7 (D2)
- new net D3: U?.8 (D3)
- new net D4: U?.13 (D4)
- new net D5: U?.14 (D5)
- new net D6: U?.17 (D6)
- new net D7: U?.18 (D7)
- new net D8: U?.3 (D0)
- new net D9: U?.4 (D1)
- no-connect marks 0 -> 8

Commit message: power added
Parts:
- added C?: 10uF, symbol Device:C
- added C? (x3): (no value), symbol Device:C
Connections:
- net +5V is gone; now on net VIN: U1.40 (VCC)
- net GND: now also C?.1, C?.2, C?.2
- net VIN: now reaches U?.20 (VCC)
- net VIN: now also U?.20 (VCC), U?.20 (VCC), C?.1, C?.1, C?.1, C?.2

Commit message: power added
Parts:
- removed C?: 10uF, symbol Device:C
- removed C? (x2): (no value), symbol Device:C
Changed lines of the file:
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@@
   (junction (at 170.18 52.07) (diameter 0) (color 0 0 0 0)
-  )
-  (junction (at 233.68 33.02) (diameter 0) (color 0 0 0 0)
-  )
-  (junction (at 135.89 30.48) (diameter 0) (color 0 0 0 0)
-  )
-  (junction (at 184.15 33.02) (diameter 0) (color 0 0 0 0)
   )
   (junction (at 129.54 30.48) (diameter 0) (color 0 0 0 0)
@@
     (stroke (width 0) (type default) (color 0 0 0 0))
   )
-  (wire (pts (xy 135.89 30.48) (xy 138.43 30.48))
+  (wire (pts (xy 129.54 30.48) (xy 138.43 30.48))
     (stroke (width 0) (type default) (color 0 0 0 0))
   )
@@
     (stroke (width 0) (type default) (color 0 0 0 0))
   )
-  (wire (pts (xy 184.15 22.86) (xy 189.23 22.86))
-    (stroke (width 0) (type default) (color 0 0 0 0))
-  )
   (wire (pts (xy 233.68 33.02) (xy 233.68 48.26))
     (stroke (width 0) (type default) (color 0 0 0 0))
@@
     (stroke (width 0) (type default) (color 0 0 0 0))
   )
-  (wire (pts (xy 129.54 30.48) (xy 135.89 30.48))
-    (stroke (width 0) (type default) (color 0 0 0 0))
-  )
   (wire (pts (xy 147.32 19.05) (xy 147.32 20.32))
     (stroke (width 0) (type default) (color 0 0 0 0))
@@
     (stroke (width 0) (type default) (color 0 0 0 0))
   )
-  (wire (pts (xy 135.89 22.86) (xy 140.97 22.86))
-    (stroke (width 0) (type default) (color 0 0 0 0))
-  )
   (bus (pts (xy 199.39 16.51) (xy 201.93 16.51))
     (stroke (width 0) (type default) (color 0 0 0 0))
@@
     (stroke (width 0) (type default) (color 0 0 0 0))
   )
-  (wire (pts (xy 233.68 30.48) (xy 233.68 33.02))
-    (stroke (width 0) (type default) (color 0 0 0 0))
-  )
   (bus (pts (xy 245.11 16.51) (xy 247.65 16.51))
     (stroke (width 0) (type default) (color 0 0 0 0))
@@
     (stroke (width 0) (type default) (color 0 0 0 0))
   )
-  (wire (pts (xy 189.23 22.86) (xy 189.23 25.4))
-    (stroke (width 0) (type default) (color 0 0 0 0))
-  )
   (bus (pts (xy 196.85 16.51) (xy 199.39 16.51))
     (stroke (width 0) (type default) (color 0 0 0 0))
@@
     (stroke (width 0) (type default) (color 0 0 0 0))
   )
-  (wire (pts (xy 233.68 22.86) (xy 237.49 22.86))
-    (stroke (width 0) (type default) (color 0 0 0 0))
-  )
   (bus (pts (xy 157.48 16.51) (xy 160.02 16.51))
     (stroke (width 0) (type default) (color 0 0 0 0))
@@
     (stroke (width 0) (type default) (color 0 0 0 0))
   )
-  (wire (pts (xy 184.15 30.48) (xy 184.15 33.02))
-    (stroke (width 0) (type default) (color 0 0 0 0))
-  )
   (wire (pts (xy 242.57 102.87) (xy 242.57 45.72))
     (stroke (width 0) (type default) (color 0 0 0 0))
@@
     (stroke (width 0) (type default) (color 0 0 0 0))
   )
-  (wire (pts (xy 237.49 22.86) (xy 237.49 25.4))
-    (stroke (width 0) (type default) (color 0 0 0 0))
-  )
   (wire (pts (xy 120.65 45.72) (xy 120.65 46.99))
     (stroke (width 0) (type default) (color 0 0 0 0))
@@
   )
   (bus (pts (xy 167.64 16.51) (xy 196.85 16.51))
-    (stroke (width 0) (type default) (color 0 0 0 0))
-  )
-  (wire (pts (xy 140.97 22.86) (xy 140.97 24.13))
     (stroke (width 0) (type default) (color 0 0 0 0))
   )
@@
   (hierarchical_label "_DEN" (shape bidirectional) (at 125.73 49.53 0)
     (effects (font (size 1.27 1.27)) (justify left))
-  )
-  (symbol (lib_id "power:GND") (at 189.23 25.4 0) (unit 1)
-    (in_bom yes) (on_board yes) (fields_autoplaced)
-    (property "Reference" "#PWR?" (id 0) (at 189.23 31.75 0)
-      (effects (font (size 1.27 1.27)) hide)
-    )
-    (property "Value" "GND" (id 1) (at 189.23 30.48 0))
-    (property "Footprint" "" (id 2) (at 189.23 25.4 0)
-      (effects (font (size 1.27 1.27)) hide)
-    )
-    (property "Datasheet" "" (id 3) (at 189.23 25.4 0)
-      (effects (font (size 1.27 1.27)) hide)
-    )
-    (pin "1")
-  )
-  (symbol (lib_id "Device:C") (at 184.15 26.67 180) (unit 1)
-    (in_bom yes) (on_board yes) (fields_autoplaced)
-    (property "Reference" "C?" (id 0) (at 180.34 27.9401 0)
-      (effects (font (size 1.27 1.27)) (justify left))
-    )
-    (property "Value" "10uF" (id 1) (at 180.34 25.4001 0)
-      (effects (font (size 1.27 1.27)) (justify left))
-    )
-    (property "Footprint" "" (id 2) (at 183.1848 22.86 0)
-      (effects (font (size 1.27 1.27)) hide)
-    )
-    (property "Datasheet" "~" (id 3) (at 184.15 26.67 0)
-      (effects (font (size 1.27 1.27)) hide)
-    )
-    (pin "1")
-    (pin "2")
   )
   (symbol (lib_id "Device:C") (at 99.06 31.75 270) (unit 1)
@@
     (pin "1")
     (pin "2")
-  )
-  (symbol (lib_id "power:GND") (at 238.76 25.4 0) (unit 1)
-    (in_bom yes) (on_board yes) (fields_autoplaced)
-    (property "Reference" "#PWR?" (id 0) (at 238.76 31.75 0)
-      (effects (font (size 1.27 1.27)) hide)
-    )
-    (property "Value" "GND" (id 1) (at 238.76 30.48 0))
-    (property "Footprint" "" (id 2) (at 238.76 25.4 0)
-      (effects (font (size 1.27 1.27)) hide)
-    )
-    (property "Datasheet" "" (id 3) (at 238.76 25.4 0)
-      (effects (font (size 1.27 1.27)) hide)
-    )
-    (pin "1")
   )
   (symbol (lib_id "MCU_Intel:8086_Min_Mode") (at 95.25 85.09 0) (unit 1)
@@
     (pin "1")
   )
-  (symbol (lib_id "power:GND") (at 140.97 24.13 0) (unit 1)
-    (in_bom yes) (on_board yes) (fields_autoplaced)
-    (property "Reference" "#PWR?" (id 0) (at 140.97 30.48 0)
-      (effects (font (size 1.27 1.27)) hide)
-    )
-    (property "Value" "" (id 1) (at 140.97 29.21 0))
-    (property "Footprint" "" (id 2) (at 140.97 24.13 0)
-      (effects (font (size 1.27 1.27)) hide)
-    )
-    (property "Datasheet" "" (id 3) (at 140.97 24.13 0)
-      (effects (font (size 1.27 1.27)) hide)
-    )
-    (pin "1")
-  )
   (symbol (lib_id "power:GND") (at 180.34 33.02 0) (unit 1)
     (in_bom yes) (on_board yes) (fields_autoplaced)
@@
     (pin "1")
   )
-  (symbol (lib_id "Device:C") (at 233.68 26.67 180) (unit 1)
-    (in_bom yes) (on_board yes) (fields_autoplaced)
-    (property "Reference" "C?" (id 0) (at 229.87 27.9401 0)
-      (effects (font (size 1.27 1.27)) (justify left))
-    )
-    (property "Value" "" (id 1) (at 229.87 25.4001 0)
-      (effects (font (size 1.27 1.27)) (justify left))
-    )
-    (property "Footprint" "" (id 2) (at 232.7148 22.86 0)
-      (effects (font (size 1.27 1.27)) hide)
-    )
-    (property "Datasheet" "~" (id 3) (at 233.68 26.67 0)
-      (effects (font (size 1.27 1.27)) hide)
-    )
-    (pin "1")
-    (pin "2")
-  )
-  (symbol (lib_id "Device:C") (at 135.89 26.67 180) (unit 1)
-    (in_bom yes) (on_board yes) (fields_autoplaced)
-    (property "Reference" "C?" (id 0) (at 132.08 27.9401 0)
-      (effects (font (size 1.27 1.27)) (justify left))
-    )
-    (property "Value" "" (id 1) (at 132.08 25.4001 0)
-      (effects (font (size 1.27 1.27)) (justify left))
-    )
-    (property "Footprint" "" (id 2) (at 134.9248 22.86 0)
-      (effects (font (size 1.27 1.27)) hide)
-    )
-    (property "Datasheet" "~" (id 3) (at 135.89 26.67 0)
-      (effects (font (size 1.27 1.27)) hide)
-    )
-    (pin "1")
-    (pin "2")
-  )
 )

Commit message: 8255
Parts:
- added J?: (no value), symbol Connector:Conn_01x15_Female
- added J?: (no value), symbol Connector:Conn_01x16_Female
- added J?: (no value), symbol Connector:Conn_01x20_Female
Connections:
- net D0: now also J?.1 (Pin_1)
- net D1: now also J?.2 (Pin_2)
- net D10: now also J?.11 (Pin_11)
- net D11: now also J?.12 (Pin_12)
- net D12: now also J?.13 (Pin_13)
- net D13: now also J?.14 (Pin_14)
- net D14: now also J?.15 (Pin_15)
- net D15: now also J?.16 (Pin_16)
- net D2: now also J?.3 (Pin_3)
- net D3: now also J?.4 (Pin_4)
- net D4: now also J?.5 (Pin_5)
- net D5: now also J?.6 (Pin_6)
- net D6: now also J?.7 (Pin_7)
- net D7: now also J?.8 (Pin_8)
- net D8: now also J?.9 (Pin_9)
- net D9: now also J?.10 (Pin_10)
- net DR/_R: now also J?.1 (Pin_1)
- net HLDA: now also J?.9 (Pin_9)
- net HOLD: now also J?.8 (Pin_8)
- net INTR: now also J?.11 (Pin_11)
- net MIN/_MAX: now also J?.7 (Pin_7)
- net M/_IO: now also J?.3 (Pin_3)
- net NMI: now also J?.12 (Pin_12)
- net READY: now also J?.14 (Pin_14)
- net RESET: now also J?.13 (Pin_13)
- net _INTA: now also J?.6 (Pin_6)
- net _RD: now also J?.5 (Pin_5)
- net _TEST: now also J?.10 (Pin_10)
- net _WR: now also J?.4 (Pin_4)
- new net A0: J?.1 (Pin_1)
- new net A1: J?.2 (Pin_2)
- new net A10: J?.11 (Pin_11)
- new net A11: J?.12 (Pin_12)
- new net A12: J?.13 (Pin_13)
- new net A13: J?.14 (Pin_14)
- new net A14: J?.15 (Pin_15)
- new net A15: J?.16 (Pin_16)
- new net A16: J?.17 (Pin_17)
- new net A17: J?.18 (Pin_18)
- new net A18: J?.19 (Pin_19)
- new net A19: J?.20 (Pin_20)
- new net A2: J?.3 (Pin_3)
- new net A3: J?.4 (Pin_4)
- new net A4: J?.5 (Pin_5)
- new net A5: J?.6 (Pin_6)
- new net A6: J?.7 (Pin_7)
- new net A7: J?.8 (Pin_8)
- new net A8: J?.9 (Pin_9)
- new net A9: J?.10 (Pin_10)
- no-connect marks 8 -> 9

Commit message: 8259
Parts:
- C?: value (none) -> .1uF
- J?: value (none) -> Conn_01x15_Female
- J?: value (none) -> Conn_01x16_Female
- J?: value (none) -> Conn_01x20_Female
- U?: value (none) -> 74AHC373
Changed lines of the file:
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@@
     (in_bom yes) (on_board yes) (fields_autoplaced)
     (property "Reference" "C?" (id 0) (at 99.06 24.13 90))
-    (property "Value" "" (id 1) (at 99.06 26.67 90))
+    (property "Value" ".1uF" (id 1) (at 99.06 26.67 90))
     (property "Footprint" "" (id 2) (at 95.25 32.7152 0)
       (effects (font (size 1.27 1.27)) hide)
@@
       (effects (font (size 1.27 1.27)) (justify left))
     )
-    (property "Value" "" (id 1) (at 176.53 137.1599 0)
+    (property "Value" "Conn_01x15_Female" (id 1) (at 176.53 137.1599 0)
       (effects (font (size 1.27 1.27)) (justify left))
     )
@@
       (effects (font (size 1.27 1.27)) hide)
     )
-    (property "Value" "" (id 1) (at 172.72 50.8 0))
+    (property "Value" "GND" (id 1) (at 172.72 50.8 0))
     (property "Footprint" "" (id 2) (at 172.72 45.72 0)
       (effects (font (size 1.27 1.27)) hide)
@@
       (effects (font (size 1.27 1.27)) hide)
     )
-    (property "Value" "" (id 1) (at 180.34 38.1 0))
+    (property "Value" "GND" (id 1) (at 180.34 38.1 0))
     (property "Footprint" "" (id 2) (at 180.34 33.02 0)
       (effects (font (size 1.27 1.27)) hide)
@@
     (in_bom yes) (on_board yes) (fields_autoplaced)
     (property "Reference" "U?" (id 0) (at 181.61 29.4386 90))
-    (property "Value" "" (id 1) (at 181.61 31.9786 90))
+    (property "Value" "74AHC373" (id 1) (at 181.61 31.9786 90))
     (property "Footprint" "" (id 2) (at 160.02 33.02 0)
       (effects (font (size 1.27 1.27)) hide)
@@
       (effects (font (size 1.27 1.27)) hide)
     )
-    (property "Value" "" (id 1) (at 105.41 39.37 0))
+    (property "Value" "GND" (id 1) (at 105.41 39.37 0))
     (property "Footprint" "" (id 2) (at 105.41 34.29 0)
       (effects (font (size 1.27 1.27)) hide)
@@
       (effects (font (size 1.27 1.27)) hide)
     )
-    (property "Value" "" (id 1) (at 219.71 50.8 0))
+    (property "Value" "GND" (id 1) (at 219.71 50.8 0))
     (property "Footprint" "" (id 2) (at 219.71 45.72 0)
       (effects (font (size 1.27 1.27)) hide)
@@
       (effects (font (size 1.27 1.27)) hide)
     )
-    (property "Value" "" (id 1) (at 267.97 50.8 0))
+    (property "Value" "GND" (id 1) (at 267.97 50.8 0))
     (property "Footprint" "" (id 2) (at 267.97 45.72 0)
       (effects (font (size 1.27 1.27)) hide)
@@
       (effects (font (size 1.27 1.27)) (justify left))
     )
-    (property "Value" "" (id 1) (at 279.4 134.6199 0)
+    (property "Value" "Conn_01x16_Female" (id 1) (at 279.4 134.6199 0)
       (effects (font (size 1.27 1.27)) (justify left))
     )
@@
       (effects (font (size 1.27 1.27)) (justify left))
     )
-    (property "Value" "" (id 1) (at 279.4 86.3599 0)
-      (effects (font (size 1.27 1.27)) (justify left))
-    )
+    (property "Value" "Conn_01x20_Female" (id 1) (at 279.4 86.3599 0)
+      (effects (font (size 1.27 1.27)) (justify left))
+    )

Commit message: fixes
Parts:
- removed J?: Conn_01x15_Female, symbol Connector:Conn_01x15_Female
- removed J?: Conn_01x16_Female, symbol Connector:Conn_01x16_Female
- removed J?: Conn_01x20_Female, symbol Connector:Conn_01x20_Female
- added J?: (no value), symbol Connector:Conn_01x16_Male
- added J?: (no value), symbol Connector:Conn_01x15_Male
- added J?: (no value), symbol Connector:Conn_01x20_Male
Connections:
- net A0: now also J?.20 (Pin_20)
- net A1: now also J?.19 (Pin_19)
- net A10: now also J?.10 (Pin_10)
- net A11: now also J?.9 (Pin_9)
- net A12: now also J?.8 (Pin_8)
- net A13: now also J?.7 (Pin_7)
- net A14: now also J?.6 (Pin_6)
- net A15: now also J?.5 (Pin_5)
- net A16: now also J?.4 (Pin_4)
- net A17: now also J?.3 (Pin_3)
- net A18: now also J?.2 (Pin_2)
- net A19: now also J?.1 (Pin_1)
- net A2: now also J?.18 (Pin_18)
- net A3: now also J?.17 (Pin_17)
- net A4: now also J?.16 (Pin_16)
- net A5: now also J?.15 (Pin_15)
- net A6: now also J?.14 (Pin_14)
- net A7: now also J?.13 (Pin_13)
- net A8: now also J?.12 (Pin_12)
- net A9: now also J?.11 (Pin_11)
- net D0: now also J?.16 (Pin_16)
- net D1: now also J?.15 (Pin_15)
- net D10: now also J?.6 (Pin_6)
- net D11: now also J?.5 (Pin_5)
- net D12: now also J?.4 (Pin_4)
- net D13: now also J?.3 (Pin_3)
- net D14: now also J?.2 (Pin_2)
- net D15: now also J?.1 (Pin_1)
- net D2: now also J?.14 (Pin_14)
- net D3: now also J?.13 (Pin_13)
- net D4: now also J?.12 (Pin_12)
- net D5: now also J?.11 (Pin_11)
- net D6: now also J?.10 (Pin_10)
- net D7: now also J?.9 (Pin_9)
- net D8: now also J?.8 (Pin_8)
- net D9: now also J?.7 (Pin_7)
- net INTR: now also J?.5 (Pin_5)
- net M/_IO: now also J?.13 (Pin_13)
- net NMI: now also J?.4 (Pin_4)
- net READY: now also J?.2 (Pin_2)
- net RESET: now also J?.3 (Pin_3)
- net _INTA: now also J?.10 (Pin_10)
- net _RD: now also J?.11 (Pin_11)
- net _TEST: now also J?.6 (Pin_6)
- net _WR: now also J?.12 (Pin_12)
- net DR/_R: no longer names the net of U1.27 (DT/~{R})
- net DR/_R: now also J?.15 (Pin_15)
- net HLDA: no longer names the net of U1.30 (HLDA)
- net HLDA: now also J?.7 (Pin_7)
- net HOLD: no longer names the net of U1.31 (HOLD)
- net HOLD: now also J?.8 (Pin_8)
- net MIN/_MAX: no longer names the net of U1.33 (MN/~{MX})
- net MIN/_MAX: now also J?.9 (Pin_9)
- net _BHE/S7: no longer names the net of U1.34 (~{BHE}/S7)
- net _DEN: no longer names the net of U1.26 (~{DEN})
- net _DEN: now also J?.14 (Pin_14)
- no-connect marks 9 -> 10
