File: 8086proj/8086_sch.kicad_sch (KiCad schematic)
At the start: 8 parts, among them U1 8086_Min_Mode

Commit message: final look
Parts:
- J201: renamed from J?; value (none) -> Conn_01x15_Male
- J202: renamed from J?; value (none) -> Conn_01x20_Male
- J203: renamed from J?; value (none) -> Conn_01x16_Male
- gave numbers to parts that had none: 4
- renumbered U1 to U201
Changed lines of the file:
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@@
   (symbol (lib_id "Device:C") (at 99.06 31.75 270) (unit 1)
     (in_bom yes) (on_board yes) (fields_autoplaced)
-    (property "Reference" "C?" (id 0) (at 99.06 24.13 90))
+    (property "Reference" "C201" (id 0) (at 99.06 24.13 90))
     (property "Value" ".1uF" (id 1) (at 99.06 26.67 90))
     (property "Footprint" "" (id 2) (at 95.25 32.7152 0)
@@
   (symbol (lib_id "Connector:Conn_01x16_Male") (at 265.43 134.62 180) (unit 1)
     (in_bom yes) (on_board yes) (fields_autoplaced)
-    (property "Reference" "J?" (id 0) (at 266.7 132.0799 0)
-      (effects (font (size 1.27 1.27)) (justify right))
-    )
-    (property "Value" "" (id 1) (at 266.7 134.6199 0)
+    (property "Reference" "J203" (id 0) (at 266.7 132.0799 0)
+      (effects (font (size 1.27 1.27)) (justify right))
+    )
+    (property "Value" "Conn_01x16_Male" (id 1) (at 266.7 134.6199 0)
       (effects (font (size 1.27 1.27)) (justify right))
     )
@@
   (symbol (lib_id "MCU_Intel:8086_Min_Mode") (at 95.25 85.09 0) (unit 1)
     (in_bom yes) (on_board yes) (fields_autoplaced)
-    (property "Reference" "U1" (id 0) (at 97.2694 38.1 0)
+    (property "Reference" "U201" (id 0) (at 97.2694 38.1 0)
       (effects (font (size 1.27 1.27)) (justify left))
     )
@@
   (symbol (lib_id "74xx:74AHC373") (at 207.01 33.02 90) (unit 1)
     (in_bom yes) (on_board yes) (fields_autoplaced)
-    (property "Reference" "U?" (id 0) (at 228.6 29.4386 90))
+    (property "Reference" "U203" (id 0) (at 228.6 29.4386 90))
     (property "Value" "74AHC373" (id 1) (at 228.6 31.9786 90))
     (property "Footprint" "" (id 2) (at 207.01 33.02 0)
@@
   (symbol (lib_id "power:GND") (at 172.72 45.72 0) (unit 1)
     (in_bom yes) (on_board yes) (fields_autoplaced)
-    (property "Reference" "#PWR0108" (id 0) (at 172.72 52.07 0)
+    (property "Reference" "#PWR0203" (id 0) (at 172.72 52.07 0)
       (effects (font (size 1.27 1.27)) hide)
     )
@@
   (symbol (lib_id "power:GND") (at 95.25 134.62 0) (unit 1)
     (in_bom yes) (on_board yes) (fields_autoplaced)
-    (property "Reference" "#PWR0102" (id 0) (at 95.25 140.97 0)
+    (property "Reference" "#PWR0201" (id 0) (at 95.25 140.97 0)
       (effects (font (size 1.27 1.27)) hide)
     )
@@
   (symbol (lib_id "power:GND") (at 180.34 33.02 0) (unit 1)
     (in_bom yes) (on_board yes) (fields_autoplaced)
-    (property "Reference" "#PWR0107" (id 0) (at 180.34 39.37 0)
+    (property "Reference" "#PWR0204" (id 0) (at 180.34 39.37 0)
       (effects (font (size 1.27 1.27)) hide)
     )
@@
   (symbol (lib_id "74xx:74AHC373") (at 255.27 33.02 90) (unit 1)
     (in_bom yes) (on_board yes) (fields_autoplaced)
-    (property "Reference" "U?" (id 0) (at 276.86 29.4386 90))
+    (property "Reference" "U204" (id 0) (at 276.86 29.4386 90))
     (property "Value" "74AHC373" (id 1) (at 276.86 31.9786 90))
     (property "Footprint" "" (id 2) (at 255.27 33.02 0)
@@
   (symbol (lib_id "Connector:Conn_01x15_Male") (at 175.26 135.89 180) (unit 1)
     (in_bom yes) (on_board yes) (fields_autoplaced)
-    (property "Reference" "J?" (id 0) (at 176.53 134.6199 0)
-      (effects (font (size 1.27 1.27)) (justify right))
-    )
-    (property "Value" "" (id 1) (at 176.53 137.1599 0)
+    (property "Reference" "J201" (id 0) (at 176.53 134.6199 0)
+      (effects (font (size 1.27 1.27)) (justify right))
+    )
+    (property "Value" "Conn_01x15_Male" (id 1) (at 176.53 137.1599 0)
       (effects (font (size 1.27 1.27)) (justify right))
     )
@@
   (symbol (lib_id "74xx:74AHC373") (at 160.02 33.02 90) (unit 1)
     (in_bom yes) (on_board yes) (fields_autoplaced)
-    (property "Reference" "U?" (id 0) (at 181.61 29.4386 90))
+    (property "Reference" "U202" (id 0) (at 181.61 29.4386 90))
     (property "Value" "74AHC373" (id 1) (at 181.61 31.9786 90))
     (property "Footprint" "" (id 2) (at 160.02 33.02 0)
@@
   (symbol (lib_id "power:GND") (at 105.41 34.29 0) (unit 1)
     (in_bom yes) (on_board yes) (fields_autoplaced)
-    (property "Reference" "#PWR0101" (id 0) (at 105.41 40.64 0)
+    (property "Reference" "#PWR0202" (id 0) (at 105.41 40.64 0)
       (effects (font (size 1.27 1.27)) hide)
     )
@@
   (symbol (lib_id "power:GND") (at 219.71 45.72 0) (unit 1)
     (in_bom yes) (on_board yes) (fields_autoplaced)
-    (property "Reference" "#PWR0103" (id 0) (at 219.71 52.07 0)
+    (property "Reference" "#PWR0205" (id 0) (at 219.71 52.07 0)
       (effects (font (size 1.27 1.27)) hide)
     )
@@
   (symbol (lib_id "power:GND") (at 267.97 45.72 0) (unit 1)
     (in_bom yes) (on_board yes) (fields_autoplaced)
-    (property "Reference" "#PWR0105" (id 0) (at 267.97 52.07 0)
+    (property "Reference" "#PWR0207" (id 0) (at 267.97 52.07 0)
       (effects (font (size 1.27 1.27)) hide)
     )
@@
   (symbol (lib_id "power:GND") (at 275.59 33.02 0) (unit 1)
     (in_bom yes) (on_board yes) (fields_autoplaced)
-    (property "Reference" "#PWR0106" (id 0) (at 275.59 39.37 0)
+    (property "Reference" "#PWR0208" (id 0) (at 275.59 39.37 0)
       (effects (font (size 1.27 1.27)) hide)
     )
@@
   (symbol (lib_id "power:GND") (at 227.33 33.02 0) (unit 1)
     (in_bom yes) (on_board yes) (fields_autoplaced)
-    (property "Reference" "#PWR0109" (id 0) (at 227.33 39.37 0)
+    (property "Reference" "#PWR0206" (id 0) (at 227.33 39.37 0)
       (effects (font (size 1.27 1.27)) hide)
     )
@@
   (symbol (lib_id "Connector:Conn_01x20_Male") (at 265.43 86.36 180) (unit 1)
     (in_bom yes) (on_board yes) (fields_autoplaced)
-    (property "Reference" "J?" (id 0) (at 266.7 83.8199 0)
-      (effects (font (size 1.27 1.27)) (justify right))
-    )
-    (property "Value" "" (id 1) (at 266.7 86.3599 0)
-      (effects (font (size 1.27 1.27)) (justify right))
-    )
+    (property "Reference" "J202" (id 0) (at 266.7 83.8199 0)
+      (effects (font (size 1.27 1.27)) (justify right))
+    )
+    (property "Value" "Conn_01x20_Male" (id 1) (at 266.7 86.3599 0)
+      (effects (font (size 1.27 1.27)) (justify right))
+    )

Commit message: footprints
Parts:
- C201: footprint (none) -> Capacitor_SMD:CP_Elec_3x5.3
Changed lines of the file:
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@@
     (property "Reference" "C201" (id 0) (at 99.06 24.13 90))
     (property "Value" ".1uF" (id 1) (at 99.06 26.67 90))
-    (property "Footprint" "" (id 2) (at 95.25 32.7152 0)
+    (property "Footprint" "Capacitor_SMD:CP_Elec_3x5.3" (id 2) (at 95.25 32.7152 0)
       (effects (font (size 1.27 1.27)) hide)
     )

Commit message: pcb
Parts:
- J201: footprint (none) -> Connector_PinHeader_1.00mm:PinHeader_1x15_P1.00mm_Vertical
- J202: footprint (none) -> Connector_PinHeader_1.00mm:PinHeader_1x20_P1.00mm_Vertical
- J203: footprint (none) -> Connector_PinHeader_1.00mm:PinHeader_1x16_P1.00mm_Vertical
- U202, U203, U204: footprint (none) -> Package_DIP:DIP-20_W7.62mm
Changed lines of the file:
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@@
       (effects (font (size 1.27 1.27)) (justify right))
     )
-    (property "Footprint" "" (id 2) (at 265.43 134.62 0)
+    (property "Footprint" "Connector_PinHeader_1.00mm:PinHeader_1x16_P1.00mm_Vertical" (id 2) (at 265.43 134.62 0)
       (effects (font (size 1.27 1.27)) hide)
     )
@@
     (property "Reference" "U203" (id 0) (at 228.6 29.4386 90))
     (property "Value" "74AHC373" (id 1) (at 228.6 31.9786 90))
-    (property "Footprint" "" (id 2) (at 207.01 33.02 0)
+    (property "Footprint" "Package_DIP:DIP-20_W7.62mm" (id 2) (at 207.01 33.02 0)
       (effects (font (size 1.27 1.27)) hide)
     )
@@
     (property "Reference" "U204" (id 0) (at 276.86 29.4386 90))
     (property "Value" "74AHC373" (id 1) (at 276.86 31.9786 90))
-    (property "Footprint" "" (id 2) (at 255.27 33.02 0)
+    (property "Footprint" "Package_DIP:DIP-20_W7.62mm" (id 2) (at 255.27 33.02 0)
       (effects (font (size 1.27 1.27)) hide)
     )
@@
       (effects (font (size 1.27 1.27)) (justify right))
     )
-    (property "Footprint" "" (id 2) (at 175.26 135.89 0)
+    (property "Footprint" "Connector_PinHeader_1.00mm:PinHeader_1x15_P1.00mm_Vertical" (id 2) (at 175.26 135.89 0)
       (effects (font (size 1.27 1.27)) hide)
     )
@@
     (property "Reference" "U202" (id 0) (at 181.61 29.4386 90))
     (property "Value" "74AHC373" (id 1) (at 181.61 31.9786 90))
-    (property "Footprint" "" (id 2) (at 160.02 33.02 0)
+    (property "Footprint" "Package_DIP:DIP-20_W7.62mm" (id 2) (at 160.02 33.02 0)
       (effects (font (size 1.27 1.27)) hide)
     )
@@
       (effects (font (size 1.27 1.27)) (justify right))
     )
-    (property "Footprint" "" (id 2) (at 265.43 86.36 0)
-      (effects (font (size 1.27 1.27)) hide)
-    )
+    (property "Footprint" "Connector_PinHeader_1.00mm:PinHeader_1x20_P1.00mm_Vertical" (id 2) (at 265.43 86.36 0)
+      (effects (font (size 1.27 1.27)) hide)
+    )

Commit message: pcb
Connections:
- net A0: now also U202.2 (O0)
- net A1: now also U202.5 (O1)
- net A10: now also U203.6 (O2)
- net A11: now also U203.9 (O3)
- net A12: now also U203.12 (O4)
- net A13: now also U203.15 (O5)
- net A14: now also U203.16 (O6)
- net A15: now also U203.19 (O7)
- net A16: now also U204.2 (O0)
- net A17: now also U204.5 (O1)
- net A18: now also U204.6 (O2)
- net A19: now also U204.9 (O3)
- net A2: now also U202.6 (O2)
- net A3: now also U202.9 (O3)
- net A4: now also U202.12 (O4)
- net A5: now also U202.15 (O5)
- net A6: now also U202.16 (O6)
- net A7: now also U202.19 (O7)
- net A8: now also U203.2 (O0)
- net A9: now also U203.5 (O1)
- net D0: now also U201.16 (AD0)
- net D1: now also U201.15 (AD1)
- net D10: now also U201.6 (AD10)
- net D11: now also U201.5 (AD11)
- net D12: now also U201.4 (AD12)
- net D13: now also U201.3 (AD13)
- net D14: now also U201.2 (AD14)
- net D15: now also U201.39 (AD15)
- net D2: now also U201.14 (AD2)
- net D3: now also U201.13 (AD3)
- net D4: now also U201.12 (AD4)
- net D5: now also U201.11 (AD5)
- net D6: now also U201.10 (AD6)
- net D7: now also U201.9 (AD7)
- net D8: now also U201.8 (AD8)
- net D9: now also U201.7 (AD9)
