File: 8086proj/8255.kicad_sch (KiCad schematic)
At the start: 3 parts

Commit message: 8255
Parts:
- added C? (x2): .1uf, symbol Device:C
- added C?: (no value), symbol Device:C
- added J?: (no value), symbol Connector:Conn_01x08_Female
- added J? (x8): Conn_01x08_Female, symbol Connector:Conn_01x08_Female
- added U?: (no value), symbol Logic_Programmable:PAL16L8
Connections:
- net at U?.1 (PA3): now also J?.4 (Pin_4) (x3)
- net at U?.10 (PC7): now also J?.8 (Pin_8) (x3)
- net at U?.11 (PC6): now also J?.7 (Pin_7) (x3)
- net at U?.12 (PC5): now also J?.6 (Pin_6) (x3)
- net at U?.13 (PC4): now also J?.5 (Pin_5) (x3)
- net at U?.14 (PC0): now also J?.1 (Pin_1) (x3)
- net at U?.15 (PC1): now also J?.2 (Pin_2) (x3)
- net at U?.16 (PC2): now also J?.3 (Pin_3) (x3)
- net at U?.17 (PC3): now also J?.4 (Pin_4) (x3)
- net at U?.18 (PB0): now also J?.1 (Pin_1) (x3)
- net at U?.19 (PB1): now also J?.2 (Pin_2) (x3)
- net at U?.2 (PA2): now also J?.3 (Pin_3) (x3)
- net at U?.20 (PB2): now also J?.3 (Pin_3) (x3)
- net at U?.21 (PB3): now also J?.4 (Pin_4) (x3)
- net at U?.22 (PB4): now also J?.5 (Pin_5) (x3)
- net at U?.23 (PB5): now also J?.6 (Pin_6) (x3)
- net at U?.24 (PB6): now also J?.7 (Pin_7) (x3)
- net at U?.25 (PB7): now also J?.8 (Pin_8) (x3)
- net VIN: now reaches U?.26 (VCC)
- net VIN: now also U?.26 (VCC), U?.26 (VCC), C?.1, C?.1, C?.1, U?.20 (VCC)
- net D7: now reaches U?.27 (D7)
- net D7: now also U?.27 (D7), U?.27 (D7)
- net D6: now reaches U?.28 (D6)
- net D6: now also U?.28 (D6), U?.28 (D6)
- net D5: now reaches U?.29 (D5)
- net D5: now also U?.29 (D5), U?.29 (D5)
- net at U?.3 (PA1): now also J?.2 (Pin_2) (x3)
- net D4: now reaches U?.30 (D4)
- net D4: now also U?.30 (D4), U?.30 (D4)
- net D3: now reaches U?.31 (D3)
- net D3: now also U?.31 (D3), U?.31 (D3)
- net D2: now reaches U?.32 (D2)
- net D2: now also U?.32 (D2), U?.32 (D2)
- net D1: now reaches U?.33 (D1)
- net D1: now also U?.33 (D1), U?.33 (D1)
- net D0: now reaches U?.34 (D0)
- net D0: now also U?.34 (D0), U?.34 (D0)
- net RESET: now reaches U?.35 (RESET)
- net RESET: now also U?.35 (RESET), U?.35 (RESET)
- net _WR: now reaches U?.36 (~{WR})
- net _WR: now also U?.36 (~{WR}), U?.36 (~{WR})
- net at U?.37 (PA7): now also J?.8 (Pin_8) (x3)
- net at U?.38 (PA6): now also J?.7 (Pin_7) (x3)
- net at U?.39 (PA5): now also J?.6 (Pin_6) (x3)
- net at U?.4 (PA0): now also J?.1 (Pin_1) (x3)
- net at U?.40 (PA4): now also J?.5 (Pin_5) (x3)
- net _RD: now reaches U?.5 (~{RD})
- net _RD: now also U?.5 (~{RD}), U?.5 (~{RD})
- net O6: now reaches U?.6 (~{CS})
- net O6: now also U?.14 (IO6)
- net GND: now reaches U?.7 (GND)
- net GND: now also U?.7 (GND), U?.7 (GND), C?.2, C?.2, C?.2, U?.10 (GND)
- net A2: now reaches U?.8 (A1)
- net A2: now also U?.8 (A1), U?.8 (A1)
- net A1: now reaches U?.9 (A0)
- net A1: now also U?.9 (A0), U?.9 (A0)
- net O7: now reaches U?.6 (~{CS})
- net O7: now also U?.13 (IO7)
- net O5: now reaches U?.6 (~{CS})
- net O5: now also U?.15 (IO5)
- new net A0: U?.1 (I1)
- new net A10: U?.9 (I9)
- new net A11: U?.11 (I10)
- new net A12: U?.19 (IO1)
- new net A13: U?.18 (IO2)
- new net A14: U?.17 (I03)
- new net A15: U?.16 (IO4)
- new net A3: U?.2 (I2)
- new net A4: U?.3 (I3)
- new net A5: U?.4 (I4)
- new net A6: U?.5 (I5)
- new net A7: U?.6 (I6)
- new net A8: U?.7 (I7)
- new net A9: U?.8 (I8)
Other:
- moved on the sheet: U?

Commit message: 8259
Parts:
- C?: value (none) -> .1uf
- J?: value (none) -> Conn_01x08_Female
- U?: value (none) -> PAL16L8
- U?: value (none) -> 8255; footprint (none) -> Package_DIP:DIP-40_W15.24mm
Changed lines of the file:
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@@
       (effects (font (size 1.27 1.27)) (justify left))
     )
-    (property "Value" "" (id 1) (at 133.35 55.8799 0)
+    (property "Value" "Conn_01x08_Female" (id 1) (at 133.35 55.8799 0)
       (effects (font (size 1.27 1.27)) (justify left))
     )
@@
       (effects (font (size 1.27 1.27)) hide)
     )
-    (property "Value" "" (id 1) (at 62.23 147.32 0))
+    (property "Value" "GND" (id 1) (at 62.23 147.32 0))
     (property "Footprint" "" (id 2) (at 62.23 142.24 0)
       (effects (font (size 1.27 1.27)) hide)
@@
     (in_bom yes) (on_board yes) (fields_autoplaced)
     (property "Reference" "C?" (id 0) (at 113.03 24.13 90))
-    (property "Value" "" (id 1) (at 113.03 26.67 90))
+    (property "Value" ".1uf" (id 1) (at 113.03 26.67 90))
     (property "Footprint" "" (id 2) (at 116.84 30.7848 0)
       (effects (font (size 1.27 1.27)) hide)
@@
       (effects (font (size 1.27 1.27)) (justify left))
     )
-    (property "Value" "" (id 1) (at 64.2494 110.49 0)
+    (property "Value" "PAL16L8" (id 1) (at 64.2494 110.49 0)
       (effects (font (size 1.27 1.27)) (justify left))
     )
@@
       (effects (font (size 1.27 1.27)) (justify left))
     )
-    (property "Value" "" (id 1) (at 221.7294 38.1 0)
-      (effects (font (size 1.27 1.27)) (justify left))
-    )
-    (property "Footprint" "" (id 2) (at 219.71 69.85 0)
+    (property "Value" "8255" (id 1) (at 221.7294 38.1 0)
+      (effects (font (size 1.27 1.27)) (justify left))
+    )
+    (property "Footprint" "Package_DIP:DIP-40_W15.24mm" (id 2) (at 219.71 69.85 0)
       (effects (font (size 1.27 1.27)) hide)
     )
@@
       (effects (font (size 1.27 1.27)) hide)
     )
-    (property "Value" "" (id 1) (at 116.84 40.64 0))
+    (property "Value" "GND" (id 1) (at 116.84 40.64 0))
     (property "Footprint" "" (id 2) (at 116.84 35.56 0)
       (effects (font (size 1.27 1.27)) hide)

Commit message: fixes
Parts:
- added SW?: (no value), symbol Switch:SW_DIP_x08
- added U? (x2): (no value), symbol 74xGxx:74AUC2G32
- added U?: 74AUC2G32, symbol 74xGxx:74AUC2G32
- added U?: (no value), symbol 74xx:74AHCT04
- added U?: (no value), symbol 4xxx:4011
- added U?: (no value), symbol 74xGxx:74LVC1G332
Connections:
- net VIN is gone; now on net GND: C?.1, C?.1, C?.1, U?.20 (VCC), U?.26 (VCC), U?.26 (VCC), U?.26 (VCC)
- net D0: now also SW?.9
- net D1: now also SW?.10
- net D2: now also SW?.11
- net D3: now also SW?.12
- net D4: now also SW?.13
- net D5: now also SW?.14
- net D6: now also SW?.15
- net D7: now also SW?.16
- net GND: now also U?.2 (GND), U?.4 (GND), U?.4 (GND), U?.4 (GND)
- net _INTA: now reaches J?.7 (Pin_7), U?.11 (PC6)
- net _INTA: now also J?.1 (Pin_1), J?.3 (Pin_3), J?.3 (Pin_3), J?.3 (Pin_3), J?.7 (Pin_7), J?.7 (Pin_7), U?.11 (PC6), U?.11 (PC6), U?.14 (PC0), U?.16 (PC2), U?.16 (PC2), U?.16 (PC2), U?.1
- net at J?.1 (Pin_1), U?.14 (PC0): now also U?.6 (x2)
- net at J?.4 (Pin_4), U?.17 (PC3): now also U?.5 (x2)
- net M/_IO: now reaches U?.12 (IO8)
- new net: U?.1, U?.3
- new net: U?.3, U?.7
- new net: U?.3, U?.6
- new net: U?.2, U?.2
- new net: SW?.1, SW?.2, SW?.3, SW?.4, SW?.5, SW?.6, SW?.7, SW?.8, U?.3
- new net INT: U?.1, U?.4
- new net VCC: U?.5 (VCC), U?.8 (VCC), U?.8 (VCC), U?.8 (VCC)
Other:
- moved on the sheet: J?, U?

Commit message: 16550
Parts:
- SW?: value (none) -> SW_DIP_x08
- U? (x2): value (none) -> 74AUC2G32
- U?: value (none) -> 74AHCT04
- U?: value (none) -> 4011
- U?: value (none) -> 74LVC1G332
Changed lines of the file:
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@@
       (effects (font (size 1.27 1.27)) (justify left))
     )
-    (property "Value" "" (id 1) (at 201.93 131.4449 90)
+    (property "Value" "74AUC2G32" (id 1) (at 201.93 131.4449 90)
       (effects (font (size 1.27 1.27)) (justify left))
     )
@@
       (effects (font (size 1.27 1.27)) (justify left))
     )
-    (property "Value" "" (id 1) (at 142.24 135.2549 90)
+    (property "Value" "74AUC2G32" (id 1) (at 142.24 135.2549 90)
       (effects (font (size 1.27 1.27)) (justify left))
     )
@@
     (in_bom yes) (on_board yes) (fields_autoplaced)
     (property "Reference" "U?" (id 0) (at 180.34 148.59 0))
-    (property "Value" "" (id 1) (at 180.34 151.13 0))
+    (property "Value" "74AHCT04" (id 1) (at 180.34 151.13 0))
     (property "Footprint" "" (id 2) (at 180.34 157.48 0)
       (effects (font (size 1.27 1.27)) hide)
@@
       (effects (font (size 1.27 1.27)) (justify left))
     )
-    (property "Value" "" (id 1) (at 147.32 171.4499 90)
+    (property "Value" "SW_DIP_x08" (id 1) (at 147.32 171.4499 90)
       (effects (font (size 1.27 1.27)) (justify left))
     )
@@
     (in_bom yes) (on_board yes) (fields_autoplaced)
     (property "Reference" "U?" (id 0) (at 165.1 151.13 0))
-    (property "Value" "" (id 1) (at 165.1 153.67 0))
+    (property "Value" "4011" (id 1) (at 165.1 153.67 0))
     (property "Footprint" "" (id 2) (at 165.1 160.02 0)
       (effects (font (size 1.27 1.27)) hide)
@@
       (effects (font (size 1.27 1.27)) (justify left))
     )
-    (property "Value" "" (id 1) (at 203.2 153.3524 90)
-      (effects (font (size 1.27 1.27)) (justify left))
-    )
+    (property "Value" "74LVC1G332" (id 1) (at 203.2 153.3524 90)
+      (effects (font (size 1.27 1.27)) (justify left))
+    )

Commit message: 7seg
Connections:
- net _INTA: now also U?.2
- net at J?.4 (Pin_4), U?.17 (PC3): now also U?.1
Changed lines of the file:
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@@
   (junction (at 173.99 30.48) (diameter 0) (color 0 0 0 0)
   )
+  (wire (pts (xy 137.16 125.73) (xy 137.16 127))
+    (stroke (width 0) (type default) (color 0 0 0 0))
+  )
   (wire (pts (xy 128.27 162.56) (xy 125.73 162.56))
     (stroke (width 0) (type default) (color 0 0 0 0))
@@
     (stroke (width 0) (type default) (color 0 0 0 0))
   )
+  (wire (pts (xy 140.97 125.73) (xy 139.7 125.73))
+    (stroke (width 0) (type default) (color 0 0 0 0))
+  )
   (wire (pts (xy 87.63 86.36) (xy 91.44 86.36))
     (stroke (width 0) (type default) (color 0 0 0 0))
@@
     (stroke (width 0) (type default) (color 0 0 0 0))
   )
+  (wire (pts (xy 139.7 125.73) (xy 139.7 127))
+    (stroke (width 0) (type default) (color 0 0 0 0))
+  )
   (wire (pts (xy 74.93 121.92) (xy 81.28 121.92))
     (stroke (width 0) (type default) (color 0 0 0 0))
@@
     (stroke (width 0) (type default) (color 0 0 0 0))
   )
-  (wire (pts (xy 132.08 125.73) (xy 135.89 125.73))
-    (stroke (width 0) (type default) (color 0 0 0 0))
-  )
+  (wire (pts (xy 132.08 125.73) (xy 137.16 125.73))
+    (stroke (width 0) (type default) (color 0 0 0 0))
+  )

Commit message: final look
Parts:
- removed J? (x9): Conn_01x08_Female, symbol Connector:Conn_01x08_Female
- added J601: (no value), symbol Connector:Conn_01x08_Male
- added J602, J603, J604, J605, J606, J607, J608, J609: Conn_01x08_Male, symbol Connector:Conn_01x08_Male
- gave numbers to parts that had none: 13
Connections:
- net _INTA: now also J603.2 (Pin_2), J603.6 (Pin_6), J603.8 (Pin_8), J606.2 (Pin_2), J606.6 (Pin_6), J609.2 (Pin_2), J609.6 (Pin_6)
- net at U602.4 (PA0): now also J601.8 (Pin_8)
- net at U602.3 (PA1): now also J601.7 (Pin_7)
- net at U602.2 (PA2): now also J601.6 (Pin_6)
- net at U602.1 (PA3): now also J601.5 (Pin_5)
- net at U602.40 (PA4): now also J601.4 (Pin_4)
- net at U602.39 (PA5): now also J601.3 (Pin_3)
- net at U602.38 (PA6): now also J601.2 (Pin_2)
- net at U602.37 (PA7): now also J601.1 (Pin_1)
- net at U605.1 (PA3): now also J604.5 (Pin_5)
- net at U605.10 (PC7): now also J606.1 (Pin_1)
- net at U605.12 (PC5): now also J606.3 (Pin_3)
- net at U605.13 (PC4): now also J606.4 (Pin_4)
- net at U603.6, U605.14 (PC0): now also J606.8 (Pin_8)
- net at U605.15 (PC1): now also J606.7 (Pin_7)
- net at U603.5, U605.17 (PC3): now also J606.5 (Pin_5)
- net at U605.18 (PB0): now also J605.8 (Pin_8)
- net at U605.19 (PB1): now also J605.7 (Pin_7)
- net at U605.2 (PA2): now also J604.6 (Pin_6)
- net at U605.20 (PB2): now also J605.6 (Pin_6)
- net at U605.21 (PB3): now also J605.5 (Pin_5)
- net at U605.22 (PB4): now also J605.4 (Pin_4)
- net at U605.23 (PB5): now also J605.3 (Pin_3)
- net at U605.24 (PB6): now also J605.2 (Pin_2)
- net at U605.25 (PB7): now also J605.1 (Pin_1)
- net at U605.3 (PA1): now also J604.7 (Pin_7)
- net at U605.37 (PA7): now also J604.1 (Pin_1)
- net at U605.38 (PA6): now also J604.2 (Pin_2)
- net at U605.39 (PA5): now also J604.3 (Pin_3)
- net at U605.4 (PA0): now also J604.8 (Pin_8)
- net at U605.40 (PA4): now also J604.4 (Pin_4)
- net at U608.18 (PB0): now also J608.8 (Pin_8)
- net at U608.19 (PB1): now also J608.7 (Pin_7)
- net at U608.20 (PB2): now also J608.6 (Pin_6)
- net at U608.21 (PB3): now also J608.5 (Pin_5)
- net at U608.22 (PB4): now also J608.4 (Pin_4)
- net at U608.23 (PB5): now also J608.3 (Pin_3)
- net at U608.24 (PB6): now also J608.2 (Pin_2)
- net at U608.25 (PB7): now also J608.1 (Pin_1)
- net at U608.14 (PC0), U609.6: now also J609.8 (Pin_8)
- net at U608.15 (PC1): now also J609.7 (Pin_7)
- net at U608.17 (PC3), U609.5: now also J609.5 (Pin_5)
- net at U608.13 (PC4): now also J609.4 (Pin_4)
- net at U608.12 (PC5): now also J609.3 (Pin_3)
- net at U608.10 (PC7): now also J609.1 (Pin_1)
- net at U602.15 (PC1): now also J603.7 (Pin_7)
- net at U602.17 (PC3), U603.1: now also J603.5 (Pin_5)
- net at U602.13 (PC4): now also J603.4 (Pin_4)
- net at U602.12 (PC5): now also J603.3 (Pin_3)
- net at U602.10 (PC7): now also J603.1 (Pin_1)
- net at U602.18 (PB0): now also J602.8 (Pin_8)
- net at U602.19 (PB1): now also J602.7 (Pin_7)
- net at U602.20 (PB2): now also J602.6 (Pin_6)
- net at U602.21 (PB3): now also J602.5 (Pin_5)
- net at U602.22 (PB4): now also J602.4 (Pin_4)
- net at U602.23 (PB5): now also J602.3 (Pin_3)
- net at U602.24 (PB6): now also J602.2 (Pin_2)
- net at U602.25 (PB7): now also J602.1 (Pin_1)
- net at U608.1 (PA3): now also J607.5 (Pin_5)
- net at U608.2 (PA2): now also J607.6 (Pin_6)
- net at U608.3 (PA1): now also J607.7 (Pin_7)
- net at U608.37 (PA7): now also J607.1 (Pin_1)
- net at U608.38 (PA6): now also J607.2 (Pin_2)
- net at U608.39 (PA5): now also J607.3 (Pin_3)
- net at U608.4 (PA0): now also J607.8 (Pin_8)
- net at U608.40 (PA4): now also J607.4 (Pin_4)
