File: 8086proj/8255.kicad_sch (KiCad schematic)
At the start: 22 parts, among them J602 Conn_01x08_Male, J603 Conn_01x08_Male, J604 Conn_01x08_Male, J605 Conn_01x08_Male, J606 Conn_01x08_Male, J607 Conn_01x08_Male, J608 Conn_01x08_Male, J609 Conn_01x08_Male, SW601 SW_DIP_x08, U601 PAL16L8, U602 8255, U603 74AUC2G32, U604 4011, U605 8255, U606 74AHCT04, U607 74LVC1G332, U608 8255, U609 74AUC2G32

Commit message: footprints
Parts:
- C601, C602, C603: footprint (none) -> Capacitor_SMD:CP_Elec_3x5.3
- J601: value (none) -> Conn_01x08_Male
Changed lines of the file:
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@@
       (effects (font (size 1.27 1.27)) (justify right))
     )
-    (property "Value" "" (id 1) (at 133.35 55.8799 0)
+    (property "Value" "Conn_01x08_Male" (id 1) (at 133.35 55.8799 0)
       (effects (font (size 1.27 1.27)) (justify right))
     )
@@
     (property "Reference" "C603" (id 0) (at 223.52 24.13 90))
     (property "Value" ".1uf" (id 1) (at 223.52 26.67 90))
-    (property "Footprint" "" (id 2) (at 227.33 30.7848 0)
+    (property "Footprint" "Capacitor_SMD:CP_Elec_3x5.3" (id 2) (at 227.33 30.7848 0)
       (effects (font (size 1.27 1.27)) hide)
     )
@@
     (property "Reference" "C601" (id 0) (at 113.03 24.13 90))
     (property "Value" ".1uf" (id 1) (at 113.03 26.67 90))
-    (property "Footprint" "" (id 2) (at 116.84 30.7848 0)
+    (property "Footprint" "Capacitor_SMD:CP_Elec_3x5.3" (id 2) (at 116.84 30.7848 0)
       (effects (font (size 1.27 1.27)) hide)
     )
@@
     (property "Reference" "C602" (id 0) (at 167.64 22.86 90))
     (property "Value" ".1uf" (id 1) (at 167.64 25.4 90))
-    (property "Footprint" "" (id 2) (at 171.45 29.5148 0)
-      (effects (font (size 1.27 1.27)) hide)
-    )
+    (property "Footprint" "Capacitor_SMD:CP_Elec_3x5.3" (id 2) (at 171.45 29.5148 0)
+      (effects (font (size 1.27 1.27)) hide)
+    )

Commit message: pcb
Parts:
- J601, J602, J603, J604, J605, J606, J607, J608, J609: footprint (none) -> Connector_PinHeader_1.00mm:PinHeader_1x08_P1.00mm_Vertical
- SW601: footprint (none) -> Button_Switch_SMD:SW_DIP_SPSTx08_Slide_6.7x21.88mm_W6.73mm_P2.54mm_LowProfile_JPin
- U601: footprint (none) -> Package_DIP:DIP-20_W7.62mm
Changed lines of the file:
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@@
       (effects (font (size 1.27 1.27)) (justify right))
     )
-    (property "Footprint" "" (id 2) (at 196.85 54.61 0)
+    (property "Footprint" "Connector_PinHeader_1.00mm:PinHeader_1x08_P1.00mm_Vertical" (id 2) (at 196.85 54.61 0)
       (effects (font (size 1.27 1.27)) hide)
     )
@@
       (effects (font (size 1.27 1.27)) (justify right))
     )
-    (property "Footprint" "" (id 2) (at 255.27 52.07 0)
+    (property "Footprint" "Connector_PinHeader_1.00mm:PinHeader_1x08_P1.00mm_Vertical" (id 2) (at 255.27 52.07 0)
       (effects (font (size 1.27 1.27)) hide)
     )
@@
       (effects (font (size 1.27 1.27)) (justify right))
     )
-    (property "Footprint" "" (id 2) (at 132.08 55.88 0)
+    (property "Footprint" "Connector_PinHeader_1.00mm:PinHeader_1x08_P1.00mm_Vertical" (id 2) (at 132.08 55.88 0)
       (effects (font (size 1.27 1.27)) hide)
     )
@@
       (effects (font (size 1.27 1.27)) (justify right))
     )
-    (property "Footprint" "" (id 2) (at 261.62 97.79 0)
+    (property "Footprint" "Connector_PinHeader_1.00mm:PinHeader_1x08_P1.00mm_Vertical" (id 2) (at 261.62 97.79 0)
       (effects (font (size 1.27 1.27)) hide)
     )
@@
       (effects (font (size 1.27 1.27)) (justify right))
     )
-    (property "Footprint" "" (id 2) (at 196.85 77.47 0)
+    (property "Footprint" "Connector_PinHeader_1.00mm:PinHeader_1x08_P1.00mm_Vertical" (id 2) (at 196.85 77.47 0)
       (effects (font (size 1.27 1.27)) hide)
     )
@@
       (effects (font (size 1.27 1.27)) (justify right))
     )
-    (property "Footprint" "" (id 2) (at 140.97 101.6 0)
+    (property "Footprint" "Connector_PinHeader_1.00mm:PinHeader_1x08_P1.00mm_Vertical" (id 2) (at 140.97 101.6 0)
       (effects (font (size 1.27 1.27)) hide)
     )
@@
       (effects (font (size 1.27 1.27)) (justify right))
     )
-    (property "Footprint" "" (id 2) (at 255.27 74.93 0)
+    (property "Footprint" "Connector_PinHeader_1.00mm:PinHeader_1x08_P1.00mm_Vertical" (id 2) (at 255.27 74.93 0)
       (effects (font (size 1.27 1.27)) hide)
     )
@@
       (effects (font (size 1.27 1.27)) (justify left))
     )
-    (property "Footprint" "" (id 2) (at 62.23 127 0)
+    (property "Footprint" "Package_DIP:DIP-20_W7.62mm" (id 2) (at 62.23 127 0)
       (effects (font (size 1.27 1.27)) hide)
     )
@@
       (effects (font (size 1.27 1.27)) (justify left))
     )
-    (property "Footprint" "" (id 2) (at 133.35 170.18 0)
+    (property "Footprint" "Button_Switch_SMD:SW_DIP_SPSTx08_Slide_6.7x21.88mm_W6.73mm_P2.54mm_LowProfile_JPin" (id 2) (at 133.35 170.18 0)
       (effects (font (size 1.27 1.27)) hide)
     )
@@
       (effects (font (size 1.27 1.27)) (justify right))
     )
-    (property "Footprint" "" (id 2) (at 132.08 78.74 0)
+    (property "Footprint" "Connector_PinHeader_1.00mm:PinHeader_1x08_P1.00mm_Vertical" (id 2) (at 132.08 78.74 0)
       (effects (font (size 1.27 1.27)) hide)
     )
@@
       (effects (font (size 1.27 1.27)) (justify right))
     )
-    (property "Footprint" "" (id 2) (at 205.74 100.33 0)
-      (effects (font (size 1.27 1.27)) hide)
-    )
+    (property "Footprint" "Connector_PinHeader_1.00mm:PinHeader_1x08_P1.00mm_Vertical" (id 2) (at 205.74 100.33 0)
+      (effects (font (size 1.27 1.27)) hide)
+    )

Commit message: pcb
Parts:
- U603, U604, U606, U607, U609: footprint (none) -> Package_DIP:DIP-14_W10.16mm
Changed lines of the file:
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@@
       (effects (font (size 1.27 1.27)) (justify left))
     )
-    (property "Footprint" "" (id 2) (at 198.12 130.81 0)
+    (property "Footprint" "Package_DIP:DIP-14_W10.16mm" (id 2) (at 198.12 130.81 0)
       (effects (font (size 1.27 1.27)) hide)
     )
@@
       (effects (font (size 1.27 1.27)) (justify left))
     )
-    (property "Footprint" "" (id 2) (at 138.43 134.62 0)
+    (property "Footprint" "Package_DIP:DIP-14_W10.16mm" (id 2) (at 138.43 134.62 0)
       (effects (font (size 1.27 1.27)) hide)
     )
@@
       (effects (font (size 1.27 1.27)) (justify left))
     )
-    (property "Footprint" "" (id 2) (at 251.46 125.73 0)
+    (property "Footprint" "Package_DIP:DIP-14_W10.16mm" (id 2) (at 251.46 125.73 0)
       (effects (font (size 1.27 1.27)) hide)
     )
@@
     (property "Reference" "U606" (id 0) (at 180.34 148.59 0))
     (property "Value" "74AHCT04" (id 1) (at 180.34 151.13 0))
-    (property "Footprint" "" (id 2) (at 180.34 157.48 0)
+    (property "Footprint" "Package_DIP:DIP-14_W10.16mm" (id 2) (at 180.34 157.48 0)
       (effects (font (size 1.27 1.27)) hide)
     )
@@
     (property "Reference" "U604" (id 0) (at 165.1 151.13 0))
     (property "Value" "4011" (id 1) (at 165.1 153.67 0))
-    (property "Footprint" "" (id 2) (at 165.1 160.02 0)
+    (property "Footprint" "Package_DIP:DIP-14_W10.16mm" (id 2) (at 165.1 160.02 0)
       (effects (font (size 1.27 1.27)) hide)
     )
@@
       (effects (font (size 1.27 1.27)) (justify left))
     )
-    (property "Footprint" "" (id 2) (at 198.12 152.4 0)
-      (effects (font (size 1.27 1.27)) hide)
-    )
+    (property "Footprint" "Package_DIP:DIP-14_W10.16mm" (id 2) (at 198.12 152.4 0)
+      (effects (font (size 1.27 1.27)) hide)
+    )
