File: 8086proj/CY7C199.kicad_sch (KiCad schematic)
At the start: 10 parts, among them U0 PAL16L8, U1 CY7C199, U2 CY7C199, U3 CY7C199, U4 CY7C199

Commit message: final look
Parts:
- gave numbers to parts that had none: 1
- renumbered C0 to C502, C1 to C503, C2 to C504, C3 to C505, U0 to U501, U1 to U502, U2 to U503, U3 to U504, U4 to U505
Changed lines of the file:
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@@
   (symbol (lib_id "power:GND") (at 59.69 87.63 180) (unit 1)
     (in_bom yes) (on_board yes) (fields_autoplaced)
-    (property "Reference" "#PWR0117" (id 0) (at 59.69 81.28 0)
+    (property "Reference" "#PWR0503" (id 0) (at 59.69 81.28 0)
       (effects (font (size 1.27 1.27)) hide)
     )
@@
   (symbol (lib_id "power:GND") (at 67.31 157.48 0) (unit 1)
     (in_bom yes) (on_board yes) (fields_autoplaced)
-    (property "Reference" "#PWR0121" (id 0) (at 67.31 163.83 0)
+    (property "Reference" "#PWR0504" (id 0) (at 67.31 163.83 0)
       (effects (font (size 1.27 1.27)) hide)
     )
@@
   (symbol (lib_id "Device:C") (at 110.49 87.63 90) (unit 1)
     (in_bom yes) (on_board yes) (fields_autoplaced)
-    (property "Reference" "C1" (id 0) (at 109.2199 83.82 0)
+    (property "Reference" "C503" (id 0) (at 109.2199 83.82 0)
       (effects (font (size 1.27 1.27)) (justify left))
     )
@@
   (symbol (lib_id "Memory_RAM:CY7C199") (at 205.74 124.46 0) (unit 1)
     (in_bom yes) (on_board yes) (fields_autoplaced)
-    (property "Reference" "U4" (id 0) (at 207.7594 92.71 0)
+    (property "Reference" "U505" (id 0) (at 207.7594 92.71 0)
       (effects (font (size 1.27 1.27)) (justify left))
     )
@@
   (symbol (lib_id "Memory_RAM:CY7C199") (at 114.3 124.46 0) (unit 1)
     (in_bom yes) (on_board yes) (fields_autoplaced)
-    (property "Reference" "U2" (id 0) (at 116.3194 92.71 0)
+    (property "Reference" "U503" (id 0) (at 116.3194 92.71 0)
       (effects (font (size 1.27 1.27)) (justify left))
     )
@@
   (symbol (lib_id "power:GND") (at 38.1 33.02 180) (unit 1)
     (in_bom yes) (on_board yes) (fields_autoplaced)
-    (property "Reference" "#PWR0122" (id 0) (at 38.1 26.67 0)
+    (property "Reference" "#PWR0501" (id 0) (at 38.1 26.67 0)
       (effects (font (size 1.27 1.27)) hide)
     )
@@
   (symbol (lib_id "Device:C") (at 201.93 87.63 90) (unit 1)
     (in_bom yes) (on_board yes) (fields_autoplaced)
-    (property "Reference" "C3" (id 0) (at 200.6599 83.82 0)
+    (property "Reference" "C505" (id 0) (at 200.6599 83.82 0)
       (effects (font (size 1.27 1.27)) (justify left))
     )
@@
   (symbol (lib_id "Memory_RAM:CY7C199") (at 67.31 124.46 0) (unit 1)
     (in_bom yes) (on_board yes) (fields_autoplaced)
-    (property "Reference" "U1" (id 0) (at 69.3294 92.71 0)
+    (property "Reference" "U502" (id 0) (at 69.3294 92.71 0)
       (effects (font (size 1.27 1.27)) (justify left))
     )
@@
   (symbol (lib_id "power:GND") (at 198.12 87.63 180) (unit 1)
     (in_bom yes) (on_board yes) (fields_autoplaced)
-    (property "Reference" "#PWR0120" (id 0) (at 198.12 81.28 0)
+    (property "Reference" "#PWR0507" (id 0) (at 198.12 81.28 0)
       (effects (font (size 1.27 1.27)) hide)
     )
@@
   (symbol (lib_id "power:GND") (at 45.72 67.31 0) (unit 1)
     (in_bom yes) (on_board yes) (fields_autoplaced)
-    (property "Reference" "#PWR0118" (id 0) (at 45.72 73.66 0)
+    (property "Reference" "#PWR0502" (id 0) (at 45.72 73.66 0)
       (effects (font (size 1.27 1.27)) hide)
     )
@@
   (symbol (lib_id "Logic_Programmable:PAL16L8") (at 45.72 52.07 0) (unit 1)
     (in_bom yes) (on_board yes) (fields_autoplaced)
-    (property "Reference" "U0" (id 0) (at 47.7394 33.02 0)
+    (property "Reference" "U501" (id 0) (at 47.7394 33.02 0)
       (effects (font (size 1.27 1.27)) (justify left))
     )
@@
   (symbol (lib_id "power:GND") (at 152.4 87.63 180) (unit 1)
     (in_bom yes) (on_board yes) (fields_autoplaced)
-    (property "Reference" "#PWR0116" (id 0) (at 152.4 81.28 0)
+    (property "Reference" "#PWR0506" (id 0) (at 152.4 81.28 0)
       (effects (font (size 1.27 1.27)) hide)
     )
@@
   (symbol (lib_id "power:GND") (at 106.68 87.63 180) (unit 1)
     (in_bom yes) (on_board yes) (fields_autoplaced)
-    (property "Reference" "#PWR0119" (id 0) (at 106.68 81.28 0)
+    (property "Reference" "#PWR0505" (id 0) (at 106.68 81.28 0)
       (effects (font (size 1.27 1.27)) hide)
     )
@@
   (symbol (lib_id "Device:C") (at 63.5 87.63 90) (unit 1)
     (in_bom yes) (on_board yes) (fields_autoplaced)
-    (property "Reference" "C0" (id 0) (at 62.2299 83.82 0)
+    (property "Reference" "C502" (id 0) (at 62.2299 83.82 0)
       (effects (font (size 1.27 1.27)) (justify left))
     )
@@
   (symbol (lib_id "Device:C") (at 41.91 33.02 90) (unit 1)
     (in_bom yes) (on_board yes)
-    (property "Reference" "C?" (id 0) (at 40.6399 29.21 0)
+    (property "Reference" "C501" (id 0) (at 40.6399 29.21 0)
       (effects (font (size 1.27 1.27)) (justify left))
     )
@@
   (symbol (lib_id "Device:C") (at 156.21 87.63 90) (unit 1)
     (in_bom yes) (on_board yes) (fields_autoplaced)
-    (property "Reference" "C2" (id 0) (at 154.9399 83.82 0)
+    (property "Reference" "C504" (id 0) (at 154.9399 83.82 0)
       (effects (font (size 1.27 1.27)) (justify left))
     )
@@
   (symbol (lib_id "Memory_RAM:CY7C199") (at 160.02 124.46 0) (unit 1)
     (in_bom yes) (on_board yes) (fields_autoplaced)
-    (property "Reference" "U3" (id 0) (at 162.0394 92.71 0)
-      (effects (font (size 1.27 1.27)) (justify left))
-    )
+    (property "Reference" "U504" (id 0) (at 162.0394 92.71 0)
+      (effects (font (size 1.27 1.27)) (justify left))
+    )
