File: 8086proj/CY7C199.kicad_sch (KiCad schematic)
At the start: 10 parts, among them U501 PAL16L8, U502 CY7C199, U503 CY7C199, U504 CY7C199, U505 CY7C199

Commit message: footprints
Parts:
- C501, C502, C503, C504, C505: footprint (none) -> Capacitor_SMD:CP_Elec_3x5.3
Changed lines of the file:
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@@
       (effects (font (size 1.27 1.27)) (justify left))
     )
-    (property "Footprint" "" (id 2) (at 114.3 86.6648 0)
+    (property "Footprint" "Capacitor_SMD:CP_Elec_3x5.3" (id 2) (at 114.3 86.6648 0)
       (effects (font (size 1.27 1.27)) hide)
     )
@@
       (effects (font (size 1.27 1.27)) (justify left))
     )
-    (property "Footprint" "" (id 2) (at 205.74 86.6648 0)
+    (property "Footprint" "Capacitor_SMD:CP_Elec_3x5.3" (id 2) (at 205.74 86.6648 0)
       (effects (font (size 1.27 1.27)) hide)
     )
@@
       (effects (font (size 1.27 1.27)) (justify left))
     )
-    (property "Footprint" "" (id 2) (at 67.31 86.6648 0)
+    (property "Footprint" "Capacitor_SMD:CP_Elec_3x5.3" (id 2) (at 67.31 86.6648 0)
       (effects (font (size 1.27 1.27)) hide)
     )
@@
       (effects (font (size 1.27 1.27)) (justify left))
     )
-    (property "Footprint" "" (id 2) (at 45.72 32.0548 0)
+    (property "Footprint" "Capacitor_SMD:CP_Elec_3x5.3" (id 2) (at 45.72 32.0548 0)
       (effects (font (size 1.27 1.27)) hide)
     )
@@
       (effects (font (size 1.27 1.27)) (justify left))
     )
-    (property "Footprint" "" (id 2) (at 160.02 86.6648 0)
-      (effects (font (size 1.27 1.27)) hide)
-    )
+    (property "Footprint" "Capacitor_SMD:CP_Elec_3x5.3" (id 2) (at 160.02 86.6648 0)
+      (effects (font (size 1.27 1.27)) hide)
+    )

Commit message: pcb
Parts:
- U501: footprint (none) -> Package_DIP:DIP-20_W7.62mm
- U502, U503, U504, U505: footprint (none) -> Package_DIP:DIP-28_W15.24mm
Changed lines of the file:
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@@
       (effects (font (size 1.27 1.27)) (justify left))
     )
-    (property "Footprint" "" (id 2) (at 205.74 124.46 0)
+    (property "Footprint" "Package_DIP:DIP-28_W15.24mm" (id 2) (at 205.74 124.46 0)
       (effects (font (size 1.27 1.27)) hide)
     )
@@
       (effects (font (size 1.27 1.27)) (justify left))
     )
-    (property "Footprint" "" (id 2) (at 114.3 124.46 0)
+    (property "Footprint" "Package_DIP:DIP-28_W15.24mm" (id 2) (at 114.3 124.46 0)
       (effects (font (size 1.27 1.27)) hide)
     )
@@
       (effects (font (size 1.27 1.27)) (justify left))
     )
-    (property "Footprint" "" (id 2) (at 67.31 124.46 0)
+    (property "Footprint" "Package_DIP:DIP-28_W15.24mm" (id 2) (at 67.31 124.46 0)
       (effects (font (size 1.27 1.27)) hide)
     )
@@
       (effects (font (size 1.27 1.27)) (justify left))
     )
-    (property "Footprint" "" (id 2) (at 45.72 52.07 0)
+    (property "Footprint" "Package_DIP:DIP-20_W7.62mm" (id 2) (at 45.72 52.07 0)
       (effects (font (size 1.27 1.27)) hide)
     )
@@
       (effects (font (size 1.27 1.27)) (justify left))
     )
-    (property "Footprint" "" (id 2) (at 160.02 124.46 0)
-      (effects (font (size 1.27 1.27)) hide)
-    )
+    (property "Footprint" "Package_DIP:DIP-28_W15.24mm" (id 2) (at 160.02 124.46 0)
+      (effects (font (size 1.27 1.27)) hide)
+    )
