File: 8086proj/power.kicad_sch (KiCad schematic)
At the start: 2 parts

Commit message: 8259
Parts:
- C1: value (none) -> 100uF
- J?: value (none) -> Barrel_Jack
Changed lines of the file:
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@@
       (effects (font (size 1.27 1.27)) (justify right))
     )
-    (property "Value" "" (id 1) (at 147.32 67.3099 0)
+    (property "Value" "100uF" (id 1) (at 147.32 67.3099 0)
       (effects (font (size 1.27 1.27)) (justify right))
     )
@@
     (in_bom yes) (on_board yes) (fields_autoplaced)
     (property "Reference" "J?" (id 0) (at 104.14 52.07 0))
-    (property "Value" "" (id 1) (at 104.14 54.61 0))
+    (property "Value" "Barrel_Jack" (id 1) (at 104.14 54.61 0))
     (property "Footprint" "" (id 2) (at 105.41 61.976 0)
       (effects (font (size 1.27 1.27)) hide)
@@
       (effects (font (size 1.27 1.27)) hide)
     )
-    (property "Value" "" (id 1) (at 119.38 74.93 0))
+    (property "Value" "GND" (id 1) (at 119.38 74.93 0))
     (property "Footprint" "" (id 2) (at 119.38 69.85 0)
       (effects (font (size 1.27 1.27)) hide)

Commit message: final look
Parts:
- gave numbers to parts that had none: 1
- renumbered C1 to C701
Changed lines of the file:
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@@
   (symbol (lib_id "Device:C") (at 143.51 66.04 180) (unit 1)
     (in_bom yes) (on_board yes) (fields_autoplaced)
-    (property "Reference" "C1" (id 0) (at 147.32 64.7699 0)
+    (property "Reference" "C701" (id 0) (at 147.32 64.7699 0)
       (effects (font (size 1.27 1.27)) (justify right))
     )
@@
   (symbol (lib_id "Connector:Barrel_Jack") (at 104.14 60.96 0) (unit 1)
     (in_bom yes) (on_board yes) (fields_autoplaced)
-    (property "Reference" "J?" (id 0) (at 104.14 52.07 0))
+    (property "Reference" "J701" (id 0) (at 104.14 52.07 0))
     (property "Value" "Barrel_Jack" (id 1) (at 104.14 54.61 0))
     (property "Footprint" "" (id 2) (at 105.41 61.976 0)
@@
   (symbol (lib_id "power:GND") (at 119.38 69.85 0) (unit 1)
     (in_bom yes) (on_board yes) (fields_autoplaced)
-    (property "Reference" "#PWR0130" (id 0) (at 119.38 76.2 0)
+    (property "Reference" "#PWR0701" (id 0) (at 119.38 76.2 0)
       (effects (font (size 1.27 1.27)) hide)
     )

Commit message: footprints
Parts:
- C701: footprint (none) -> Capacitor_SMD:CP_Elec_3x5.3
- J701: footprint (none) -> Connector_BarrelJack:BarrelJack_CUI_PJ-063AH_Horizontal
Changed lines of the file:
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@@
       (effects (font (size 1.27 1.27)) (justify right))
     )
-    (property "Footprint" "" (id 2) (at 142.5448 62.23 0)
+    (property "Footprint" "Capacitor_SMD:CP_Elec_3x5.3" (id 2) (at 142.5448 62.23 0)
       (effects (font (size 1.27 1.27)) hide)
     )
@@
     (property "Reference" "J701" (id 0) (at 104.14 52.07 0))
     (property "Value" "Barrel_Jack" (id 1) (at 104.14 54.61 0))
-    (property "Footprint" "" (id 2) (at 105.41 61.976 0)
+    (property "Footprint" "Connector_BarrelJack:BarrelJack_CUI_PJ-063AH_Horizontal" (id 2) (at 105.41 61.976 0)
       (effects (font (size 1.27 1.27)) hide)
     )
