File: 8086proj/ClockFinal.kicad_sch (KiCad schematic)
At the start: 6 parts

Commit message: started sram
Parts:
- C1: value (none) -> 10uF
- D1: value (none) -> LED
- R1: value (none) -> 10k
- SW1: value (none) -> SW_DIP_x01
Changed lines of the file:
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@@
     (in_bom yes) (on_board yes) (fields_autoplaced)
     (property "Reference" "SW1" (id 0) (at 93.98 85.09 0))
-    (property "Value" "" (id 1) (at 93.98 82.55 0))
+    (property "Value" "SW_DIP_x01" (id 1) (at 93.98 82.55 0))
     (property "Footprint" "" (id 2) (at 93.98 77.47 0)
       (effects (font (size 1.27 1.27)) hide)
@@
       (effects (font (size 1.27 1.27)) (justify left))
     )
-    (property "Value" "" (id 1) (at 104.14 71.1201 0)
+    (property "Value" "10k" (id 1) (at 104.14 71.1201 0)
       (effects (font (size 1.27 1.27)) (justify left))
     )
@@
       (effects (font (size 1.27 1.27)) (justify right))
     )
-    (property "Value" "" (id 1) (at 115.57 75.2474 90)
+    (property "Value" "LED" (id 1) (at 115.57 75.2474 90)
       (effects (font (size 1.27 1.27)) (justify right))
     )
@@
       (effects (font (size 1.27 1.27)) (justify left))
     )
-    (property "Value" "" (id 1) (at 105.41 82.5501 0)
+    (property "Value" "10uF" (id 1) (at 105.41 82.5501 0)
       (effects (font (size 1.27 1.27)) (justify left))
     )

Commit message: power added
Parts:
- added C2: (no value), symbol Device:C
Connections:
- net GND: now also C2.1
- net VCC renamed VIN
- net VIN: now also C2.2
Changed lines of the file:
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@@
   (junction (at 111.76 67.31) (diameter 0) (color 0 0 0 0)
   )
+  (junction (at 129.54 66.04) (diameter 0) (color 0 0 0 0)
+  )
+  (junction (at 129.54 69.85) (diameter 0) (color 0 0 0 0)
+  )
   (junction (at 109.22 77.47) (diameter 0) (color 0 0 0 0)
   )
-  (junction (at 129.54 69.85) (diameter 0) (color 0 0 0 0)
-  )
   (junction (at 129.54 114.3) (diameter 0) (color 0 0 0 0)
   )
@@
     (stroke (width 0) (type default) (color 0 0 0 0))
   )
-  (wire (pts (xy 129.54 68.58) (xy 129.54 69.85))
-    (stroke (width 0) (type default) (color 0 0 0 0))
-  )
   (wire (pts (xy 85.09 97.79) (xy 109.22 97.79))
     (stroke (width 0) (type default) (color 0 0 0 0))
@@
     (stroke (width 0) (type default) (color 0 0 0 0))
   )
+  (wire (pts (xy 139.7 66.04) (xy 139.7 67.31))
+    (stroke (width 0) (type default) (color 0 0 0 0))
+  )
+  (wire (pts (xy 129.54 60.96) (xy 129.54 66.04))
+    (stroke (width 0) (type default) (color 0 0 0 0))
+  )
   (wire (pts (xy 139.7 102.87) (xy 142.24 102.87))
     (stroke (width 0) (type default) (color 0 0 0 0))
@@
     (stroke (width 0) (type default) (color 0 0 0 0))
   )
+  (wire (pts (xy 129.54 66.04) (xy 129.54 69.85))
+    (stroke (width 0) (type default) (color 0 0 0 0))
+  )
   (wire (pts (xy 109.22 77.47) (xy 109.22 80.01))
     (stroke (width 0) (type default) (color 0 0 0 0))
@@
     (stroke (width 0) (type default) (color 0 0 0 0))
   )
+  (wire (pts (xy 137.16 66.04) (xy 139.7 66.04))
+    (stroke (width 0) (type default) (color 0 0 0 0))
+  )
   (wire (pts (xy 111.76 67.31) (xy 106.68 67.31))
     (stroke (width 0) (type default) (color 0 0 0 0))
@@
   (wire (pts (xy 106.68 77.47) (xy 109.22 77.47))
     (stroke (width 0) (type default) (color 0 0 0 0))
+  )
+  (hierarchical_label "VIN" (shape input) (at 129.54 60.96 90)
+    (effects (font (size 1.27 1.27)) (justify left))
   )
   (hierarchical_label "READY" (shape output) (at 143.51 82.55 0)
@@
     (pin "1")
     (pin "2")
+  )
+  (symbol (lib_id "power:GND") (at 139.7 67.31 0) (unit 1)
+    (in_bom yes) (on_board yes) (fields_autoplaced)
+    (property "Reference" "#PWR?" (id 0) (at 139.7 73.66 0)
+      (effects (font (size 1.27 1.27)) hide)
+    )
+    (property "Value" "" (id 1) (at 139.7 72.39 0))
+    (property "Footprint" "" (id 2) (at 139.7 67.31 0)
+      (effects (font (size 1.27 1.27)) hide)
+    )
+    (property "Datasheet" "" (id 3) (at 139.7 67.31 0)
+      (effects (font (size 1.27 1.27)) hide)
+    )
+    (pin "1")
   )
   (symbol (lib_id "Timer:8284") (at 129.54 92.71 0) (unit 1)
@@
     (pin "2")
   )
-  (symbol (lib_id "power:VCC") (at 129.54 68.58 0) (unit 1)
-    (in_bom yes) (on_board yes) (fields_autoplaced)
-    (property "Reference" "#PWR0103" (id 0) (at 129.54 72.39 0)
-      (effects (font (size 1.27 1.27)) hide)
-    )
-    (property "Value" "~" (id 1) (at 129.54 63.5 0))
-    (property "Footprint" "" (id 2) (at 129.54 68.58 0)
-      (effects (font (size 1.27 1.27)) hide)
-    )
-    (property "Datasheet" "" (id 3) (at 129.54 68.58 0)
-      (effects (font (size 1.27 1.27)) hide)
-    )
-    (pin "1")
-  )
   (symbol (lib_id "Device:LED") (at 111.76 72.39 90) (unit 1)
     (in_bom yes) (on_board yes) (fields_autoplaced)
@@
       (effects (font (size 1.27 1.27)) hide)
     )
+    (pin "1")
+    (pin "2")
+  )
+  (symbol (lib_id "Device:C") (at 133.35 66.04 270) (unit 1)
+    (in_bom yes) (on_board yes) (fields_autoplaced)
+    (property "Reference" "C2" (id 0) (at 133.35 58.42 90))
+    (property "Value" "" (id 1) (at 133.35 60.96 90))
+    (property "Footprint" "" (id 2) (at 129.54 67.0052 0)
+      (effects (font (size 1.27 1.27)) hide)
+    )
+    (property "Datasheet" "~" (id 3) (at 133.35 66.04 0)
+      (effects (font (size 1.27 1.27)) hide)
+    )

Commit message: 8259
Parts:
- C2: value (none) -> .1uF
Changed lines of the file:
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@@
       (effects (font (size 1.27 1.27)) hide)
     )
-    (property "Value" "" (id 1) (at 139.7 72.39 0))
+    (property "Value" "GND" (id 1) (at 139.7 72.39 0))
     (property "Footprint" "" (id 2) (at 139.7 67.31 0)
       (effects (font (size 1.27 1.27)) hide)
@@
     (in_bom yes) (on_board yes) (fields_autoplaced)
     (property "Reference" "C2" (id 0) (at 133.35 58.42 90))
-    (property "Value" "" (id 1) (at 133.35 60.96 90))
+    (property "Value" ".1uF" (id 1) (at 133.35 60.96 90))
     (property "Footprint" "" (id 2) (at 129.54 67.0052 0)
       (effects (font (size 1.27 1.27)) hide)

Commit message: fixes
Connections:
- no-connect marks 0 -> 8
Changed lines of the file:
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@@
   (junction (at 129.54 66.04) (diameter 0) (color 0 0 0 0)
   )
-  (junction (at 129.54 69.85) (diameter 0) (color 0 0 0 0)
+  (junction (at 129.54 67.31) (diameter 0) (color 0 0 0 0)
   )
   (junction (at 109.22 77.47) (diameter 0) (color 0 0 0 0)
@@
   (junction (at 118.11 97.79) (diameter 0) (color 0 0 0 0)
   )
+  (no_connect (at 119.38 107.95))
+  (no_connect (at 119.38 82.55))
+  (no_connect (at 119.38 85.09))
+  (no_connect (at 119.38 87.63))
+  (no_connect (at 119.38 90.17))
+  (no_connect (at 139.7 92.71))
+  (no_connect (at 139.7 95.25))
+  (no_connect (at 119.38 95.25))
   (wire (pts (xy 142.24 109.22) (xy 142.24 107.95))
     (stroke (width 0) (type default) (color 0 0 0 0))
@@
     (stroke (width 0) (type default) (color 0 0 0 0))
   )
-  (wire (pts (xy 114.3 67.31) (xy 111.76 67.31))
+  (wire (pts (xy 111.76 67.31) (xy 129.54 67.31))
     (stroke (width 0) (type default) (color 0 0 0 0))
   )
@@
   )
   (wire (pts (xy 101.6 77.47) (xy 106.68 77.47))
-    (stroke (width 0) (type default) (color 0 0 0 0))
-  )
-  (wire (pts (xy 114.3 69.85) (xy 114.3 67.31))
     (stroke (width 0) (type default) (color 0 0 0 0))
   )
@@
     (stroke (width 0) (type default) (color 0 0 0 0))
   )
-  (wire (pts (xy 129.54 69.85) (xy 129.54 72.39))
+  (wire (pts (xy 129.54 67.31) (xy 129.54 72.39))
     (stroke (width 0) (type default) (color 0 0 0 0))
   )
-  (wire (pts (xy 129.54 66.04) (xy 129.54 69.85))
+  (wire (pts (xy 129.54 66.04) (xy 129.54 67.31))
     (stroke (width 0) (type default) (color 0 0 0 0))
   )
@@
     (stroke (width 0) (type default) (color 0 0 0 0))
   )
-  (wire (pts (xy 129.54 69.85) (xy 114.3 69.85))
-    (stroke (width 0) (type default) (color 0 0 0 0))
-  )

Commit message: final look
Parts:
- renumbered C1 to C301, C2 to C302, D1 to D301, R1 to R301, SW1 to SW301, U2 to U301, Y1 to Y301
Changed lines of the file:
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@@
   (symbol (lib_id "Switch:SW_DIP_x01") (at 93.98 77.47 180) (unit 1)
     (in_bom yes) (on_board yes) (fields_autoplaced)
-    (property "Reference" "SW1" (id 0) (at 93.98 85.09 0))
+    (property "Reference" "SW301" (id 0) (at 93.98 85.09 0))
     (property "Value" "SW_DIP_x01" (id 1) (at 93.98 82.55 0))
     (property "Footprint" "" (id 2) (at 93.98 77.47 0)
@@
   (symbol (lib_id "Device:R") (at 106.68 72.39 180) (unit 1)
     (in_bom yes) (on_board yes) (fields_autoplaced)
-    (property "Reference" "R1" (id 0) (at 104.14 73.6601 0)
+    (property "Reference" "R301" (id 0) (at 104.14 73.6601 0)
       (effects (font (size 1.27 1.27)) (justify left))
     )
@@
   (symbol (lib_id "power:GND") (at 139.7 67.31 0) (unit 1)
     (in_bom yes) (on_board yes) (fields_autoplaced)
-    (property "Reference" "#PWR0110" (id 0) (at 139.7 73.66 0)
+    (property "Reference" "#PWR0302" (id 0) (at 139.7 73.66 0)
       (effects (font (size 1.27 1.27)) hide)
     )
@@
   (symbol (lib_id "Timer:8284") (at 129.54 92.71 0) (unit 1)
     (in_bom yes) (on_board yes) (fields_autoplaced)
-    (property "Reference" "U2" (id 0) (at 131.5594 69.85 0)
+    (property "Reference" "U301" (id 0) (at 131.5594 69.85 0)
       (effects (font (size 1.27 1.27)) (justify left))
     )
@@
   (symbol (lib_id "Device:Crystal") (at 146.05 105.41 90) (unit 1)
     (in_bom yes) (on_board yes) (fields_autoplaced)
-    (property "Reference" "Y1" (id 0) (at 149.86 104.1399 90)
+    (property "Reference" "Y301" (id 0) (at 149.86 104.1399 90)
       (effects (font (size 1.27 1.27)) (justify right))
     )
@@
   (symbol (lib_id "Device:LED") (at 111.76 72.39 90) (unit 1)
     (in_bom yes) (on_board yes) (fields_autoplaced)
-    (property "Reference" "D1" (id 0) (at 115.57 72.7074 90)
+    (property "Reference" "D301" (id 0) (at 115.57 72.7074 90)
       (effects (font (size 1.27 1.27)) (justify right))
     )
@@
   (symbol (lib_id "power:GND") (at 129.54 115.57 0) (unit 1)
     (in_bom yes) (on_board yes) (fields_autoplaced)
-    (property "Reference" "#PWR0104" (id 0) (at 129.54 121.92 0)
+    (property "Reference" "#PWR0301" (id 0) (at 129.54 121.92 0)
       (effects (font (size 1.27 1.27)) hide)
     )
@@
   (symbol (lib_id "Device:C") (at 109.22 83.82 180) (unit 1)
     (in_bom yes) (on_board yes) (fields_autoplaced)
-    (property "Reference" "C1" (id 0) (at 105.41 85.0901 0)
+    (property "Reference" "C301" (id 0) (at 105.41 85.0901 0)
       (effects (font (size 1.27 1.27)) (justify left))
     )
@@
   (symbol (lib_id "Device:C") (at 133.35 66.04 270) (unit 1)
     (in_bom yes) (on_board yes) (fields_autoplaced)
-    (property "Reference" "C2" (id 0) (at 133.35 58.42 90))
+    (property "Reference" "C302" (id 0) (at 133.35 58.42 90))
     (property "Value" ".1uF" (id 1) (at 133.35 60.96 90))
     (property "Footprint" "" (id 2) (at 129.54 67.0052 0)

Commit message: footprints
Parts:
- C301, C302: footprint (none) -> Capacitor_SMD:CP_Elec_3x5.3
- D301: footprint (none) -> LED_SMD:LED_0201_0603Metric
Changed lines of the file:
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@@
       (effects (font (size 1.27 1.27)) (justify right))
     )
-    (property "Footprint" "" (id 2) (at 111.76 72.39 0)
+    (property "Footprint" "LED_SMD:LED_0201_0603Metric" (id 2) (at 111.76 72.39 0)
       (effects (font (size 1.27 1.27)) hide)
     )
@@
       (effects (font (size 1.27 1.27)) (justify left))
     )
-    (property "Footprint" "" (id 2) (at 108.2548 80.01 0)
+    (property "Footprint" "Capacitor_SMD:CP_Elec_3x5.3" (id 2) (at 108.2548 80.01 0)
       (effects (font (size 1.27 1.27)) hide)
     )
@@
     (property "Reference" "C302" (id 0) (at 133.35 58.42 90))
     (property "Value" ".1uF" (id 1) (at 133.35 60.96 90))
-    (property "Footprint" "" (id 2) (at 129.54 67.0052 0)
+    (property "Footprint" "Capacitor_SMD:CP_Elec_3x5.3" (id 2) (at 129.54 67.0052 0)
       (effects (font (size 1.27 1.27)) hide)
     )

Commit message: pcb
Parts:
- R301: footprint (none) -> Resistor_SMD:R_0201_0603Metric
- SW301: footprint (none) -> Button_Switch_SMD:SW_DIP_SPSTx01_Slide_6.7x4.1mm_W6.73mm_P2.54mm_LowProfile_JPin
Changed lines of the file:
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@@
     (property "Reference" "SW301" (id 0) (at 93.98 85.09 0))
     (property "Value" "SW_DIP_x01" (id 1) (at 93.98 82.55 0))
-    (property "Footprint" "" (id 2) (at 93.98 77.47 0)
+    (property "Footprint" "Button_Switch_SMD:SW_DIP_SPSTx01_Slide_6.7x4.1mm_W6.73mm_P2.54mm_LowProfile_JPin" (id 2) (at 93.98 77.47 0)
       (effects (font (size 1.27 1.27)) hide)
     )
@@
       (effects (font (size 1.27 1.27)) (justify left))
     )
-    (property "Footprint" "" (id 2) (at 108.458 72.39 90)
+    (property "Footprint" "Resistor_SMD:R_0201_0603Metric" (id 2) (at 108.458 72.39 90)
       (effects (font (size 1.27 1.27)) hide)
     )
