File: 8086proj/ClockFinal.kicad_sch (KiCad schematic)
At the start: 7 parts, among them SW301 SW_DIP_x01

Commit message: pcb update
Parts:
- U301: footprint (none) -> Package_DIP:DIP-18_W7.62mm
- Y301: footprint (none) -> Crystal:Crystal_AT310_D3.0mm_L10.0mm_Horizontal
Changed lines of the file:
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@@
       (effects (font (size 1.27 1.27)) (justify left))
     )
-    (property "Footprint" "" (id 2) (at 129.54 92.71 0)
+    (property "Footprint" "Package_DIP:DIP-18_W7.62mm" (id 2) (at 129.54 92.71 0)
       (effects (font (size 1.27 1.27) italic) hide)
     )
@@
       (effects (font (size 1.27 1.27)) (justify right))
     )
-    (property "Footprint" "" (id 2) (at 146.05 105.41 0)
+    (property "Footprint" "Crystal:Crystal_AT310_D3.0mm_L10.0mm_Horizontal" (id 2) (at 146.05 105.41 0)
       (effects (font (size 1.27 1.27)) hide)
     )
