File: 8086proj/LCD.kicad_sch (KiCad schematic)
At the start: 5 parts

Commit message: 74244
Parts:
- C?: value (none) -> C
- DS?: value (none) -> LCD4x20; footprint (none) -> LCD4x20
- R?: value (none) -> R
- U?: value (none) -> PAL16L8
Changed lines of the file:
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@@
       (effects (font (size 1.27 1.27)) hide)
     )
-    (property "Value" "" (id 1) (at 193.04 107.9499 90)
+    (property "Value" "GND" (id 1) (at 193.04 107.9499 90)
       (effects (font (size 1.27 1.27)) (justify right))
     )
@@
     (in_bom yes) (on_board yes) (fields_autoplaced)
     (property "Reference" "R?" (id 0) (at 157.48 93.98 90))
-    (property "Value" "" (id 1) (at 157.48 96.52 90))
+    (property "Value" "R" (id 1) (at 157.48 96.52 90))
     (property "Footprint" "" (id 2) (at 157.48 102.108 90)
       (effects (font (size 1.27 1.27)) hide)
@@
       (effects (font (size 1.27 1.27)) hide)
     )
-    (property "Value" "" (id 1) (at 170.18 85.0899 90)
+    (property "Value" "GND" (id 1) (at 170.18 85.0899 90)
       (effects (font (size 1.27 1.27)) (justify right))
     )
@@
       (effects (font (size 1.27 1.27)) hide)
     )
-    (property "Value" "" (id 1) (at 73.66 116.84 0))
+    (property "Value" "GND" (id 1) (at 73.66 116.84 0))
     (property "Footprint" "" (id 2) (at 73.66 111.76 0)
       (effects (font (size 1.27 1.27)) hide)
@@
     (in_bom yes) (on_board yes) (fields_autoplaced)
     (property "Reference" "C?" (id 0) (at 161.29 76.2 90))
-    (property "Value" "" (id 1) (at 161.29 78.74 90))
+    (property "Value" "C" (id 1) (at 161.29 78.74 90))
     (property "Footprint" "" (id 2) (at 165.1 82.8548 0)
       (effects (font (size 1.27 1.27)) hide)
@@
       (effects (font (size 1.27 1.27)) (justify left))
     )
-    (property "Value" "" (id 1) (at 75.6794 80.01 0)
+    (property "Value" "PAL16L8" (id 1) (at 75.6794 80.01 0)
       (effects (font (size 1.27 1.27)) (justify left))
     )
@@
     (in_bom yes) (on_board yes) (fields_autoplaced)
     (property "Reference" "DS?" (id 0) (at 175.26 87.63 0))
-    (property "Value" "" (id 1) (at 175.26 90.17 0))
-    (property "Footprint" "" (id 2) (at 185.42 92.71 0)
+    (property "Value" "LCD4x20" (id 1) (at 175.26 90.17 0))
+    (property "Footprint" "LCD4x20" (id 2) (at 185.42 92.71 0)
       (effects (font (size 1.27 1.27)) (justify left) hide)
     )

Commit message: final look
Parts:
- gave numbers to parts that had none: 5
Changed lines of the file:
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@@
   (symbol (lib_id "power:GND") (at 189.23 107.95 90) (unit 1)
     (in_bom yes) (on_board yes) (fields_autoplaced)
-    (property "Reference" "#PWR?" (id 0) (at 195.58 107.95 0)
+    (property "Reference" "#PWR01205" (id 0) (at 195.58 107.95 0)
       (effects (font (size 1.27 1.27)) hide)
     )
@@
   (symbol (lib_id "Device:R") (at 157.48 100.33 90) (unit 1)
     (in_bom yes) (on_board yes) (fields_autoplaced)
-    (property "Reference" "R?" (id 0) (at 157.48 93.98 90))
+    (property "Reference" "R1201" (id 0) (at 157.48 93.98 90))
     (property "Value" "R" (id 1) (at 157.48 96.52 90))
     (property "Footprint" "" (id 2) (at 157.48 102.108 90)
@@
   (symbol (lib_id "power:GND") (at 96.52 74.93 90) (unit 1)
     (in_bom yes) (on_board yes) (fields_autoplaced)
-    (property "Reference" "#PWR?" (id 0) (at 102.87 74.93 0)
+    (property "Reference" "#PWR01202" (id 0) (at 102.87 74.93 0)
       (effects (font (size 1.27 1.27)) hide)
     )
@@
   (symbol (lib_id "Device:C") (at 91.44 73.66 90) (unit 1)
     (in_bom yes) (on_board yes) (fields_autoplaced)
-    (property "Reference" "C?" (id 0) (at 91.44 66.04 90))
+    (property "Reference" "C1201" (id 0) (at 91.44 66.04 90))
     (property "Value" "C" (id 1) (at 91.44 68.58 90))
     (property "Footprint" "" (id 2) (at 95.25 72.6948 0)
@@
   (symbol (lib_id "power:GND") (at 166.37 85.09 90) (unit 1)
     (in_bom yes) (on_board yes) (fields_autoplaced)
-    (property "Reference" "#PWR?" (id 0) (at 172.72 85.09 0)
+    (property "Reference" "#PWR01204" (id 0) (at 172.72 85.09 0)
       (effects (font (size 1.27 1.27)) hide)
     )
@@
   (symbol (lib_id "power:GND") (at 73.66 111.76 0) (unit 1)
     (in_bom yes) (on_board yes) (fields_autoplaced)
-    (property "Reference" "#PWR?" (id 0) (at 73.66 118.11 0)
+    (property "Reference" "#PWR01201" (id 0) (at 73.66 118.11 0)
       (effects (font (size 1.27 1.27)) hide)
     )
@@
   (symbol (lib_id "power:GND") (at 161.29 95.25 0) (unit 1)
     (in_bom yes) (on_board yes) (fields_autoplaced)
-    (property "Reference" "#PWR?" (id 0) (at 161.29 101.6 0)
+    (property "Reference" "#PWR01203" (id 0) (at 161.29 101.6 0)
       (effects (font (size 1.27 1.27)) hide)
     )
@@
   (symbol (lib_id "Device:C") (at 161.29 83.82 90) (unit 1)
     (in_bom yes) (on_board yes) (fields_autoplaced)
-    (property "Reference" "C?" (id 0) (at 161.29 76.2 90))
+    (property "Reference" "C1202" (id 0) (at 161.29 76.2 90))
     (property "Value" "C" (id 1) (at 161.29 78.74 90))
     (property "Footprint" "" (id 2) (at 165.1 82.8548 0)
@@
   (symbol (lib_id "Logic_Programmable:PAL16L8") (at 73.66 96.52 0) (unit 1)
     (in_bom yes) (on_board yes) (fields_autoplaced)
-    (property "Reference" "U?" (id 0) (at 75.6794 77.47 0)
+    (property "Reference" "U1201" (id 0) (at 75.6794 77.47 0)
       (effects (font (size 1.27 1.27)) (justify left))
     )
@@
   (symbol (lib_id "LCD4x20:LCD4x20") (at 161.29 95.25 0) (unit 1)
     (in_bom yes) (on_board yes) (fields_autoplaced)
-    (property "Reference" "DS?" (id 0) (at 175.26 87.63 0))
+    (property "Reference" "DS1201" (id 0) (at 175.26 87.63 0))
     (property "Value" "LCD4x20" (id 1) (at 175.26 90.17 0))
     (property "Footprint" "LCD4x20" (id 2) (at 185.42 92.71 0)

Commit message: footprints
Parts:
- C1201, C1202: footprint (none) -> Capacitor_SMD:CP_Elec_3x5.3
Changed lines of the file:
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@@
     (property "Reference" "C1201" (id 0) (at 91.44 66.04 90))
     (property "Value" "C" (id 1) (at 91.44 68.58 90))
-    (property "Footprint" "" (id 2) (at 95.25 72.6948 0)
+    (property "Footprint" "Capacitor_SMD:CP_Elec_3x5.3" (id 2) (at 95.25 72.6948 0)
       (effects (font (size 1.27 1.27)) hide)
     )
@@
     (property "Reference" "C1202" (id 0) (at 161.29 76.2 90))
     (property "Value" "C" (id 1) (at 161.29 78.74 90))
-    (property "Footprint" "" (id 2) (at 165.1 82.8548 0)
+    (property "Footprint" "Capacitor_SMD:CP_Elec_3x5.3" (id 2) (at 165.1 82.8548 0)
       (effects (font (size 1.27 1.27)) hide)
     )

Commit message: pcb
Parts:
- DS1201: footprint LCD4x20 -> Display:LCD-016N002L
- R1201: footprint (none) -> Resistor_SMD:R_0201_0603Metric
- U1201: footprint (none) -> Package_DIP:DIP-20_W7.62mm
Changed lines of the file:
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@@
     (property "Reference" "R1201" (id 0) (at 157.48 93.98 90))
     (property "Value" "R" (id 1) (at 157.48 96.52 90))
-    (property "Footprint" "" (id 2) (at 157.48 102.108 90)
+    (property "Footprint" "Resistor_SMD:R_0201_0603Metric" (id 2) (at 157.48 102.108 90)
       (effects (font (size 1.27 1.27)) hide)
     )
@@
       (effects (font (size 1.27 1.27)) (justify left))
     )
-    (property "Footprint" "" (id 2) (at 73.66 96.52 0)
+    (property "Footprint" "Package_DIP:DIP-20_W7.62mm" (id 2) (at 73.66 96.52 0)
       (effects (font (size 1.27 1.27)) hide)
     )
@@
     (property "Reference" "DS1201" (id 0) (at 175.26 87.63 0))
     (property "Value" "LCD4x20" (id 1) (at 175.26 90.17 0))
-    (property "Footprint" "LCD4x20" (id 2) (at 185.42 92.71 0)
+    (property "Footprint" "Display:LCD-016N002L" (id 2) (at 185.42 92.71 0)
       (effects (font (size 1.27 1.27)) (justify left) hide)
     )
