File: 8086proj/8254.kicad_sch (KiCad schematic)
At the start: 10 parts, among them J0 Conn_01x01_Female, J1 Conn_01x01_Female

Commit message: fixes
Parts:
- removed J0, J1: Conn_01x01_Female, symbol Connector:Conn_01x01_Female
- added J?: (no value), symbol Connector:Conn_01x03_Male
- added J?: (no value), symbol Connector:Conn_01x02_Male
- added J?: Conn_01x03_Male, symbol Connector:Conn_01x03_Male
Connections:
- net at U?.10 (OUT0): now also J?.1 (Pin_1)
- net at U?.11 (G0): now also J?.2 (Pin_2)
- net at U?.14 (G1): now also J?.1 (Pin_1)
- net at U?.16 (G2): now also J?.2 (Pin_2)
- net at U?.17 (OUT2): now also J?.1 (Pin_1)
- removed net CLK: U?.15 (CLK1), U?.18 (CLK2), U?.9 (CLK0)
- new net: J?.3 (Pin_3), U?.9 (CLK0)
- new net: J?.2 (Pin_2), U?.15 (CLK1)
- new net: J?.3 (Pin_3), U?.18 (CLK2)
Changed lines of the file:
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@@
 (kicad_sch (version 20211123) (generator eeschema)
   (paper "A4")
-  (junction (at 168.91 90.17) (diameter 0) (color 0 0 0 0)
-  )
   (junction (at 156.21 78.74) (diameter 0) (color 0 0 0 0)
   )
   (junction (at 76.2 83.82) (diameter 0) (color 0 0 0 0)
-  )
-  (junction (at 168.91 102.87) (diameter 0) (color 0 0 0 0)
   )
   (no_connect (at 88.9 107.95))
@@
     (stroke (width 0) (type default) (color 0 0 0 0))
   )
-  (wire (pts (xy 166.37 115.57) (xy 168.91 115.57))
-    (stroke (width 0) (type default) (color 0 0 0 0))
-  )
   (bus (pts (xy 31.75 29.21) (xy 71.12 29.21))
     (stroke (width 0) (type default) (color 0 0 0 0))
@@
     (stroke (width 0) (type default) (color 0 0 0 0))
   )
-  (wire (pts (xy 168.91 102.87) (xy 168.91 90.17))
-    (stroke (width 0) (type default) (color 0 0 0 0))
-  )
   (wire (pts (xy 76.2 80.01) (xy 76.2 83.82))
     (stroke (width 0) (type default) (color 0 0 0 0))
@@
     (stroke (width 0) (type default) (color 0 0 0 0))
   )
-  (wire (pts (xy 166.37 102.87) (xy 168.91 102.87))
-    (stroke (width 0) (type default) (color 0 0 0 0))
-  )
   (wire (pts (xy 60.96 95.25) (xy 63.5 95.25))
     (stroke (width 0) (type default) (color 0 0 0 0))
@@
     (stroke (width 0) (type default) (color 0 0 0 0))
   )
-  (wire (pts (xy 166.37 90.17) (xy 168.91 90.17))
-    (stroke (width 0) (type default) (color 0 0 0 0))
-  )
   (wire (pts (xy 33.02 88.9) (xy 35.56 88.9))
     (stroke (width 0) (type default) (color 0 0 0 0))
@@
     (stroke (width 0) (type default) (color 0 0 0 0))
   )
-  (wire (pts (xy 166.37 107.95) (xy 173.99 107.95))
-    (stroke (width 0) (type default) (color 0 0 0 0))
-  )
-  (wire (pts (xy 168.91 90.17) (xy 171.45 90.17))
-    (stroke (width 0) (type default) (color 0 0 0 0))
-  )
   (wire (pts (xy 31.75 31.75) (xy 40.64 31.75))
     (stroke (width 0) (type default) (color 0 0 0 0))
@@
   )
   (wire (pts (xy 60.96 92.71) (xy 63.5 92.71))
-    (stroke (width 0) (type default) (color 0 0 0 0))
-  )
-  (wire (pts (xy 168.91 115.57) (xy 168.91 102.87))
     (stroke (width 0) (type default) (color 0 0 0 0))
   )
@@
     (effects (font (size 1.27 1.27)) (justify right bottom))
   )
-  (hierarchical_label "C2out" (shape input) (at 173.99 107.95 0)
+  (label "VIN" (at 40.64 31.75 180)
+    (effects (font (size 1.27 1.27)) (justify right bottom))
+  )
+  (hierarchical_label "C2out" (shape input) (at 166.37 107.95 0)
     (effects (font (size 1.27 1.27)) (justify left))
   )
@@
   (hierarchical_label "_RD" (shape output) (at 146.05 110.49 180)
     (effects (font (size 1.27 1.27)) (justify right))
-  )
-  (hierarchical_label "CLK" (shape output) (at 171.45 90.17 0)
-    (effects (font (size 1.27 1.27)) (justify left))
   )
   (hierarchical_label "_WR" (shape output) (at 146.05 113.03 180)
@@
     (pin "7")
   )
+  (symbol (lib_id "Connector:Conn_01x03_Male") (at 171.45 92.71 180) (unit 1)
+    (in_bom yes) (on_board yes) (fields_autoplaced)
+    (property "Reference" "J?" (id 0) (at 172.72 91.4399 0)
+      (effects (font (size 1.27 1.27)) (justify right))
+    )
+    (property "Value" "" (id 1) (at 172.72 93.9799 0)
+      (effects (font (size 1.27 1.27)) (justify right))
+    )
+    (property "Footprint" "" (id 2) (at 171.45 92.71 0)
+      (effects (font (size 1.27 1.27)) hide)
+    )
+    (property "Datasheet" "~" (id 3) (at 171.45 92.71 0)
+      (effects (font (size 1.27 1.27)) hide)
+    )
+    (pin "1")
+    (pin "2")
+    (pin "3")
+  )
+  (symbol (lib_id "Connector:Conn_01x02_Male") (at 171.45 105.41 180) (unit 1)
+    (in_bom yes) (on_board yes) (fields_autoplaced)
+    (property "Reference" "J?" (id 0) (at 172.72 102.8699 0)
+      (effects (font (size 1.27 1.27)) (justify right))
+    )
+    (property "Value" "" (id 1) (at 172.72 105.4099 0)
+      (effects (font (size 1.27 1.27)) (justify right))
+    )
+    (property "Footprint" "" (id 2) (at 171.45 105.41 0)
+      (effects (font (size 1.27 1.27)) hide)
+    )
+    (property "Datasheet" "~" (id 3) (at 171.45 105.41 0)
+      (effects (font (size 1.27 1.27)) hide)
+    )
+    (pin "1")
+    (pin "2")
+  )
   (symbol (lib_id "power:GND") (at 68.58 83.82 180) (unit 1)
     (in_bom yes) (on_board yes) (fields_autoplaced)
@@
     )
     (property "Datasheet" "" (id 3) (at 148.59 78.74 0)
-      (effects (font (size 1.27 1.27)) hide)
-    )
-    (pin "1")
-  )
-  (symbol (lib_id "Connector:Conn_01x01_Female") (at 171.45 95.25 0) (unit 1)
-    (in_bom yes) (on_board yes) (fields_autoplaced)
-    (property "Reference" "J0" (id 0) (at 172.72 93.9799 0)
-      (effects (font (size 1.27 1.27)) (justify left))
-    )
-    (property "Value" "Conn_01x01_Female" (id 1) (at 172.72 96.5199 0)
-      (effects (font (size 1.27 1.27)) (justify left))
-    )
-    (property "Footprint" "" (id 2) (at 171.45 95.25 0)
-      (effects (font (size 1.27 1.27)) hide)
-    )
-    (property "Datasheet" "~" (id 3) (at 171.45 95.25 0)
       (effects (font (size 1.27 1.27)) hide)
     )
@@
     (pin "2")
   )
-  (symbol (lib_id "Connector:Conn_01x01_Female") (at 171.45 120.65 0) (unit 1)
-    (in_bom yes) (on_board yes) (fields_autoplaced)
-    (property "Reference" "J1" (id 0) (at 172.72 119.3799 0)
-      (effects (font (size 1.27 1.27)) (justify left))
-    )
-    (property "Value" "Conn_01x01_Female" (id 1) (at 172.72 121.9199 0)
-      (effects (font (size 1.27 1.27)) (justify left))
-    )
-    (property "Footprint" "" (id 2) (at 171.45 120.65 0)
-      (effects (font (size 1.27 1.27)) hide)
-    )
-    (property "Datasheet" "~" (id 3) (at 171.45 120.65 0)
-      (effects (font (size 1.27 1.27)) hide)
-    )
-    (pin "1")
-  )
   (symbol (lib_id "power:GND") (at 76.2 118.11 0) (unit 1)
     (in_bom yes) (on_board yes) (fields_autoplaced)
@@
     (pin "9")
   )
+  (symbol (lib_id "Connector:Conn_01x03_Male") (at 171.45 118.11 180) (unit 1)
+    (in_bom yes) (on_board yes) (fields_autoplaced)
+    (property "Reference" "J?" (id 0) (at 172.72 116.8399 0)
+      (effects (font (size 1.27 1.27)) (justify right))
+    )
+    (property "Value" "Conn_01x03_Male" (id 1) (at 172.72 119.3799 0)
+      (effects (font (size 1.27 1.27)) (justify right))
+    )
+    (property "Footprint" "" (id 2) (at 171.45 118.11 0)
+      (effects (font (size 1.27 1.27)) hide)
+    )
+    (property "Datasheet" "~" (id 3) (at 171.45 118.11 0)
+      (effects (font (size 1.27 1.27)) hide)
+    )
+    (pin "1")
+    (pin "2")
+    (pin "3")
+  )
 )

Commit message: final look
Parts:
- J1001: renamed from J?; value (none) -> Conn_01x03_Male
- J1002: renamed from J?; value (none) -> Conn_01x02_Male
- gave numbers to parts that had none: 9
Changed lines of the file:
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@@
   (symbol (lib_id "74xx:74LS21") (at 43.18 109.22 0) (unit 2)
     (in_bom yes) (on_board yes) (fields_autoplaced)
-    (property "Reference" "U?" (id 0) (at 43.18 99.06 0))
+    (property "Reference" "U1002" (id 0) (at 43.18 99.06 0))
     (property "Value" "74LS21" (id 1) (at 43.18 101.6 0))
     (property "Footprint" "" (id 2) (at 43.18 109.22 0)
@@
   (symbol (lib_id "74xx:74LS21") (at 43.18 125.73 0) (unit 2)
     (in_bom yes) (on_board yes) (fields_autoplaced)
-    (property "Reference" "U?" (id 0) (at 43.18 115.57 0))
+    (property "Reference" "U1003" (id 0) (at 43.18 115.57 0))
     (property "Value" "74LS21" (id 1) (at 43.18 118.11 0))
     (property "Footprint" "" (id 2) (at 43.18 125.73 0)
@@
   (symbol (lib_id "Connector:Conn_01x03_Male") (at 171.45 92.71 180) (unit 1)
     (in_bom yes) (on_board yes) (fields_autoplaced)
-    (property "Reference" "J?" (id 0) (at 172.72 91.4399 0)
-      (effects (font (size 1.27 1.27)) (justify right))
-    )
-    (property "Value" "" (id 1) (at 172.72 93.9799 0)
+    (property "Reference" "J1001" (id 0) (at 172.72 91.4399 0)
+      (effects (font (size 1.27 1.27)) (justify right))
+    )
+    (property "Value" "Conn_01x03_Male" (id 1) (at 172.72 93.9799 0)
       (effects (font (size 1.27 1.27)) (justify right))
     )
@@
   (symbol (lib_id "Connector:Conn_01x02_Male") (at 171.45 105.41 180) (unit 1)
     (in_bom yes) (on_board yes) (fields_autoplaced)
-    (property "Reference" "J?" (id 0) (at 172.72 102.8699 0)
-      (effects (font (size 1.27 1.27)) (justify right))
-    )
-    (property "Value" "" (id 1) (at 172.72 105.4099 0)
+    (property "Reference" "J1002" (id 0) (at 172.72 102.8699 0)
+      (effects (font (size 1.27 1.27)) (justify right))
+    )
+    (property "Value" "Conn_01x02_Male" (id 1) (at 172.72 105.4099 0)
       (effects (font (size 1.27 1.27)) (justify right))
     )
@@
   (symbol (lib_id "power:GND") (at 68.58 83.82 180) (unit 1)
     (in_bom yes) (on_board yes) (fields_autoplaced)
-    (property "Reference" "#PWR?" (id 0) (at 68.58 77.47 0)
+    (property "Reference" "#PWR01001" (id 0) (at 68.58 77.47 0)
       (effects (font (size 1.27 1.27)) hide)
     )
@@
   (symbol (lib_id "74xx:74LS21") (at 43.18 92.71 0) (unit 1)
     (in_bom yes) (on_board yes) (fields_autoplaced)
-    (property "Reference" "U?" (id 0) (at 43.18 82.55 0))
+    (property "Reference" "U802" (id 0) (at 43.18 82.55 0))
     (property "Value" "74LS21" (id 1) (at 43.18 85.09 0))
     (property "Footprint" "" (id 2) (at 43.18 92.71 0)
@@
   (symbol (lib_id "power:GND") (at 148.59 78.74 180) (unit 1)
     (in_bom yes) (on_board yes) (fields_autoplaced)
-    (property "Reference" "#PWR?" (id 0) (at 148.59 72.39 0)
+    (property "Reference" "#PWR01003" (id 0) (at 148.59 72.39 0)
       (effects (font (size 1.27 1.27)) hide)
     )
@@
   (symbol (lib_id "Timer:8254") (at 156.21 105.41 0) (unit 1)
     (in_bom yes) (on_board yes) (fields_autoplaced)
-    (property "Reference" "U?" (id 0) (at 158.2294 77.47 0)
+    (property "Reference" "U1005" (id 0) (at 158.2294 77.47 0)
       (effects (font (size 1.27 1.27)) (justify left))
     )
@@
   (symbol (lib_id "Device:C") (at 152.4 78.74 90) (unit 1)
     (in_bom yes) (on_board yes)
-    (property "Reference" "C?" (id 0) (at 151.1299 74.93 0)
+    (property "Reference" "C1002" (id 0) (at 151.1299 74.93 0)
       (effects (font (size 1.27 1.27)) (justify left))
     )
@@
   (symbol (lib_id "power:GND") (at 76.2 118.11 0) (unit 1)
     (in_bom yes) (on_board yes) (fields_autoplaced)
-    (property "Reference" "#PWR?" (id 0) (at 76.2 124.46 0)
+    (property "Reference" "#PWR01002" (id 0) (at 76.2 124.46 0)
       (effects (font (size 1.27 1.27)) hide)
     )
@@
   (symbol (lib_id "Device:C") (at 72.39 83.82 90) (unit 1)
     (in_bom yes) (on_board yes)
-    (property "Reference" "C?" (id 0) (at 71.1199 80.01 0)
+    (property "Reference" "C1001" (id 0) (at 71.1199 80.01 0)
       (effects (font (size 1.27 1.27)) (justify left))
     )
@@
   (symbol (lib_id "power:GND") (at 156.21 130.81 0) (unit 1)
     (in_bom yes) (on_board yes) (fields_autoplaced)
-    (property "Reference" "#PWR?" (id 0) (at 156.21 137.16 0)
+    (property "Reference" "#PWR01004" (id 0) (at 156.21 137.16 0)
       (effects (font (size 1.27 1.27)) hide)
     )
@@
   (symbol (lib_id "74xx:74LS04") (at 27.94 91.44 0) (unit 1)
     (in_bom yes) (on_board yes) (fields_autoplaced)
-    (property "Reference" "U?" (id 0) (at 27.94 82.55 0))
+    (property "Reference" "U1001" (id 0) (at 27.94 82.55 0))
     (property "Value" "74LS04" (id 1) (at 27.94 85.09 0))
     (property "Footprint" "" (id 2) (at 27.94 91.44 0)
@@
   (symbol (lib_id "Logic_Programmable:PAL16L8") (at 76.2 102.87 0) (unit 1)
     (in_bom yes) (on_board yes) (fields_autoplaced)
-    (property "Reference" "U?" (id 0) (at 78.2194 83.82 0)
+    (property "Reference" "U1004" (id 0) (at 78.2194 83.82 0)
       (effects (font (size 1.27 1.27)) (justify left))
     )
@@
   (symbol (lib_id "Connector:Conn_01x03_Male") (at 171.45 118.11 180) (unit 1)
     (in_bom yes) (on_board yes) (fields_autoplaced)
-    (property "Reference" "J?" (id 0) (at 172.72 116.8399 0)
-      (effects (font (size 1.27 1.27)) (justify right))
-    )
+    (property "Reference" "J1003" (id 0) (at 172.72 116.8399 0)
+      (effects (font (size 1.27 1.27)) (justify right))
+    )

Commit message: footprints
Parts:
- C1001, C1002: footprint (none) -> Capacitor_SMD:CP_Elec_3x5.3
Changed lines of the file:
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@@
       (effects (font (size 1.27 1.27)) (justify left))
     )
-    (property "Footprint" "" (id 2) (at 156.21 77.7748 0)
+    (property "Footprint" "Capacitor_SMD:CP_Elec_3x5.3" (id 2) (at 156.21 77.7748 0)
       (effects (font (size 1.27 1.27)) hide)
     )
@@
       (effects (font (size 1.27 1.27)) (justify left))
     )
-    (property "Footprint" "" (id 2) (at 76.2 82.8548 0)
+    (property "Footprint" "Capacitor_SMD:CP_Elec_3x5.3" (id 2) (at 76.2 82.8548 0)
       (effects (font (size 1.27 1.27)) hide)
     )

Commit message: pcb
Parts:
- J1001, J1003: footprint (none) -> Connector_PinHeader_1.00mm:PinHeader_1x03_P1.00mm_Vertical
- J1002: footprint (none) -> Connector_PinHeader_1.00mm:PinHeader_1x02_P1.00mm_Vertical
- U1004: footprint (none) -> Package_DIP:DIP-20_W7.62mm
Changed lines of the file:
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@@
       (effects (font (size 1.27 1.27)) (justify right))
     )
-    (property "Footprint" "" (id 2) (at 171.45 92.71 0)
+    (property "Footprint" "Connector_PinHeader_1.00mm:PinHeader_1x03_P1.00mm_Vertical" (id 2) (at 171.45 92.71 0)
       (effects (font (size 1.27 1.27)) hide)
     )
@@
       (effects (font (size 1.27 1.27)) (justify right))
     )
-    (property "Footprint" "" (id 2) (at 171.45 105.41 0)
+    (property "Footprint" "Connector_PinHeader_1.00mm:PinHeader_1x02_P1.00mm_Vertical" (id 2) (at 171.45 105.41 0)
       (effects (font (size 1.27 1.27)) hide)
     )
@@
       (effects (font (size 1.27 1.27)) (justify left))
     )
-    (property "Footprint" "" (id 2) (at 76.2 102.87 0)
+    (property "Footprint" "Package_DIP:DIP-20_W7.62mm" (id 2) (at 76.2 102.87 0)
       (effects (font (size 1.27 1.27)) hide)
     )
@@
       (effects (font (size 1.27 1.27)) (justify right))
     )
-    (property "Footprint" "" (id 2) (at 171.45 118.11 0)
-      (effects (font (size 1.27 1.27)) hide)
-    )
+    (property "Footprint" "Connector_PinHeader_1.00mm:PinHeader_1x03_P1.00mm_Vertical" (id 2) (at 171.45 118.11 0)
+      (effects (font (size 1.27 1.27)) hide)
+    )

Commit message: pcb
Parts:
- U1001, U1002, U1003, U802: footprint (none) -> Package_DIP:DIP-14_W10.16mm
Changed lines of the file:
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@@
     (property "Reference" "U1002" (id 0) (at 43.18 99.06 0))
     (property "Value" "74LS21" (id 1) (at 43.18 101.6 0))
-    (property "Footprint" "" (id 2) (at 43.18 109.22 0)
+    (property "Footprint" "Package_DIP:DIP-14_W10.16mm" (id 2) (at 43.18 109.22 0)
       (effects (font (size 1.27 1.27)) hide)
     )
@@
     (property "Reference" "U1003" (id 0) (at 43.18 115.57 0))
     (property "Value" "74LS21" (id 1) (at 43.18 118.11 0))
-    (property "Footprint" "" (id 2) (at 43.18 125.73 0)
+    (property "Footprint" "Package_DIP:DIP-14_W10.16mm" (id 2) (at 43.18 125.73 0)
       (effects (font (size 1.27 1.27)) hide)
     )
@@
     (property "Reference" "U802" (id 0) (at 43.18 82.55 0))
     (property "Value" "74LS21" (id 1) (at 43.18 85.09 0))
-    (property "Footprint" "" (id 2) (at 43.18 92.71 0)
+    (property "Footprint" "Package_DIP:DIP-14_W10.16mm" (id 2) (at 43.18 92.71 0)
       (effects (font (size 1.27 1.27)) hide)
     )
@@
     (property "Reference" "U1001" (id 0) (at 27.94 82.55 0))
     (property "Value" "74LS04" (id 1) (at 27.94 85.09 0))
-    (property "Footprint" "" (id 2) (at 27.94 91.44 0)
-      (effects (font (size 1.27 1.27)) hide)
-    )
+    (property "Footprint" "Package_DIP:DIP-14_W10.16mm" (id 2) (at 27.94 91.44 0)
+      (effects (font (size 1.27 1.27)) hide)
+    )
