File: 8086proj/8259.kicad_sch (KiCad schematic)
At the start: 9 parts

Commit message: fixes
Parts:
- C0, C1: value (none) -> .1uF
- J?: value (none) -> Conn_01x04_Female
- R0: value (none) -> 10k
- U0: value (none) -> PAL16L8
- U1: value (none) -> 8259; footprint (none) -> Package_DIP:DIP-28_W15.24mm
- U? (x2): value (none) -> 74LS21
Changed lines of the file:
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@@
     (effects (font (size 1.27 1.27)) (justify right))
   )
-  (hierarchical_label "VIN" (shape output) (at 26.67 21.59 180)
+  (hierarchical_label "VIN" (shape input) (at 26.67 21.59 180)
     (effects (font (size 1.27 1.27)) (justify right))
   )
@@
     (in_bom yes) (on_board yes) (fields_autoplaced)
     (property "Reference" "U?" (id 0) (at 38.1 72.39 0))
-    (property "Value" "" (id 1) (at 38.1 74.93 0))
+    (property "Value" "74LS21" (id 1) (at 38.1 74.93 0))
     (property "Footprint" "" (id 2) (at 38.1 82.55 0)
       (effects (font (size 1.27 1.27)) hide)
@@
     (in_bom yes) (on_board yes) (fields_autoplaced)
     (property "Reference" "R0" (id 0) (at 160.02 106.68 90))
-    (property "Value" "" (id 1) (at 160.02 109.22 90))
+    (property "Value" "10k" (id 1) (at 160.02 109.22 90))
     (property "Footprint" "" (id 2) (at 160.02 114.808 90)
       (effects (font (size 1.27 1.27)) hide)
@@
       (effects (font (size 1.27 1.27)) (justify left))
     )
-    (property "Value" "" (id 1) (at 160.02 85.0899 0)
+    (property "Value" "Conn_01x04_Female" (id 1) (at 160.02 85.0899 0)
       (effects (font (size 1.27 1.27)) (justify left))
     )
@@
       (effects (font (size 1.27 1.27)) (justify left))
     )
-    (property "Value" "" (id 1) (at 135.8899 67.31 0)
+    (property "Value" ".1uF" (id 1) (at 135.8899 67.31 0)
       (effects (font (size 1.27 1.27)) (justify left))
     )
@@
       (effects (font (size 1.27 1.27)) (justify left))
     )
-    (property "Value" "" (id 1) (at 73.1394 76.2 0)
+    (property "Value" "PAL16L8" (id 1) (at 73.1394 76.2 0)
       (effects (font (size 1.27 1.27)) (justify left))
     )
@@
       (effects (font (size 1.27 1.27)) (justify left))
     )
-    (property "Value" "" (id 1) (at 140.4494 73.66 0)
-      (effects (font (size 1.27 1.27)) (justify left))
-    )
-    (property "Footprint" "" (id 2) (at 138.43 100.33 0)
+    (property "Value" "8259" (id 1) (at 140.4494 73.66 0)
+      (effects (font (size 1.27 1.27)) (justify left))
+    )
+    (property "Footprint" "Package_DIP:DIP-28_W15.24mm" (id 2) (at 138.43 100.33 0)
       (effects (font (size 1.27 1.27) italic) hide)
     )
@@
     (in_bom yes) (on_board yes) (fields_autoplaced)
     (property "Reference" "U?" (id 0) (at 38.1 88.9 0))
-    (property "Value" "" (id 1) (at 38.1 91.44 0))
+    (property "Value" "74LS21" (id 1) (at 38.1 91.44 0))
     (property "Footprint" "" (id 2) (at 38.1 99.06 0)
       (effects (font (size 1.27 1.27)) hide)
@@
       (effects (font (size 1.27 1.27)) (justify left))
     )
-    (property "Value" "" (id 1) (at 68.5799 69.85 0)
+    (property "Value" ".1uF" (id 1) (at 68.5799 69.85 0)
       (effects (font (size 1.27 1.27)) (justify left))
     )
@@
       (effects (font (size 1.27 1.27)) hide)
     )
-    (property "Value" "" (id 1) (at 138.43 133.35 0))
+    (property "Value" "GND" (id 1) (at 138.43 133.35 0))
     (property "Footprint" "" (id 2) (at 138.43 128.27 0)
       (effects (font (size 1.27 1.27)) hide)

Commit message: test
Connections:
- net A1: now also U1.27 (A0); no longer U0.3 (I3)
- net A2: now also U0.3 (I3); no longer U0.4 (I4)
- net A3: now also U0.4 (I4); no longer U0.5 (I5)
- net at U?.6: now also U0.5 (I5); no longer U0.6 (I6)
- net at U?.8: now also U0.7 (I7); no longer U0.8 (I8)
- net at U?.8: now also U0.6 (I6); no longer U0.7 (I7)
- net IR0: now reaches U1.18 (IR0)
- net COMM: no longer names the net of U0.19 (IO1)
- net COMM: now also U1.1 (~{CS}); no longer U1.27 (A0)
- net DATA: no longer names the net of U0.18 (IO2)
- net DATA: no longer U1.1 (~{CS})
- no-connect marks 11 -> 13
Changed lines of the file:
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@@
   (no_connect (at 83.82 97.79))
   (no_connect (at 83.82 90.17))
+  (no_connect (at 83.82 82.55))
+  (no_connect (at 58.42 97.79))
   (no_connect (at 153.67 102.87))
   (no_connect (at 153.67 105.41))
@@
     (stroke (width 0) (type default) (color 0 0 0 0))
   )
+  (wire (pts (xy 46.99 90.17) (xy 58.42 90.17))
+    (stroke (width 0) (type default) (color 0 0 0 0))
+  )
   (wire (pts (xy 27.94 95.25) (xy 30.48 95.25))
     (stroke (width 0) (type default) (color 0 0 0 0))
   )
-  (wire (pts (xy 48.26 115.57) (xy 48.26 97.79))
-    (stroke (width 0) (type default) (color 0 0 0 0))
-  )
   (wire (pts (xy 27.94 78.74) (xy 30.48 78.74))
     (stroke (width 0) (type default) (color 0 0 0 0))
   )
+  (wire (pts (xy 55.88 85.09) (xy 58.42 85.09))
+    (stroke (width 0) (type default) (color 0 0 0 0))
+  )
   (wire (pts (xy 27.94 83.82) (xy 30.48 83.82))
     (stroke (width 0) (type default) (color 0 0 0 0))
   )
-  (wire (pts (xy 118.11 102.87) (xy 123.19 102.87))
-    (stroke (width 0) (type default) (color 0 0 0 0))
-  )
   (wire (pts (xy 27.94 100.33) (xy 30.48 100.33))
     (stroke (width 0) (type default) (color 0 0 0 0))
@@
     (stroke (width 0) (type default) (color 0 0 0 0))
   )
+  (wire (pts (xy 45.72 82.55) (xy 46.99 82.55))
+    (stroke (width 0) (type default) (color 0 0 0 0))
+  )
+  (wire (pts (xy 120.65 102.87) (xy 123.19 102.87))
+    (stroke (width 0) (type default) (color 0 0 0 0))
+  )
   (wire (pts (xy 119.38 87.63) (xy 123.19 87.63))
     (stroke (width 0) (type default) (color 0 0 0 0))
   )
-  (wire (pts (xy 55.88 85.09) (xy 58.42 85.09))
-    (stroke (width 0) (type default) (color 0 0 0 0))
-  )
-  (wire (pts (xy 83.82 82.55) (xy 87.63 82.55))
+  (wire (pts (xy 83.82 80.01) (xy 100.33 80.01))
     (stroke (width 0) (type default) (color 0 0 0 0))
   )
@@
     (stroke (width 0) (type default) (color 0 0 0 0))
   )
-  (wire (pts (xy 83.82 80.01) (xy 87.63 80.01))
+  (wire (pts (xy 153.67 113.03) (xy 156.21 113.03))
+    (stroke (width 0) (type default) (color 0 0 0 0))
+  )
+  (wire (pts (xy 46.99 82.55) (xy 46.99 90.17))
+    (stroke (width 0) (type default) (color 0 0 0 0))
+  )
+  (wire (pts (xy 163.83 113.03) (xy 167.64 113.03))
+    (stroke (width 0) (type default) (color 0 0 0 0))
+  )
+  (wire (pts (xy 48.26 115.57) (xy 48.26 95.25))
+    (stroke (width 0) (type default) (color 0 0 0 0))
+  )
+  (wire (pts (xy 119.38 80.01) (xy 123.19 80.01))
+    (stroke (width 0) (type default) (color 0 0 0 0))
+  )
+  (wire (pts (xy 46.99 92.71) (xy 58.42 92.71))
+    (stroke (width 0) (type default) (color 0 0 0 0))
+  )
+  (wire (pts (xy 26.67 21.59) (xy 35.56 21.59))
+    (stroke (width 0) (type default) (color 0 0 0 0))
+  )
+  (wire (pts (xy 48.26 95.25) (xy 58.42 95.25))
+    (stroke (width 0) (type default) (color 0 0 0 0))
+  )
+  (wire (pts (xy 27.94 116.84) (xy 30.48 116.84))
+    (stroke (width 0) (type default) (color 0 0 0 0))
+  )
+  (wire (pts (xy 71.12 73.66) (xy 71.12 74.93))
+    (stroke (width 0) (type default) (color 0 0 0 0))
+  )
+  (wire (pts (xy 27.94 86.36) (xy 30.48 86.36))
+    (stroke (width 0) (type default) (color 0 0 0 0))
+  )
+  (wire (pts (xy 46.99 99.06) (xy 46.99 92.71))
+    (stroke (width 0) (type default) (color 0 0 0 0))
+  )
+  (wire (pts (xy 138.43 67.31) (xy 138.43 71.12))
+    (stroke (width 0) (type default) (color 0 0 0 0))
+  )
+  (wire (pts (xy 27.94 111.76) (xy 30.48 111.76))
+    (stroke (width 0) (type default) (color 0 0 0 0))
+  )
+  (wire (pts (xy 55.88 80.01) (xy 58.42 80.01))
+    (stroke (width 0) (type default) (color 0 0 0 0))
+  )
+  (wire (pts (xy 119.38 85.09) (xy 123.19 85.09))
+    (stroke (width 0) (type default) (color 0 0 0 0))
+  )
+  (wire (pts (xy 27.94 114.3) (xy 30.48 114.3))
+    (stroke (width 0) (type default) (color 0 0 0 0))
+  )
+  (wire (pts (xy 119.38 97.79) (xy 123.19 97.79))
+    (stroke (width 0) (type default) (color 0 0 0 0))
+  )
+  (wire (pts (xy 55.88 87.63) (xy 58.42 87.63))
+    (stroke (width 0) (type default) (color 0 0 0 0))
+  )
+  (wire (pts (xy 27.94 97.79) (xy 30.48 97.79))
+    (stroke (width 0) (type default) (color 0 0 0 0))
+  )
+  (wire (pts (xy 119.38 82.55) (xy 123.19 82.55))
+    (stroke (width 0) (type default) (color 0 0 0 0))
+  )
+  (wire (pts (xy 100.33 107.95) (xy 123.19 107.95))
+    (stroke (width 0) (type default) (color 0 0 0 0))
+  )
+  (wire (pts (xy 138.43 71.12) (xy 138.43 72.39))
+    (stroke (width 0) (type default) (color 0 0 0 0))
+  )
+  (wire (pts (xy 100.33 80.01) (xy 100.33 107.95))
+    (stroke (width 0) (type default) (color 0 0 0 0))
+  )
+  (bus (pts (xy 26.67 16.51) (xy 85.09 16.51))
     (stroke (width 0) (type default) (color 0 0 0 0))
   )
@@
     (stroke (width 0) (type default) (color 0 0 0 0))
   )
-  (wire (pts (xy 153.67 113.03) (xy 156.21 113.03))
-    (stroke (width 0) (type default) (color 0 0 0 0))
-  )
-  (wire (pts (xy 163.83 113.03) (xy 167.64 113.03))
-    (stroke (width 0) (type default) (color 0 0 0 0))
-  )
-  (wire (pts (xy 118.11 107.95) (xy 123.19 107.95))
-    (stroke (width 0) (type default) (color 0 0 0 0))
-  )
-  (wire (pts (xy 119.38 80.01) (xy 123.19 80.01))
-    (stroke (width 0) (type default) (color 0 0 0 0))
-  )
-  (wire (pts (xy 46.99 99.06) (xy 46.99 95.25))
-    (stroke (width 0) (type default) (color 0 0 0 0))
-  )
-  (wire (pts (xy 26.67 21.59) (xy 35.56 21.59))
-    (stroke (width 0) (type default) (color 0 0 0 0))
-  )
-  (wire (pts (xy 27.94 116.84) (xy 30.48 116.84))
-    (stroke (width 0) (type default) (color 0 0 0 0))
-  )
-  (wire (pts (xy 71.12 73.66) (xy 71.12 74.93))
-    (stroke (width 0) (type default) (color 0 0 0 0))
-  )
-  (wire (pts (xy 27.94 86.36) (xy 30.48 86.36))
-    (stroke (width 0) (type default) (color 0 0 0 0))
-  )
-  (wire (pts (xy 138.43 67.31) (xy 138.43 71.12))
-    (stroke (width 0) (type default) (color 0 0 0 0))
-  )
-  (wire (pts (xy 27.94 111.76) (xy 30.48 111.76))
-    (stroke (width 0) (type default) (color 0 0 0 0))
-  )
-  (wire (pts (xy 55.88 80.01) (xy 58.42 80.01))
-    (stroke (width 0) (type default) (color 0 0 0 0))
-  )
-  (wire (pts (xy 119.38 85.09) (xy 123.19 85.09))
-    (stroke (width 0) (type default) (color 0 0 0 0))
-  )
-  (wire (pts (xy 27.94 114.3) (xy 30.48 114.3))
-    (stroke (width 0) (type default) (color 0 0 0 0))
-  )
   (wire (pts (xy 45.72 99.06) (xy 46.99 99.06))
     (stroke (width 0) (type default) (color 0 0 0 0))
   )
-  (wire (pts (xy 119.38 97.79) (xy 123.19 97.79))
-    (stroke (width 0) (type default) (color 0 0 0 0))
-  )
-  (wire (pts (xy 55.88 87.63) (xy 58.42 87.63))
-    (stroke (width 0) (type default) (color 0 0 0 0))
-  )
-  (wire (pts (xy 27.94 97.79) (xy 30.48 97.79))
-    (stroke (width 0) (type default) (color 0 0 0 0))
-  )
-  (wire (pts (xy 46.99 82.55) (xy 46.99 92.71))
-    (stroke (width 0) (type default) (color 0 0 0 0))
-  )
-  (wire (pts (xy 55.88 90.17) (xy 58.42 90.17))
-    (stroke (width 0) (type default) (color 0 0 0 0))
-  )
-  (wire (pts (xy 119.38 82.55) (xy 123.19 82.55))
-    (stroke (width 0) (type default) (color 0 0 0 0))
-  )
-  (wire (pts (xy 138.43 71.12) (xy 138.43 72.39))
-    (stroke (width 0) (type default) (color 0 0 0 0))
-  )
-  (bus (pts (xy 26.67 16.51) (xy 85.09 16.51))
-    (stroke (width 0) (type default) (color 0 0 0 0))
-  )
-  (wire (pts (xy 45.72 82.55) (xy 46.99 82.55))
-    (stroke (width 0) (type default) (color 0 0 0 0))
-  )
-  (wire (pts (xy 46.99 95.25) (xy 58.42 95.25))
-    (stroke (width 0) (type default) (color 0 0 0 0))
-  )
   (wire (pts (xy 27.94 119.38) (xy 30.48 119.38))
     (stroke (width 0) (type default) (color 0 0 0 0))
@@
     (stroke (width 0) (type default) (color 0 0 0 0))
   )
-  (wire (pts (xy 46.99 92.71) (xy 58.42 92.71))
-    (stroke (width 0) (type default) (color 0 0 0 0))
-  )
-  (wire (pts (xy 48.26 97.79) (xy 58.42 97.79))
-    (stroke (width 0) (type default) (color 0 0 0 0))
-  )
   (wire (pts (xy 27.94 81.28) (xy 30.48 81.28))
     (stroke (width 0) (type default) (color 0 0 0 0))
@@
     (effects (font (size 1.27 1.27)) (justify left bottom))
   )
-  (label "A2" (at 55.88 87.63 0)
+  (label "A3" (at 55.88 87.63 0)
+    (effects (font (size 1.27 1.27)) (justify left bottom))
+  )
+  (label "A2" (at 55.88 85.09 0)
     (effects (font (size 1.27 1.27)) (justify left bottom))
   )
@@
     (effects (font (size 1.27 1.27)) (justify left bottom))
   )
-  (label "COMM" (at 87.63 80.01 0)
-    (effects (font (size 1.27 1.27)) (justify left bottom))
-  )
   (label "A10" (at 27.94 100.33 0)
     (effects (font (size 1.27 1.27)) (justify left bottom))
   )
-  (label "DATA" (at 87.63 82.55 0)
-    (effects (font (size 1.27 1.27)) (justify left bottom))
-  )
   (label "A14" (at 27.94 116.84 0)
     (effects (font (size 1.27 1.27)) (justify left bottom))
@@
     (effects (font (size 1.27 1.27)) (justify left bottom))
   )
-  (label "DATA" (at 118.11 107.95 0)
-    (effects (font (size 1.27 1.27)) (justify left bottom))
-  )
-  (label "COMM" (at 118.11 102.87 0)
-    (effects (font (size 1.27 1.27)) (justify left bottom))
-  )
-  (label "A3" (at 55.88 90.17 0)
-    (effects (font (size 1.27 1.27)) (justify left bottom))
-  )
   (label "D[0..15]" (at 85.09 16.51 180)
     (effects (font (size 1.27 1.27)) (justify right bottom))
@@
     (effects (font (size 1.27 1.27)) (justify left bottom))
   )
+  (label "A1" (at 120.65 102.87 0)
+    (effects (font (size 1.27 1.27)) (justify left bottom))
+  )
   (label "D3" (at 119.38 87.63 0)
     (effects (font (size 1.27 1.27)) (justify left bottom))
   )
   (label "D6" (at 119.38 95.25 0)
-    (effects (font (size 1.27 1.27)) (justify left bottom))
-  )
-  (label "A1" (at 55.88 85.09 0)
     (effects (font (size 1.27 1.27)) (justify left bottom))
   )
@@
     (effects (font (size 1.27 1.27)) (justify right))
   )
+  (hierarchical_label "IR0" (shape output) (at 153.67 97.79 0)
+    (effects (font (size 1.27 1.27)) (justify left))
+  )
   (hierarchical_label "M{slash}_IO" (shape output) (at 55.88 80.01 180)

Commit message: fixes
Parts:
- removed J?: Conn_01x04_Female, symbol Connector:Conn_01x04_Female
- added J?: (no value), symbol Connector:Conn_01x04_Male
- added R?: (no value), symbol Device:R
- added SW?: (no value), symbol Switch:SW_Push
Connections:
- net GND: now also R?.2
- net VIN: now also SW?.2
- net at U1.25 (IR7): now also J?.4 (Pin_4)
- net at U1.24 (IR6): now also J?.3 (Pin_3)
- net at U1.23 (IR5): now also J?.2 (Pin_2)
- net at U1.22 (IR4): now also J?.1 (Pin_1)
- net IR0: no longer names the net of U1.18 (IR0)
- net IR0: now also R?.1, SW?.1
Changed lines of the file:
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@@
   (junction (at 71.12 73.66) (diameter 0) (color 0 0 0 0)
+  )
+  (junction (at 171.45 97.79) (diameter 0) (color 0 0 0 0)
   )
   (no_connect (at 83.82 92.71))
@@
     (stroke (width 0) (type default) (color 0 0 0 0))
   )
+  (wire (pts (xy 171.45 106.68) (xy 173.99 106.68))
+    (stroke (width 0) (type default) (color 0 0 0 0))
+  )
   (wire (pts (xy 27.94 86.36) (xy 30.48 86.36))
     (stroke (width 0) (type default) (color 0 0 0 0))
@@
     (stroke (width 0) (type default) (color 0 0 0 0))
   )
+  (wire (pts (xy 171.45 97.79) (xy 172.72 97.79))
+    (stroke (width 0) (type default) (color 0 0 0 0))
+  )
   (wire (pts (xy 119.38 85.09) (xy 123.19 85.09))
     (stroke (width 0) (type default) (color 0 0 0 0))
@@
     (stroke (width 0) (type default) (color 0 0 0 0))
   )
+  (wire (pts (xy 171.45 97.79) (xy 171.45 106.68))
+    (stroke (width 0) (type default) (color 0 0 0 0))
+  )
+  (wire (pts (xy 153.67 97.79) (xy 171.45 97.79))
+    (stroke (width 0) (type default) (color 0 0 0 0))
+  )
+  (wire (pts (xy 182.88 97.79) (xy 189.23 97.79))
+    (stroke (width 0) (type default) (color 0 0 0 0))
+  )
   (bus (pts (xy 26.67 16.51) (xy 85.09 16.51))
     (stroke (width 0) (type default) (color 0 0 0 0))
@@
     (effects (font (size 1.27 1.27)) (justify left bottom))
   )
+  (label "VIN" (at 35.56 21.59 180)
+    (effects (font (size 1.27 1.27)) (justify right bottom))
+  )
   (label "D[0..15]" (at 85.09 16.51 180)
     (effects (font (size 1.27 1.27)) (justify right bottom))
@@
   (label "A11" (at 27.94 102.87 0)
     (effects (font (size 1.27 1.27)) (justify left bottom))
+  )
+  (label "VIN" (at 189.23 97.79 180)
+    (effects (font (size 1.27 1.27)) (justify right bottom))
   )
   (label "A1" (at 120.65 102.87 0)
@@
   (hierarchical_label "INT" (shape output) (at 123.19 118.11 180)
     (effects (font (size 1.27 1.27)) (justify right))
-  )
-  (hierarchical_label "IR0" (shape output) (at 153.67 97.79 0)
-    (effects (font (size 1.27 1.27)) (justify left))
   )
   (hierarchical_label "M{slash}_IO" (shape output) (at 55.88 80.01 180)
@@
     (pin "2")
   )
-  (symbol (lib_id "Connector:Conn_01x04_Female") (at 158.75 82.55 0) (unit 1)
-    (in_bom yes) (on_board yes) (fields_autoplaced)
-    (property "Reference" "J?" (id 0) (at 160.02 82.5499 0)
-      (effects (font (size 1.27 1.27)) (justify left))
-    )
-    (property "Value" "Conn_01x04_Female" (id 1) (at 160.02 85.0899 0)
-      (effects (font (size 1.27 1.27)) (justify left))
-    )
-    (property "Footprint" "" (id 2) (at 158.75 82.55 0)
-      (effects (font (size 1.27 1.27)) hide)
-    )
-    (property "Datasheet" "~" (id 3) (at 158.75 82.55 0)
-      (effects (font (size 1.27 1.27)) hide)
-    )
-    (pin "1")
-    (pin "2")
-    (pin "3")
-    (pin "4")
+  (symbol (lib_id "Device:R") (at 177.8 106.68 90) (unit 1)
+    (in_bom yes) (on_board yes) (fields_autoplaced)
+    (property "Reference" "R?" (id 0) (at 177.8 100.33 90))
+    (property "Value" "" (id 1) (at 177.8 102.87 90))
+    (property "Footprint" "" (id 2) (at 177.8 108.458 90)
+      (effects (font (size 1.27 1.27)) hide)
+    )
+    (property "Datasheet" "~" (id 3) (at 177.8 106.68 0)
+      (effects (font (size 1.27 1.27)) hide)
+    )
+    (pin "1")
+    (pin "2")
   )
   (symbol (lib_id "74xx:74LS21") (at 38.1 115.57 0) (unit 2)
@@
     (pin "14")
     (pin "7")
+  )
+  (symbol (lib_id "Connector:Conn_01x04_Male") (at 158.75 85.09 180) (unit 1)
+    (in_bom yes) (on_board yes) (fields_autoplaced)
+    (property "Reference" "J?" (id 0) (at 160.02 82.5499 0)
+      (effects (font (size 1.27 1.27)) (justify right))
+    )
+    (property "Value" "" (id 1) (at 160.02 85.0899 0)
+      (effects (font (size 1.27 1.27)) (justify right))
+    )
+    (property "Footprint" "" (id 2) (at 158.75 85.09 0)
+      (effects (font (size 1.27 1.27)) hide)
+    )
+    (property "Datasheet" "~" (id 3) (at 158.75 85.09 0)
+      (effects (font (size 1.27 1.27)) hide)
+    )
+    (pin "1")
+    (pin "2")
+    (pin "3")
+    (pin "4")
+  )
+  (symbol (lib_id "power:GND") (at 181.61 106.68 90) (unit 1)
+    (in_bom yes) (on_board yes) (fields_autoplaced)
+    (property "Reference" "#PWR?" (id 0) (at 187.96 106.68 0)
+      (effects (font (size 1.27 1.27)) hide)
+    )
+    (property "Value" "" (id 1) (at 185.42 106.6799 90)
+      (effects (font (size 1.27 1.27)) (justify right))
+    )
+    (property "Footprint" "" (id 2) (at 181.61 106.68 0)
+      (effects (font (size 1.27 1.27)) hide)
+    )
+    (property "Datasheet" "" (id 3) (at 181.61 106.68 0)
+      (effects (font (size 1.27 1.27)) hide)
+    )
+    (pin "1")
   )
   (symbol (lib_id "Device:C") (at 134.62 71.12 90) (unit 1)
@@
     (pin "1")
   )
+  (symbol (lib_id "Switch:SW_Push") (at 177.8 97.79 0) (unit 1)
+    (in_bom yes) (on_board yes) (fields_autoplaced)
+    (property "Reference" "SW?" (id 0) (at 177.8 90.17 0))
+    (property "Value" "" (id 1) (at 177.8 92.71 0))
+    (property "Footprint" "" (id 2) (at 177.8 92.71 0)
+      (effects (font (size 1.27 1.27)) hide)
+    )
+    (property "Datasheet" "~" (id 3) (at 177.8 92.71 0)
+      (effects (font (size 1.27 1.27)) hide)
+    )
+    (pin "1")
+    (pin "2")
+  )
   (symbol (lib_id "power:GND") (at 130.81 71.12 180) (unit 1)
