File: 8086proj/8259.kicad_sch (KiCad schematic)
At the start: 11 parts, among them U0 PAL16L8, U1 8259

Commit message: final look
Parts:
- J801: renamed from J?; value (none) -> Conn_01x04_Male
- R802: renamed from R?; value (none) -> 10k
- SW801: renamed from SW?; value (none) -> SW_Push
- gave numbers to parts that had none: 2
- renumbered C0 to C801, C1 to C802, R0 to R801, U0 to U803, U1 to U804
Changed lines of the file:
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@@
   (symbol (lib_id "74xx:74LS21") (at 38.1 82.55 0) (unit 1)
     (in_bom yes) (on_board yes) (fields_autoplaced)
-    (property "Reference" "U?" (id 0) (at 38.1 72.39 0))
+    (property "Reference" "U801" (id 0) (at 38.1 72.39 0))
     (property "Value" "74LS21" (id 1) (at 38.1 74.93 0))
     (property "Footprint" "" (id 2) (at 38.1 82.55 0)
@@
   (symbol (lib_id "Device:R") (at 160.02 113.03 90) (unit 1)
     (in_bom yes) (on_board yes) (fields_autoplaced)
-    (property "Reference" "R0" (id 0) (at 160.02 106.68 90))
+    (property "Reference" "R801" (id 0) (at 160.02 106.68 90))
     (property "Value" "10k" (id 1) (at 160.02 109.22 90))
     (property "Footprint" "" (id 2) (at 160.02 114.808 90)
@@
   (symbol (lib_id "Device:R") (at 177.8 106.68 90) (unit 1)
     (in_bom yes) (on_board yes) (fields_autoplaced)
-    (property "Reference" "R?" (id 0) (at 177.8 100.33 90))
-    (property "Value" "" (id 1) (at 177.8 102.87 90))
+    (property "Reference" "R802" (id 0) (at 177.8 100.33 90))
+    (property "Value" "10k" (id 1) (at 177.8 102.87 90))
     (property "Footprint" "" (id 2) (at 177.8 108.458 90)
       (effects (font (size 1.27 1.27)) hide)
@@
   (symbol (lib_id "74xx:74LS21") (at 38.1 115.57 0) (unit 2)
     (in_bom yes) (on_board yes) (fields_autoplaced)
-    (property "Reference" "U?" (id 0) (at 38.1 105.41 0))
+    (property "Reference" "U802" (id 0) (at 38.1 105.41 0))
     (property "Value" "74LS21" (id 1) (at 38.1 107.95 0))
     (property "Footprint" "" (id 2) (at 38.1 115.57 0)
@@
   (symbol (lib_id "Connector:Conn_01x04_Male") (at 158.75 85.09 180) (unit 1)
     (in_bom yes) (on_board yes) (fields_autoplaced)
-    (property "Reference" "J?" (id 0) (at 160.02 82.5499 0)
+    (property "Reference" "J801" (id 0) (at 160.02 82.5499 0)
       (effects (font (size 1.27 1.27)) (justify right))
     )
-    (property "Value" "" (id 1) (at 160.02 85.0899 0)
+    (property "Value" "Conn_01x04_Male" (id 1) (at 160.02 85.0899 0)
       (effects (font (size 1.27 1.27)) (justify right))
     )
@@
   (symbol (lib_id "power:GND") (at 181.61 106.68 90) (unit 1)
     (in_bom yes) (on_board yes) (fields_autoplaced)
-    (property "Reference" "#PWR?" (id 0) (at 187.96 106.68 0)
-      (effects (font (size 1.27 1.27)) hide)
-    )
-    (property "Value" "" (id 1) (at 185.42 106.6799 90)
+    (property "Reference" "#PWR0805" (id 0) (at 187.96 106.68 0)
+      (effects (font (size 1.27 1.27)) hide)
+    )
+    (property "Value" "GND" (id 1) (at 185.42 106.6799 90)
       (effects (font (size 1.27 1.27)) (justify right))
     )
@@
   (symbol (lib_id "Device:C") (at 134.62 71.12 90) (unit 1)
     (in_bom yes) (on_board yes)
-    (property "Reference" "C1" (id 0) (at 133.3499 67.31 0)
+    (property "Reference" "C802" (id 0) (at 133.3499 67.31 0)
       (effects (font (size 1.27 1.27)) (justify left))
     )
@@
   (symbol (lib_id "Logic_Programmable:PAL16L8") (at 71.12 92.71 0) (unit 1)
     (in_bom yes) (on_board yes) (fields_autoplaced)
-    (property "Reference" "U0" (id 0) (at 73.1394 73.66 0)
+    (property "Reference" "U803" (id 0) (at 73.1394 73.66 0)
       (effects (font (size 1.27 1.27)) (justify left))
     )
@@
   (symbol (lib_id "Interface:8259") (at 138.43 100.33 0) (unit 1)
     (in_bom yes) (on_board yes) (fields_autoplaced)
-    (property "Reference" "U1" (id 0) (at 140.4494 71.12 0)
+    (property "Reference" "U804" (id 0) (at 140.4494 71.12 0)
       (effects (font (size 1.27 1.27)) (justify left))
     )
@@
   (symbol (lib_id "74xx:74LS21") (at 38.1 99.06 0) (unit 2)
     (in_bom yes) (on_board yes) (fields_autoplaced)
-    (property "Reference" "U?" (id 0) (at 38.1 88.9 0))
+    (property "Reference" "U801" (id 0) (at 38.1 88.9 0))
     (property "Value" "74LS21" (id 1) (at 38.1 91.44 0))
     (property "Footprint" "" (id 2) (at 38.1 99.06 0)
@@
   (symbol (lib_id "Device:C") (at 67.31 73.66 90) (unit 1)
     (in_bom yes) (on_board yes)
-    (property "Reference" "C0" (id 0) (at 66.0399 69.85 0)
+    (property "Reference" "C801" (id 0) (at 66.0399 69.85 0)
       (effects (font (size 1.27 1.27)) (justify left))
     )
@@
   (symbol (lib_id "power:GND") (at 138.43 128.27 0) (unit 1)
     (in_bom yes) (on_board yes) (fields_autoplaced)
-    (property "Reference" "#PWR0133" (id 0) (at 138.43 134.62 0)
+    (property "Reference" "#PWR0804" (id 0) (at 138.43 134.62 0)
       (effects (font (size 1.27 1.27)) hide)
     )
@@
   (symbol (lib_id "Switch:SW_Push") (at 177.8 97.79 0) (unit 1)
     (in_bom yes) (on_board yes) (fields_autoplaced)
-    (property "Reference" "SW?" (id 0) (at 177.8 90.17 0))
-    (property "Value" "" (id 1) (at 177.8 92.71 0))
+    (property "Reference" "SW801" (id 0) (at 177.8 90.17 0))
+    (property "Value" "SW_Push" (id 1) (at 177.8 92.71 0))
     (property "Footprint" "" (id 2) (at 177.8 92.71 0)
       (effects (font (size 1.27 1.27)) hide)
@@
   (symbol (lib_id "power:GND") (at 130.81 71.12 180) (unit 1)
     (in_bom yes) (on_board yes) (fields_autoplaced)
-    (property "Reference" "#PWR0134" (id 0) (at 130.81 64.77 0)
+    (property "Reference" "#PWR0803" (id 0) (at 130.81 64.77 0)
       (effects (font (size 1.27 1.27)) hide)
     )
@@
   (symbol (lib_id "power:GND") (at 71.12 107.95 0) (unit 1)
     (in_bom yes) (on_board yes) (fields_autoplaced)
-    (property "Reference" "#PWR0132" (id 0) (at 71.12 114.3 0)
+    (property "Reference" "#PWR0802" (id 0) (at 71.12 114.3 0)
       (effects (font (size 1.27 1.27)) hide)
     )
@@
   (symbol (lib_id "power:GND") (at 63.5 73.66 180) (unit 1)
     (in_bom yes) (on_board yes) (fields_autoplaced)
-    (property "Reference" "#PWR0131" (id 0) (at 63.5 67.31 0)
-      (effects (font (size 1.27 1.27)) hide)
-    )
+    (property "Reference" "#PWR0801" (id 0) (at 63.5 67.31 0)
+      (effects (font (size 1.27 1.27)) hide)
+    )

Commit message: footprints
Parts:
- C801, C802: footprint (none) -> Capacitor_SMD:CP_Elec_3x5.3
- J801: footprint (none) -> Connector_PinHeader_1.00mm:PinHeader_1x04_P1.00mm_Vertical
Changed lines of the file:
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@@
       (effects (font (size 1.27 1.27)) (justify right))
     )
-    (property "Footprint" "" (id 2) (at 158.75 85.09 0)
+    (property "Footprint" "Connector_PinHeader_1.00mm:PinHeader_1x04_P1.00mm_Vertical" (id 2) (at 158.75 85.09 0)
       (effects (font (size 1.27 1.27)) hide)
     )
@@
       (effects (font (size 1.27 1.27)) (justify left))
     )
-    (property "Footprint" "" (id 2) (at 138.43 70.1548 0)
+    (property "Footprint" "Capacitor_SMD:CP_Elec_3x5.3" (id 2) (at 138.43 70.1548 0)
       (effects (font (size 1.27 1.27)) hide)
     )
@@
       (effects (font (size 1.27 1.27)) (justify left))
     )
-    (property "Footprint" "" (id 2) (at 71.12 72.6948 0)
+    (property "Footprint" "Capacitor_SMD:CP_Elec_3x5.3" (id 2) (at 71.12 72.6948 0)
       (effects (font (size 1.27 1.27)) hide)
     )

Commit message: pcb
Parts:
- R801, R802: footprint (none) -> Resistor_SMD:R_0201_0603Metric
- SW801: footprint (none) -> Button_Switch_Keyboard:SW_Cherry_MX_1.00u_PCB
- U803: footprint (none) -> Package_DIP:DIP-20_W7.62mm
Changed lines of the file:
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@@
     (property "Reference" "R801" (id 0) (at 160.02 106.68 90))
     (property "Value" "10k" (id 1) (at 160.02 109.22 90))
-    (property "Footprint" "" (id 2) (at 160.02 114.808 90)
+    (property "Footprint" "Resistor_SMD:R_0201_0603Metric" (id 2) (at 160.02 114.808 90)
       (effects (font (size 1.27 1.27)) hide)
     )
@@
     (property "Reference" "R802" (id 0) (at 177.8 100.33 90))
     (property "Value" "10k" (id 1) (at 177.8 102.87 90))
-    (property "Footprint" "" (id 2) (at 177.8 108.458 90)
+    (property "Footprint" "Resistor_SMD:R_0201_0603Metric" (id 2) (at 177.8 108.458 90)
       (effects (font (size 1.27 1.27)) hide)
     )
@@
       (effects (font (size 1.27 1.27)) (justify left))
     )
-    (property "Footprint" "" (id 2) (at 71.12 92.71 0)
+    (property "Footprint" "Package_DIP:DIP-20_W7.62mm" (id 2) (at 71.12 92.71 0)
       (effects (font (size 1.27 1.27)) hide)
     )
@@
     (property "Reference" "SW801" (id 0) (at 177.8 90.17 0))
     (property "Value" "SW_Push" (id 1) (at 177.8 92.71 0))
-    (property "Footprint" "" (id 2) (at 177.8 92.71 0)
-      (effects (font (size 1.27 1.27)) hide)
-    )
+    (property "Footprint" "Button_Switch_Keyboard:SW_Cherry_MX_1.00u_PCB" (id 2) (at 177.8 92.71 0)
+      (effects (font (size 1.27 1.27)) hide)
+    )

Commit message: pcb
Parts:
- U801, U802: footprint (none) -> Package_DIP:DIP-14_W10.16mm
Changed lines of the file:
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@@
     (property "Reference" "U801" (id 0) (at 38.1 72.39 0))
     (property "Value" "74LS21" (id 1) (at 38.1 74.93 0))
-    (property "Footprint" "" (id 2) (at 38.1 82.55 0)
+    (property "Footprint" "Package_DIP:DIP-14_W10.16mm" (id 2) (at 38.1 82.55 0)
       (effects (font (size 1.27 1.27)) hide)
     )
@@
     (property "Reference" "U802" (id 0) (at 38.1 105.41 0))
     (property "Value" "74LS21" (id 1) (at 38.1 107.95 0))
-    (property "Footprint" "" (id 2) (at 38.1 115.57 0)
+    (property "Footprint" "Package_DIP:DIP-14_W10.16mm" (id 2) (at 38.1 115.57 0)
       (effects (font (size 1.27 1.27)) hide)
     )
@@
     (property "Reference" "U801" (id 0) (at 38.1 88.9 0))
     (property "Value" "74LS21" (id 1) (at 38.1 91.44 0))
-    (property "Footprint" "" (id 2) (at 38.1 99.06 0)
-      (effects (font (size 1.27 1.27)) hide)
-    )
+    (property "Footprint" "Package_DIP:DIP-14_W10.16mm" (id 2) (at 38.1 99.06 0)
+      (effects (font (size 1.27 1.27)) hide)
+    )
