File: 8086proj/8259.kicad_sch (KiCad schematic)
At the start: 10 parts, among them J801 Conn_01x04_Male, SW801 SW_Push, U801 74LS21, U802 74LS21, U803 PAL16L8, U804 8259

Commit message: pcb update
Changed lines of the file:
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@@
+    (stroke (width 0) (type default) (color 0 0 0 0))
+  )
+  (wire (pts (xy 71.12 109.22) (xy 71.12 107.95))
     (stroke (width 0) (type default) (color 0 0 0 0))
   )
@@
     (pin "1")
   )
-  (symbol (lib_id "power:GND") (at 71.12 107.95 0) (unit 1)
-    (in_bom yes) (on_board yes) (fields_autoplaced)
-    (property "Reference" "#PWR0802" (id 0) (at 71.12 114.3 0)
-      (effects (font (size 1.27 1.27)) hide)
-    )
-    (property "Value" "GND" (id 1) (at 71.12 113.03 0))
-    (property "Footprint" "" (id 2) (at 71.12 107.95 0)
-      (effects (font (size 1.27 1.27)) hide)
-    )
-    (property "Datasheet" "" (id 3) (at 71.12 107.95 0)
-      (effects (font (size 1.27 1.27)) hide)
-    )
+  (symbol (lib_id "power:GND") (at 71.12 109.22 0) (unit 1)
+    (in_bom yes) (on_board yes) (fields_autoplaced)
+    (property "Reference" "#PWR0802" (id 0) (at 71.12 115.57 0)
+      (effects (font (size 1.27 1.27)) hide)
+    )
+    (property "Value" "GND" (id 1) (at 71.12 114.3 0))
+    (property "Footprint" "" (id 2) (at 71.12 109.22 0)
+      (effects (font (size 1.27 1.27)) hide)
+    )
+    (property "Datasheet" "" (id 3) (at 71.12 109.22 0)
+      (effects (font (size 1.27 1.27)) hide)
+    )
