File: 8086proj/74374.kicad_sch (KiCad schematic)
At the start: 10 parts

Commit message: fixes
Parts:
- SW?: value (none) -> SW_DIP_x08
- U?: value (none) -> 74LS244
- U? (x2): value (none) -> 74LS04
Connections:
- net GND: no longer U?.19 (OEb)
- net _CS: now also U?.19 (OEb)
- net D3: now reaches U?.12 (O3a)
- net D2: now reaches U?.14 (O2a)
- net D1: now reaches U?.16 (O1a)
- net D0: now reaches U?.18 (O0a)
- net D7: now reaches U?.3 (O3b)
- net D6: now reaches U?.5 (O2b)
- net D5: now reaches U?.7 (O1b)
- net D4: now reaches U?.9 (O0b)
Changed lines of the file:
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@@
   (junction (at 133.35 91.44) (diameter 0) (color 0 0 0 0)
   )
-  (junction (at 161.29 123.19) (diameter 0) (color 0 0 0 0)
-  )
   (junction (at 133.35 99.06) (diameter 0) (color 0 0 0 0)
+  )
+  (junction (at 147.32 111.76) (diameter 0) (color 0 0 0 0)
   )
   (junction (at 133.35 96.52) (diameter 0) (color 0 0 0 0)
@@
     (stroke (width 0) (type default) (color 0 0 0 0))
   )
+  (wire (pts (xy 147.32 111.76) (xy 147.32 114.3))
+    (stroke (width 0) (type default) (color 0 0 0 0))
+  )
   (wire (pts (xy 100.33 78.74) (xy 100.33 82.55))
     (stroke (width 0) (type default) (color 0 0 0 0))
@@
     (stroke (width 0) (type default) (color 0 0 0 0))
   )
+  (wire (pts (xy 147.32 114.3) (xy 148.59 114.3))
+    (stroke (width 0) (type default) (color 0 0 0 0))
+  )
   (wire (pts (xy 55.88 133.35) (xy 58.42 133.35))
     (stroke (width 0) (type default) (color 0 0 0 0))
   )
-  (wire (pts (xy 161.29 121.92) (xy 161.29 123.19))
-    (stroke (width 0) (type default) (color 0 0 0 0))
-  )
   (wire (pts (xy 133.35 88.9) (xy 133.35 91.44))
     (stroke (width 0) (type default) (color 0 0 0 0))
@@
     (stroke (width 0) (type default) (color 0 0 0 0))
   )
-  (wire (pts (xy 148.59 114.3) (xy 147.32 114.3))
-    (stroke (width 0) (type default) (color 0 0 0 0))
-  )
   (wire (pts (xy 161.29 76.2) (xy 161.29 80.01))
     (stroke (width 0) (type default) (color 0 0 0 0))
@@
     (stroke (width 0) (type default) (color 0 0 0 0))
   )
+  (wire (pts (xy 147.32 111.76) (xy 148.59 111.76))
+    (stroke (width 0) (type default) (color 0 0 0 0))
+  )
   (wire (pts (xy 74.93 101.6) (xy 87.63 101.6))
     (stroke (width 0) (type default) (color 0 0 0 0))
@@
     (stroke (width 0) (type default) (color 0 0 0 0))
   )
-  (wire (pts (xy 147.32 114.3) (xy 147.32 123.19))
-    (stroke (width 0) (type default) (color 0 0 0 0))
-  )
   (wire (pts (xy 48.26 90.17) (xy 48.26 95.25))
     (stroke (width 0) (type default) (color 0 0 0 0))
@@
     (stroke (width 0) (type default) (color 0 0 0 0))
   )
-  (wire (pts (xy 147.32 123.19) (xy 161.29 123.19))
-    (stroke (width 0) (type default) (color 0 0 0 0))
-  )
   (wire (pts (xy 48.26 102.87) (xy 48.26 97.79))
     (stroke (width 0) (type default) (color 0 0 0 0))
   )
-  (wire (pts (xy 144.78 111.76) (xy 148.59 111.76))
+  (wire (pts (xy 144.78 111.76) (xy 147.32 111.76))
     (stroke (width 0) (type default) (color 0 0 0 0))
   )
@@
     (stroke (width 0) (type default) (color 0 0 0 0))
   )
-  (wire (pts (xy 161.29 123.19) (xy 161.29 124.46))
-    (stroke (width 0) (type default) (color 0 0 0 0))
-  )
   (wire (pts (xy 55.88 128.27) (xy 58.42 128.27))
     (stroke (width 0) (type default) (color 0 0 0 0))
@@
     (stroke (width 0) (type default) (color 0 0 0 0))
   )
+  (label "D6" (at 177.8 104.14 180)
+    (effects (font (size 1.27 1.27)) (justify right bottom))
+  )
   (label "A1" (at 83.82 91.44 0)
     (effects (font (size 1.27 1.27)) (justify left bottom))
   )
+  (label "D4" (at 177.8 99.06 180)
+    (effects (font (size 1.27 1.27)) (justify right bottom))
+  )
   (label "A15" (at 55.88 135.89 0)
     (effects (font (size 1.27 1.27)) (justify left bottom))
@@
     (effects (font (size 1.27 1.27)) (justify left bottom))
   )
+  (label "VIN" (at 40.64 24.13 180)
+    (effects (font (size 1.27 1.27)) (justify right bottom))
+  )
   (label "_CS" (at 144.78 111.76 0)
     (effects (font (size 1.27 1.27)) (justify left bottom))
@@
     (effects (font (size 1.27 1.27)) (justify left bottom))
   )
+  (label "D1" (at 177.8 91.44 180)
+    (effects (font (size 1.27 1.27)) (justify right bottom))
+  )
   (label "A8" (at 55.88 111.76 0)
     (effects (font (size 1.27 1.27)) (justify left bottom))
@@
     (effects (font (size 1.27 1.27)) (justify left bottom))
   )
+  (label "D5" (at 177.8 101.6 180)
+    (effects (font (size 1.27 1.27)) (justify right bottom))
+  )
+  (label "D0" (at 177.8 88.9 180)
+    (effects (font (size 1.27 1.27)) (justify right bottom))
+  )
+  (label "D3" (at 177.8 96.52 180)
+    (effects (font (size 1.27 1.27)) (justify right bottom))
+  )
   (label "VIN" (at 100.33 78.74 270)
     (effects (font (size 1.27 1.27)) (justify right bottom))
   )
+  (label "D2" (at 177.8 93.98 180)
+    (effects (font (size 1.27 1.27)) (justify right bottom))
+  )
   (label "D[0..15]" (at 90.17 19.05 180)
     (effects (font (size 1.27 1.27)) (justify right bottom))
   )
   (label "A[0..19]" (at 71.12 21.59 180)
+    (effects (font (size 1.27 1.27)) (justify right bottom))
+  )
+  (label "D7" (at 177.8 106.68 180)
     (effects (font (size 1.27 1.27)) (justify right bottom))
   )
@@
     (in_bom yes) (on_board yes) (fields_autoplaced)
     (property "Reference" "SW?" (id 0) (at 140.97 81.28 0))
-    (property "Value" "" (id 1) (at 140.97 83.82 0))
+    (property "Value" "SW_DIP_x08" (id 1) (at 140.97 83.82 0))
     (property "Footprint" "" (id 2) (at 140.97 99.06 0)
       (effects (font (size 1.27 1.27)) hide)
@@
       (effects (font (size 1.27 1.27)) (justify left))
     )
-    (property "Value" "" (id 1) (at 163.3094 83.82 0)
+    (property "Value" "74LS244" (id 1) (at 163.3094 83.82 0)
       (effects (font (size 1.27 1.27)) (justify left))
     )
@@
     (pin "9")
   )
-  (symbol (lib_id "power:GND") (at 161.29 124.46 0) (unit 1)
-    (in_bom yes) (on_board yes) (fields_autoplaced)
-    (property "Reference" "#PWR?" (id 0) (at 161.29 130.81 0)
-      (effects (font (size 1.27 1.27)) hide)
-    )
-    (property "Value" "" (id 1) (at 161.29 129.54 0))
-    (property "Footprint" "" (id 2) (at 161.29 124.46 0)
-      (effects (font (size 1.27 1.27)) hide)
-    )
-    (property "Datasheet" "" (id 3) (at 161.29 124.46 0)
+  (symbol (lib_id "power:GND") (at 161.29 121.92 0) (unit 1)
+    (in_bom yes) (on_board yes) (fields_autoplaced)
+    (property "Reference" "#PWR?" (id 0) (at 161.29 128.27 0)
+      (effects (font (size 1.27 1.27)) hide)
+    )
+    (property "Value" "GND" (id 1) (at 161.29 127 0))
+    (property "Footprint" "" (id 2) (at 161.29 121.92 0)
+      (effects (font (size 1.27 1.27)) hide)
+    )
+    (property "Datasheet" "" (id 3) (at 161.29 121.92 0)
       (effects (font (size 1.27 1.27)) hide)
     )
@@
     (in_bom yes) (on_board yes) (fields_autoplaced)
     (property "Reference" "U?" (id 0) (at 39.37 81.28 0))
-    (property "Value" "" (id 1) (at 39.37 83.82 0))
+    (property "Value" "74LS04" (id 1) (at 39.37 83.82 0))
     (property "Footprint" "" (id 2) (at 39.37 90.17 0)
       (effects (font (size 1.27 1.27)) hide)
@@
     (in_bom yes) (on_board yes) (fields_autoplaced)
     (property "Reference" "U?" (id 0) (at 39.37 93.98 0))
-    (property "Value" "" (id 1) (at 39.37 96.52 0))
+    (property "Value" "74LS04" (id 1) (at 39.37 96.52 0))
     (property "Footprint" "" (id 2) (at 39.37 102.87 0)
       (effects (font (size 1.27 1.27)) hide)

Commit message: final look
Parts:
- gave numbers to parts that had none: 10
Changed lines of the file:
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@@
   (symbol (lib_id "power:GND") (at 153.67 80.01 180) (unit 1)
     (in_bom yes) (on_board yes) (fields_autoplaced)
-    (property "Reference" "#PWR?" (id 0) (at 153.67 73.66 0)
+    (property "Reference" "#PWR01403" (id 0) (at 153.67 73.66 0)
       (effects (font (size 1.27 1.27)) hide)
     )
@@
   (symbol (lib_id "Switch:SW_DIP_x08") (at 140.97 99.06 0) (unit 1)
     (in_bom yes) (on_board yes) (fields_autoplaced)
-    (property "Reference" "SW?" (id 0) (at 140.97 81.28 0))
+    (property "Reference" "SW1401" (id 0) (at 140.97 81.28 0))
     (property "Value" "SW_DIP_x08" (id 1) (at 140.97 83.82 0))
     (property "Footprint" "" (id 2) (at 140.97 99.06 0)
@@
   (symbol (lib_id "74xx:74LS244") (at 161.29 101.6 0) (unit 1)
     (in_bom yes) (on_board yes) (fields_autoplaced)
-    (property "Reference" "U?" (id 0) (at 163.3094 81.28 0)
+    (property "Reference" "U1405" (id 0) (at 163.3094 81.28 0)
       (effects (font (size 1.27 1.27)) (justify left))
     )
@@
   (symbol (lib_id "power:GND") (at 161.29 121.92 0) (unit 1)
     (in_bom yes) (on_board yes) (fields_autoplaced)
-    (property "Reference" "#PWR?" (id 0) (at 161.29 128.27 0)
+    (property "Reference" "#PWR01404" (id 0) (at 161.29 128.27 0)
       (effects (font (size 1.27 1.27)) hide)
     )
@@
   (symbol (lib_id "power:GND") (at 92.71 82.55 180) (unit 1)
     (in_bom yes) (on_board yes) (fields_autoplaced)
-    (property "Reference" "#PWR?" (id 0) (at 92.71 76.2 0)
+    (property "Reference" "#PWR01401" (id 0) (at 92.71 76.2 0)
       (effects (font (size 1.27 1.27)) hide)
     )
@@
   (symbol (lib_id "Device:C") (at 157.48 80.01 90) (unit 1)
     (in_bom yes) (on_board yes)
-    (property "Reference" "C?" (id 0) (at 156.2099 76.2 0)
+    (property "Reference" "C1402" (id 0) (at 156.2099 76.2 0)
       (effects (font (size 1.27 1.27)) (justify left))
     )
@@
   (symbol (lib_id "74xx:74LS04") (at 39.37 90.17 0) (unit 1)
     (in_bom yes) (on_board yes) (fields_autoplaced)
-    (property "Reference" "U?" (id 0) (at 39.37 81.28 0))
+    (property "Reference" "U1401" (id 0) (at 39.37 81.28 0))
     (property "Value" "74LS04" (id 1) (at 39.37 83.82 0))
     (property "Footprint" "" (id 2) (at 39.37 90.17 0)
@@
   (symbol (lib_id "power:GND") (at 100.33 116.84 0) (unit 1)
     (in_bom yes) (on_board yes) (fields_autoplaced)
-    (property "Reference" "#PWR?" (id 0) (at 100.33 123.19 0)
+    (property "Reference" "#PWR01402" (id 0) (at 100.33 123.19 0)
       (effects (font (size 1.27 1.27)) hide)
     )
@@
   (symbol (lib_id "74xx:74LS21") (at 66.04 99.06 0) (unit 1)
     (in_bom yes) (on_board yes) (fields_autoplaced)
-    (property "Reference" "U?" (id 0) (at 66.04 88.9 0))
+    (property "Reference" "U1003" (id 0) (at 66.04 88.9 0))
     (property "Value" "74LS21" (id 1) (at 66.04 91.44 0))
     (property "Footprint" "" (id 2) (at 66.04 99.06 0)
@@
   (symbol (lib_id "Logic_Programmable:PAL16L8") (at 100.33 101.6 0) (unit 1)
     (in_bom yes) (on_board yes) (fields_autoplaced)
-    (property "Reference" "U?" (id 0) (at 102.3494 82.55 0)
+    (property "Reference" "U1404" (id 0) (at 102.3494 82.55 0)
       (effects (font (size 1.27 1.27)) (justify left))
     )
@@
   (symbol (lib_id "74xx:74LS04") (at 39.37 102.87 0) (unit 2)
     (in_bom yes) (on_board yes) (fields_autoplaced)
-    (property "Reference" "U?" (id 0) (at 39.37 93.98 0))
+    (property "Reference" "U1001" (id 0) (at 39.37 93.98 0))
     (property "Value" "74LS04" (id 1) (at 39.37 96.52 0))
     (property "Footprint" "" (id 2) (at 39.37 102.87 0)
@@
   (symbol (lib_id "Device:C") (at 96.52 82.55 90) (unit 1)
     (in_bom yes) (on_board yes)
-    (property "Reference" "C?" (id 0) (at 95.2499 78.74 0)
+    (property "Reference" "C1401" (id 0) (at 95.2499 78.74 0)
       (effects (font (size 1.27 1.27)) (justify left))
     )
@@
   (symbol (lib_id "74xx:74LS21") (at 66.04 132.08 0) (unit 2)
     (in_bom yes) (on_board yes) (fields_autoplaced)
-    (property "Reference" "U?" (id 0) (at 66.04 121.92 0))
+    (property "Reference" "U1403" (id 0) (at 66.04 121.92 0))
     (property "Value" "74LS21" (id 1) (at 66.04 124.46 0))
     (property "Footprint" "" (id 2) (at 66.04 132.08 0)
@@
   (symbol (lib_id "74xx:74LS21") (at 66.04 115.57 0) (unit 2)
     (in_bom yes) (on_board yes) (fields_autoplaced)
-    (property "Reference" "U?" (id 0) (at 66.04 105.41 0))
+    (property "Reference" "U1402" (id 0) (at 66.04 105.41 0))
     (property "Value" "74LS21" (id 1) (at 66.04 107.95 0))
     (property "Footprint" "" (id 2) (at 66.04 115.57 0)

Commit message: footprints
Parts:
- C1401, C1402: footprint (none) -> Capacitor_SMD:CP_Elec_3x5.3
Changed lines of the file:
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@@
       (effects (font (size 1.27 1.27)) (justify left))
     )
-    (property "Footprint" "" (id 2) (at 161.29 79.0448 0)
+    (property "Footprint" "Capacitor_SMD:CP_Elec_3x5.3" (id 2) (at 161.29 79.0448 0)
       (effects (font (size 1.27 1.27)) hide)
     )
@@
       (effects (font (size 1.27 1.27)) (justify left))
     )
-    (property "Footprint" "" (id 2) (at 100.33 81.5848 0)
+    (property "Footprint" "Capacitor_SMD:CP_Elec_3x5.3" (id 2) (at 100.33 81.5848 0)
       (effects (font (size 1.27 1.27)) hide)
     )

Commit message: pcb
Parts:
- SW1401: footprint (none) -> Button_Switch_SMD:SW_DIP_SPSTx08_Slide_6.7x21.88mm_W6.73mm_P2.54mm_LowProfile_JPin
- U1404: footprint (none) -> Package_DIP:DIP-20_W7.62mm
Changed lines of the file:
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@@
     (property "Reference" "SW1401" (id 0) (at 140.97 81.28 0))
     (property "Value" "SW_DIP_x08" (id 1) (at 140.97 83.82 0))
-    (property "Footprint" "" (id 2) (at 140.97 99.06 0)
+    (property "Footprint" "Button_Switch_SMD:SW_DIP_SPSTx08_Slide_6.7x21.88mm_W6.73mm_P2.54mm_LowProfile_JPin" (id 2) (at 140.97 99.06 0)
       (effects (font (size 1.27 1.27)) hide)
     )
@@
       (effects (font (size 1.27 1.27)) (justify left))
     )
-    (property "Footprint" "" (id 2) (at 100.33 101.6 0)
+    (property "Footprint" "Package_DIP:DIP-20_W7.62mm" (id 2) (at 100.33 101.6 0)
       (effects (font (size 1.27 1.27)) hide)
     )

Commit message: pcb
Parts:
- U1001, U1003, U1401, U1402, U1403, U1405: footprint (none) -> Package_DIP:DIP-14_W10.16mm
Changed lines of the file:
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@@
       (effects (font (size 1.27 1.27)) (justify left))
     )
-    (property "Footprint" "" (id 2) (at 161.29 101.6 0)
+    (property "Footprint" "Package_DIP:DIP-14_W10.16mm" (id 2) (at 161.29 101.6 0)
       (effects (font (size 1.27 1.27)) hide)
     )
@@
     (property "Reference" "U1401" (id 0) (at 39.37 81.28 0))
     (property "Value" "74LS04" (id 1) (at 39.37 83.82 0))
-    (property "Footprint" "" (id 2) (at 39.37 90.17 0)
+    (property "Footprint" "Package_DIP:DIP-14_W10.16mm" (id 2) (at 39.37 90.17 0)
       (effects (font (size 1.27 1.27)) hide)
     )
@@
     (property "Reference" "U1003" (id 0) (at 66.04 88.9 0))
     (property "Value" "74LS21" (id 1) (at 66.04 91.44 0))
-    (property "Footprint" "" (id 2) (at 66.04 99.06 0)
+    (property "Footprint" "Package_DIP:DIP-14_W10.16mm" (id 2) (at 66.04 99.06 0)
       (effects (font (size 1.27 1.27)) hide)
     )
@@
     (property "Reference" "U1001" (id 0) (at 39.37 93.98 0))
     (property "Value" "74LS04" (id 1) (at 39.37 96.52 0))
-    (property "Footprint" "" (id 2) (at 39.37 102.87 0)
+    (property "Footprint" "Package_DIP:DIP-14_W10.16mm" (id 2) (at 39.37 102.87 0)
       (effects (font (size 1.27 1.27)) hide)
     )
@@
     (property "Reference" "U1403" (id 0) (at 66.04 121.92 0))
     (property "Value" "74LS21" (id 1) (at 66.04 124.46 0))
-    (property "Footprint" "" (id 2) (at 66.04 132.08 0)
+    (property "Footprint" "Package_DIP:DIP-14_W10.16mm" (id 2) (at 66.04 132.08 0)
       (effects (font (size 1.27 1.27)) hide)
     )
@@
     (property "Reference" "U1402" (id 0) (at 66.04 105.41 0))
     (property "Value" "74LS21" (id 1) (at 66.04 107.95 0))
-    (property "Footprint" "" (id 2) (at 66.04 115.57 0)
-      (effects (font (size 1.27 1.27)) hide)
-    )
+    (property "Footprint" "Package_DIP:DIP-14_W10.16mm" (id 2) (at 66.04 115.57 0)
+      (effects (font (size 1.27 1.27)) hide)
+    )

Commit message: pcb update
Parts:
- U1405: footprint Package_DIP:DIP-14_W10.16mm -> (none)
Changed lines of the file:
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@@
       (effects (font (size 1.27 1.27)) (justify left))
     )
-    (property "Footprint" "Package_DIP:DIP-14_W10.16mm" (id 2) (at 161.29 101.6 0)
+    (property "Footprint" "" (id 2) (at 161.29 101.6 0)
       (effects (font (size 1.27 1.27)) hide)
     )

Commit message: pcb edit
Parts:
- U1405: footprint (none) -> Package_DIP:DIP-20_W7.62mm
Changed lines of the file:
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@@
       (effects (font (size 1.27 1.27)) (justify left))
     )
-    (property "Footprint" "" (id 2) (at 161.29 101.6 0)
+    (property "Footprint" "Package_DIP:DIP-20_W7.62mm" (id 2) (at 161.29 101.6 0)
       (effects (font (size 1.27 1.27)) hide)
     )
