File: 8086proj/8279.kicad_sch (KiCad schematic)
At the start: 34 parts

Commit message: fix
Parts:
- SW?: value (none) -> SW_Push_45deg
- U?: value (none) -> 74LS138
- U?: value (none) -> pkd8279; footprint (none) -> pkd8279
- U?: value (none) -> PAL16L8
Changed lines of the file:
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@@
     (in_bom yes) (on_board yes) (fields_autoplaced)
     (property "Reference" "U?" (id 0) (at 215.9 128.4986 90))
-    (property "Value" "" (id 1) (at 215.9 131.0386 90))
+    (property "Value" "74LS138" (id 1) (at 215.9 131.0386 90))
     (property "Footprint" "" (id 2) (at 198.12 132.08 0)
       (effects (font (size 1.27 1.27)) hide)
@@
       (effects (font (size 1.524 1.524)))
     )
-    (property "Value" "" (id 1) (at 103.505 69.85 0)
+    (property "Value" "pkd8279" (id 1) (at 103.505 69.85 0)
       (effects (font (size 1.524 1.524)))
     )
-    (property "Footprint" "" (id 2) (at 102.87 67.564 0)
+    (property "Footprint" "pkd8279" (id 2) (at 102.87 67.564 0)
       (effects (font (size 1.524 1.524)) hide)
     )
@@
     (in_bom yes) (on_board yes) (fields_autoplaced)
     (property "Reference" "SW?" (id 0) (at 187.96 39.37 0))
-    (property "Value" "" (id 1) (at 187.96 41.91 0))
+    (property "Value" "SW_Push_45deg" (id 1) (at 187.96 41.91 0))
     (property "Footprint" "" (id 2) (at 187.96 46.99 0)
       (effects (font (size 1.27 1.27)) hide)
@@
       (effects (font (size 1.27 1.27)) (justify left))
     )
-    (property "Value" "" (id 1) (at 49.0094 87.63 0)
+    (property "Value" "PAL16L8" (id 1) (at 49.0094 87.63 0)
       (effects (font (size 1.27 1.27)) (justify left))
     )
@@
       (effects (font (size 1.27 1.27)) hide)
     )
-    (property "Value" "" (id 1) (at 46.99 124.46 0))
+    (property "Value" "GND" (id 1) (at 46.99 124.46 0))
     (property "Footprint" "" (id 2) (at 46.99 119.38 0)
       (effects (font (size 1.27 1.27)) hide)

Commit message: fixes
Connections:
- net IR0 renamed 8279 IRQ
Changed lines of the file:
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@@
     (effects (font (size 1.27 1.27)) (justify left bottom))
+  )
+  (label "VIN" (at 38.1 26.67 180)
+    (effects (font (size 1.27 1.27)) (justify right bottom))
   )
   (label "D4" (at 73.66 115.57 0)
@@
     (effects (font (size 1.27 1.27)) (justify right))
   )
-  (hierarchical_label "IR0" (shape output) (at 232.41 96.52 180)
+  (hierarchical_label "8279 IRQ" (shape output) (at 232.41 96.52 180)
     (effects (font (size 1.27 1.27)) (justify right))
   )

Commit message: final look
Parts:
- gave numbers to parts that had none: 34

Commit message: footprints
Parts:
- C1101, C1102, C1103: footprint (none) -> Capacitor_SMD:CP_Elec_3x5.3
Changed lines of the file:
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@@
       (effects (font (size 1.27 1.27)) (justify left))
     )
-    (property "Footprint" "" (id 2) (at 46.99 84.1248 0)
+    (property "Footprint" "Capacitor_SMD:CP_Elec_3x5.3" (id 2) (at 46.99 84.1248 0)
       (effects (font (size 1.27 1.27)) hide)
     )
@@
       (effects (font (size 1.27 1.27)) (justify left))
     )
-    (property "Footprint" "" (id 2) (at 131.7752 77.47 0)
+    (property "Footprint" "Capacitor_SMD:CP_Elec_3x5.3" (id 2) (at 131.7752 77.47 0)
       (effects (font (size 1.27 1.27)) hide)
     )
@@
       (effects (font (size 1.27 1.27)) (justify left))
     )
-    (property "Footprint" "" (id 2) (at 176.8348 132.08 0)
-      (effects (font (size 1.27 1.27)) hide)
-    )
+    (property "Footprint" "Capacitor_SMD:CP_Elec_3x5.3" (id 2) (at 176.8348 132.08 0)
+      (effects (font (size 1.27 1.27)) hide)
+    )

Commit message: pcb
Parts:
- SW1101, SW1102, SW1103, SW1104, SW1105, SW1106, SW1107, SW1108, SW1109, SW1110, SW1111, SW1112, SW1113, SW1114, SW1115, SW1116, SW1117, SW1118, SW1119, SW1120, SW1121, SW1122, SW1123, SW1124, SW1125: footprint (none) -> Button_Switch_Keyboard:SW_Cherry_MX_1.00u_Plate
- U1103: footprint (none) -> Package_DIP:DIP-20_W7.62mm
- U1104: footprint pkd8279 -> (none)
Changed lines of the file:
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@@
     (property "Reference" "SW1111" (id 0) (at 219.71 39.37 0))
     (property "Value" "SW_Push_45deg" (id 1) (at 219.71 41.91 0))
-    (property "Footprint" "" (id 2) (at 219.71 46.99 0)
+    (property "Footprint" "Button_Switch_Keyboard:SW_Cherry_MX_1.00u_Plate" (id 2) (at 219.71 46.99 0)
       (effects (font (size 1.27 1.27)) hide)
     )
@@
     (property "Reference" "SW1124" (id 0) (at 250.19 77.47 0))
     (property "Value" "SW_Push_45deg" (id 1) (at 250.19 80.01 0))
-    (property "Footprint" "" (id 2) (at 250.19 85.09 0)
+    (property "Footprint" "Button_Switch_Keyboard:SW_Cherry_MX_1.00u_Plate" (id 2) (at 250.19 85.09 0)
       (effects (font (size 1.27 1.27)) hide)
     )
@@
     (property "Reference" "SW1115" (id 0) (at 219.71 91.44 0))
     (property "Value" "SW_Push_45deg" (id 1) (at 219.71 93.98 0))
-    (property "Footprint" "" (id 2) (at 219.71 99.06 0)
+    (property "Footprint" "Button_Switch_Keyboard:SW_Cherry_MX_1.00u_Plate" (id 2) (at 219.71 99.06 0)
       (effects (font (size 1.27 1.27)) hide)
     )
@@
     (property "Reference" "SW1123" (id 0) (at 250.19 64.77 0))
     (property "Value" "SW_Push_45deg" (id 1) (at 250.19 67.31 0))
-    (property "Footprint" "" (id 2) (at 250.19 72.39 0)
+    (property "Footprint" "Button_Switch_Keyboard:SW_Cherry_MX_1.00u_Plate" (id 2) (at 250.19 72.39 0)
       (effects (font (size 1.27 1.27)) hide)
     )
@@
     (property "Reference" "SW1106" (id 0) (at 204.47 39.37 0))
     (property "Value" "SW_Push_45deg" (id 1) (at 204.47 41.91 0))
-    (property "Footprint" "" (id 2) (at 204.47 46.99 0)
+    (property "Footprint" "Button_Switch_Keyboard:SW_Cherry_MX_1.00u_Plate" (id 2) (at 204.47 46.99 0)
       (effects (font (size 1.27 1.27)) hide)
     )
@@
     (property "Reference" "SW1114" (id 0) (at 219.71 77.47 0))
     (property "Value" "SW_Push_45deg" (id 1) (at 219.71 80.01 0))
-    (property "Footprint" "" (id 2) (at 219.71 85.09 0)
+    (property "Footprint" "Button_Switch_Keyboard:SW_Cherry_MX_1.00u_Plate" (id 2) (at 219.71 85.09 0)
       (effects (font (size 1.27 1.27)) hide)
     )
@@
     (property "Reference" "SW1107" (id 0) (at 204.47 52.07 0))
     (property "Value" "SW_Push_45deg" (id 1) (at 204.47 54.61 0))
-    (property "Footprint" "" (id 2) (at 204.47 59.69 0)
+    (property "Footprint" "Button_Switch_Keyboard:SW_Cherry_MX_1.00u_Plate" (id 2) (at 204.47 59.69 0)
       (effects (font (size 1.27 1.27)) hide)
     )
@@
     (property "Reference" "SW1102" (id 0) (at 187.96 52.07 0))
     (property "Value" "SW_Push_45deg" (id 1) (at 187.96 54.61 0))
-    (property "Footprint" "" (id 2) (at 187.96 59.69 0)
+    (property "Footprint" "Button_Switch_Keyboard:SW_Cherry_MX_1.00u_Plate" (id 2) (at 187.96 59.69 0)
       (effects (font (size 1.27 1.27)) hide)
     )
@@
     (property "Reference" "SW1122" (id 0) (at 250.19 52.07 0))
     (property "Value" "SW_Push_45deg" (id 1) (at 250.19 54.61 0))
-    (property "Footprint" "" (id 2) (at 250.19 59.69 0)
+    (property "Footprint" "Button_Switch_Keyboard:SW_Cherry_MX_1.00u_Plate" (id 2) (at 250.19 59.69 0)
       (effects (font (size 1.27 1.27)) hide)
     )
@@
     (property "Reference" "SW1105" (id 0) (at 187.96 91.44 0))
     (property "Value" "SW_Push_45deg" (id 1) (at 187.96 93.98 0))
-    (property "Footprint" "" (id 2) (at 187.96 99.06 0)
+    (property "Footprint" "Button_Switch_Keyboard:SW_Cherry_MX_1.00u_Plate" (id 2) (at 187.96 99.06 0)
       (effects (font (size 1.27 1.27)) hide)
     )
@@
     (property "Reference" "SW1121" (id 0) (at 250.19 39.37 0))
     (property "Value" "SW_Push_45deg" (id 1) (at 250.19 41.91 0))
-    (property "Footprint" "" (id 2) (at 250.19 46.99 0)
+    (property "Footprint" "Button_Switch_Keyboard:SW_Cherry_MX_1.00u_Plate" (id 2) (at 250.19 46.99 0)
       (effects (font (size 1.27 1.27)) hide)
     )
@@
     (property "Reference" "SW1119" (id 0) (at 234.95 77.47 0))
     (property "Value" "SW_Push_45deg" (id 1) (at 234.95 80.01 0))
-    (property "Footprint" "" (id 2) (at 234.95 85.09 0)
+    (property "Footprint" "Button_Switch_Keyboard:SW_Cherry_MX_1.00u_Plate" (id 2) (at 234.95 85.09 0)
       (effects (font (size 1.27 1.27)) hide)
     )
@@
     (property "Reference" "SW1125" (id 0) (at 250.19 91.44 0))
     (property "Value" "SW_Push_45deg" (id 1) (at 250.19 93.98 0))
-    (property "Footprint" "" (id 2) (at 250.19 99.06 0)
+    (property "Footprint" "Button_Switch_Keyboard:SW_Cherry_MX_1.00u_Plate" (id 2) (at 250.19 99.06 0)
       (effects (font (size 1.27 1.27)) hide)
     )
@@
     (property "Reference" "SW1117" (id 0) (at 234.95 52.07 0))
     (property "Value" "SW_Push_45deg" (id 1) (at 234.95 54.61 0))
-    (property "Footprint" "" (id 2) (at 234.95 59.69 0)
+    (property "Footprint" "Button_Switch_Keyboard:SW_Cherry_MX_1.00u_Plate" (id 2) (at 234.95 59.69 0)
       (effects (font (size 1.27 1.27)) hide)
     )
@@
     (property "Reference" "SW1116" (id 0) (at 234.95 39.37 0))
     (property "Value" "SW_Push_45deg" (id 1) (at 234.95 41.91 0))
-    (property "Footprint" "" (id 2) (at 234.95 46.99 0)
+    (property "Footprint" "Button_Switch_Keyboard:SW_Cherry_MX_1.00u_Plate" (id 2) (at 234.95 46.99 0)
       (effects (font (size 1.27 1.27)) hide)
     )
@@
       (effects (font (size 1.524 1.524)))
     )
-    (property "Footprint" "pkd8279" (id 2) (at 102.87 67.564 0)
+    (property "Footprint" "" (id 2) (at 102.87 67.564 0)
       (effects (font (size 1.524 1.524)) hide)
     )
@@
     (property "Reference" "SW1104" (id 0) (at 187.96 77.47 0))
     (property "Value" "SW_Push_45deg" (id 1) (at 187.96 80.01 0))
-    (property "Footprint" "" (id 2) (at 187.96 85.09 0)
+    (property "Footprint" "Button_Switch_Keyboard:SW_Cherry_MX_1.00u_Plate" (id 2) (at 187.96 85.09 0)
       (effects (font (size 1.27 1.27)) hide)
     )
@@
     (property "Reference" "SW1118" (id 0) (at 234.95 64.77 0))
     (property "Value" "SW_Push_45deg" (id 1) (at 234.95 67.31 0))
-    (property "Footprint" "" (id 2) (at 234.95 72.39 0)
+    (property "Footprint" "Button_Switch_Keyboard:SW_Cherry_MX_1.00u_Plate" (id 2) (at 234.95 72.39 0)
       (effects (font (size 1.27 1.27)) hide)
     )
@@
     (property "Reference" "SW1101" (id 0) (at 187.96 39.37 0))
     (property "Value" "SW_Push_45deg" (id 1) (at 187.96 41.91 0))
-    (property "Footprint" "" (id 2) (at 187.96 46.99 0)
+    (property "Footprint" "Button_Switch_Keyboard:SW_Cherry_MX_1.00u_Plate" (id 2) (at 187.96 46.99 0)
       (effects (font (size 1.27 1.27)) hide)
     )
@@
     (property "Reference" "SW1110" (id 0) (at 204.47 91.44 0))
     (property "Value" "SW_Push_45deg" (id 1) (at 204.47 93.98 0))
-    (property "Footprint" "" (id 2) (at 204.47 99.06 0)
+    (property "Footprint" "Button_Switch_Keyboard:SW_Cherry_MX_1.00u_Plate" (id 2) (at 204.47 99.06 0)
       (effects (font (size 1.27 1.27)) hide)
     )
@@
     (property "Reference" "SW1112" (id 0) (at 219.71 52.07 0))
     (property "Value" "SW_Push_45deg" (id 1) (at 219.71 54.61 0))
-    (property "Footprint" "" (id 2) (at 219.71 59.69 0)
+    (property "Footprint" "Button_Switch_Keyboard:SW_Cherry_MX_1.00u_Plate" (id 2) (at 219.71 59.69 0)
       (effects (font (size 1.27 1.27)) hide)
     )
@@
     (property "Reference" "SW1113" (id 0) (at 219.71 64.77 0))
     (property "Value" "SW_Push_45deg" (id 1) (at 219.71 67.31 0))
-    (property "Footprint" "" (id 2) (at 219.71 72.39 0)
+    (property "Footprint" "Button_Switch_Keyboard:SW_Cherry_MX_1.00u_Plate" (id 2) (at 219.71 72.39 0)
       (effects (font (size 1.27 1.27)) hide)
     )
@@
     (property "Reference" "SW1109" (id 0) (at 204.47 77.47 0))
     (property "Value" "SW_Push_45deg" (id 1) (at 204.47 80.01 0))
-    (property "Footprint" "" (id 2) (at 204.47 85.09 0)
+    (property "Footprint" "Button_Switch_Keyboard:SW_Cherry_MX_1.00u_Plate" (id 2) (at 204.47 85.09 0)
       (effects (font (size 1.27 1.27)) hide)
     )
@@
     (property "Reference" "SW1120" (id 0) (at 234.95 91.44 0))
     (property "Value" "SW_Push_45deg" (id 1) (at 234.95 93.98 0))
-    (property "Footprint" "" (id 2) (at 234.95 99.06 0)
+    (property "Footprint" "Button_Switch_Keyboard:SW_Cherry_MX_1.00u_Plate" (id 2) (at 234.95 99.06 0)
       (effects (font (size 1.27 1.27)) hide)
     )
@@
     (property "Reference" "SW1103" (id 0) (at 187.96 64.77 0))
     (property "Value" "SW_Push_45deg" (id 1) (at 187.96 67.31 0))
-    (property "Footprint" "" (id 2) (at 187.96 72.39 0)
+    (property "Footprint" "Button_Switch_Keyboard:SW_Cherry_MX_1.00u_Plate" (id 2) (at 187.96 72.39 0)
       (effects (font (size 1.27 1.27)) hide)
     )
@@
       (effects (font (size 1.27 1.27)) (justify left))
     )
-    (property "Footprint" "" (id 2) (at 46.99 104.14 0)
+    (property "Footprint" "Package_DIP:DIP-20_W7.62mm" (id 2) (at 46.99 104.14 0)
       (effects (font (size 1.27 1.27)) hide)
     )
@@
     (property "Reference" "SW1108" (id 0) (at 204.47 64.77 0))
     (property "Value" "SW_Push_45deg" (id 1) (at 204.47 67.31 0))
-    (property "Footprint" "" (id 2) (at 204.47 72.39 0)
-      (effects (font (size 1.27 1.27)) hide)
-    )
+    (property "Footprint" "Button_Switch_Keyboard:SW_Cherry_MX_1.00u_Plate" (id 2) (at 204.47 72.39 0)
+      (effects (font (size 1.27 1.27)) hide)
+    )

Commit message: pcb
Parts:
- U1002, U1101, U1102, U1105: footprint (none) -> Package_DIP:DIP-14_W10.16mm
- U1104: footprint (none) -> Package_DIP:DIP-40_W25.4mm
Changed lines of the file:
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@@
     (property "Reference" "U1102" (id 0) (at 22.86 137.16 0))
     (property "Value" "74LS21" (id 1) (at 22.86 139.7 0))
-    (property "Footprint" "" (id 2) (at 22.86 147.32 0)
+    (property "Footprint" "Package_DIP:DIP-14_W10.16mm" (id 2) (at 22.86 147.32 0)
       (effects (font (size 1.27 1.27)) hide)
     )
@@
     (property "Reference" "U1105" (id 0) (at 215.9 128.4986 90))
     (property "Value" "74LS138" (id 1) (at 215.9 131.0386 90))
-    (property "Footprint" "" (id 2) (at 198.12 132.08 0)
+    (property "Footprint" "Package_DIP:DIP-14_W10.16mm" (id 2) (at 198.12 132.08 0)
       (effects (font (size 1.27 1.27)) hide)
     )
@@
       (effects (font (size 1.524 1.524)))
     )
-    (property "Footprint" "" (id 2) (at 102.87 67.564 0)
+    (property "Footprint" "Package_DIP:DIP-40_W25.4mm" (id 2) (at 102.87 67.564 0)
       (effects (font (size 1.524 1.524)) hide)
     )
@@
     (property "Reference" "U1101" (id 0) (at 22.86 120.65 0))
     (property "Value" "74LS21" (id 1) (at 22.86 123.19 0))
-    (property "Footprint" "" (id 2) (at 22.86 130.81 0)
+    (property "Footprint" "Package_DIP:DIP-14_W10.16mm" (id 2) (at 22.86 130.81 0)
       (effects (font (size 1.27 1.27)) hide)
     )
@@
     (property "Reference" "U1002" (id 0) (at 22.86 104.14 0))
     (property "Value" "74LS21" (id 1) (at 22.86 106.68 0))
-    (property "Footprint" "" (id 2) (at 22.86 114.3 0)
-      (effects (font (size 1.27 1.27)) hide)
-    )
+    (property "Footprint" "Package_DIP:DIP-14_W10.16mm" (id 2) (at 22.86 114.3 0)
+      (effects (font (size 1.27 1.27)) hide)
+    )

Commit message: chip size
Parts:
- U1105: footprint Package_DIP:DIP-14_W10.16mm -> (none)
Changed lines of the file:
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@@
     (property "Reference" "U1105" (id 0) (at 215.9 128.4986 90))
     (property "Value" "74LS138" (id 1) (at 215.9 131.0386 90))
-    (property "Footprint" "Package_DIP:DIP-14_W10.16mm" (id 2) (at 198.12 132.08 0)
+    (property "Footprint" "" (id 2) (at 198.12 132.08 0)
       (effects (font (size 1.27 1.27)) hide)
     )

Commit message: pcb edits
Parts:
- U1105: footprint (none) -> Package_DIP:DIP-16_W7.62mm
Connections:
- no-connect marks 26 -> 27
Changed lines of the file:
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@@
   (no_connect (at 59.69 101.6))
   (no_connect (at 59.69 104.14))
+  (no_connect (at 129.54 120.65))
   (wire (pts (xy 74.93 80.01) (xy 77.47 80.01))
     (stroke (width 0) (type default) (color 0 0 0 0))
@@
     (property "Reference" "U1105" (id 0) (at 215.9 128.4986 90))
     (property "Value" "74LS138" (id 1) (at 215.9 131.0386 90))
-    (property "Footprint" "" (id 2) (at 198.12 132.08 0)
-      (effects (font (size 1.27 1.27)) hide)
-    )
+    (property "Footprint" "Package_DIP:DIP-16_W7.62mm" (id 2) (at 198.12 132.08 0)
+      (effects (font (size 1.27 1.27)) hide)
+    )
