File: 8086proj/8279.kicad_sch (KiCad schematic)
At the start: 34 parts, among them SW1101 SW_Push_45deg, SW1102 SW_Push_45deg, SW1103 SW_Push_45deg, SW1104 SW_Push_45deg, SW1105 SW_Push_45deg, SW1106 SW_Push_45deg, SW1107 SW_Push_45deg, SW1108 SW_Push_45deg, SW1109 SW_Push_45deg, SW1110 SW_Push_45deg, SW1111 SW_Push_45deg, SW1112 SW_Push_45deg, SW1113 SW_Push_45deg, SW1114 SW_Push_45deg, SW1115 SW_Push_45deg, SW1116 SW_Push_45deg, SW1117 SW_Push_45deg, SW1118 SW_Push_45deg, SW1119 SW_Push_45deg, SW1120 SW_Push_45deg, SW1121 SW_Push_45deg, SW1122 SW_Push_45deg, SW1123 SW_Push_45deg, SW1124 SW_Push_45deg, SW1125 SW_Push_45deg, U1002 74LS21, U1101 74LS21, U1102 74LS21, U1103 PAL16L8, U1104 pkd8279, U1105 74LS138

Commit message: pcb
Connections:
- no-connect marks 27 -> 26
Changed lines of the file:
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@@
   (no_connect (at 59.69 101.6))
   (no_connect (at 59.69 104.14))
-  (no_connect (at 129.54 120.65))
   (wire (pts (xy 74.93 80.01) (xy 77.47 80.01))
     (stroke (width 0) (type default) (color 0 0 0 0))
