File: 8086proj/16550.kicad_sch (KiCad schematic)
At the start: 7 parts

Commit message: 16550
Connections:
- net GND: now also J?.3 (TDX), J?.7 (RTS), J?.8 (CTS), U?.20 (*EN), U?.24 (R3IN), U?.36 (~{CTS}), U?.37 (~{DSR}), U?.38 (~{DCD}), U?.39 (~{RI})
- net at U?.15 (T3IN): now also U?.34 (~{OUT1})
- net at U?.2 (T3OUT): now also J?.9 (RI)
- net at U?.23 (DDIS): no longer U?.20 (*EN)
- net at U?.4 (T2OUT): now also J?.2 (RDX)
- net at U?.6 (R2OUT): now also U?.10 (SIN)
- net at U?.7 (T2IN): now also U?.11 (SOUT)
- net at U?.24 (~{TXRDY}): no longer J?.2 (RDX)
- net at U?.29 (~{RXRDY}): no longer J?.3 (TDX)
- net at U?.32 (~{RTS}): no longer J?.8 (CTS)
- net at J?.1 (DCD), J?.6 (DSR): now also J?.4 (DTR); no longer U?.33 (~{DTR})
- no-connect marks 7 -> 11
Other:
- moved on the sheet: J?

Commit message: 8254 and 8279
Parts:
- C?: value (none) -> .1uF
- J?: value (none) -> DSUB-9; footprint (none) -> DSUB-9
- R?: value (none) -> 1kohm
- U?: value (none) -> max235cpg; footprint (none) -> max235cpg
- U?: value (none) -> PAL16L8
- U?: value (none) -> 16550; footprint (none) -> Package_DIP:DIP-40_W15.24mm
Changed lines of the file:
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@@
       (effects (font (size 1.524 1.524)))
     )
-    (property "Value" "" (id 1) (at 205.74 46.99 0)
-      (effects (font (size 1.524 1.524)))
-    )
-    (property "Footprint" "" (id 2) (at 205.74 48.514 0)
+    (property "Value" "max235cpg" (id 1) (at 205.74 46.99 0)
+      (effects (font (size 1.524 1.524)))
+    )
+    (property "Footprint" "max235cpg" (id 2) (at 205.74 48.514 0)
       (effects (font (size 1.524 1.524)) hide)
     )
@@
       (effects (font (size 1.27 1.27)) hide)
     )
-    (property "Value" "" (id 1) (at 146.05 58.42 0))
+    (property "Value" "GND" (id 1) (at 146.05 58.42 0))
     (property "Footprint" "" (id 2) (at 146.05 53.34 0)
       (effects (font (size 1.27 1.27)) hide)
@@
       (effects (font (size 1.27 1.27)) (justify left))
     )
-    (property "Value" "" (id 1) (at 40.1194 74.93 0)
+    (property "Value" "PAL16L8" (id 1) (at 40.1194 74.93 0)
       (effects (font (size 1.27 1.27)) (justify left))
     )
@@
       (effects (font (size 1.27 1.27)) (justify left))
     )
-    (property "Value" "" (id 1) (at 120.1294 33.02 0)
-      (effects (font (size 1.27 1.27)) (justify left))
-    )
-    (property "Footprint" "" (id 2) (at 118.11 74.93 0)
+    (property "Value" "16550" (id 1) (at 120.1294 33.02 0)
+      (effects (font (size 1.27 1.27)) (justify left))
+    )
+    (property "Footprint" "Package_DIP:DIP-40_W15.24mm" (id 2) (at 118.11 74.93 0)
       (effects (font (size 1.27 1.27) italic) hide)
     )
@@
       (effects (font (size 1.27 1.27)) (justify left))
     )
-    (property "Value" "" (id 1) (at 85.09 54.6099 0)
+    (property "Value" "1kohm" (id 1) (at 85.09 54.6099 0)
       (effects (font (size 1.27 1.27)) (justify left))
     )
@@
       (effects (font (size 1.27 1.27)) hide)
     )
-    (property "Value" "" (id 1) (at 88.9 105.4099 90)
+    (property "Value" "GND" (id 1) (at 88.9 105.4099 90)
       (effects (font (size 1.27 1.27)) (justify right))
     )
@@
       (effects (font (size 1.524 1.524)) (justify left))
     )
-    (property "Value" "" (id 1) (at 278.13 96.52 0)
+    (property "Value" "DSUB-9" (id 1) (at 278.13 96.52 0)
       (effects (font (size 1.524 1.524)) (justify left))
     )
-    (property "Footprint" "" (id 2) (at 271.78 92.964 0)
+    (property "Footprint" "DSUB-9" (id 2) (at 271.78 92.964 0)
       (effects (font (size 1.524 1.524)) hide)
     )
@@
       (effects (font (size 1.27 1.27)) hide)
     )
-    (property "Value" "" (id 1) (at 252.73 63.4999 90)
+    (property "Value" "GND" (id 1) (at 252.73 63.4999 90)
       (effects (font (size 1.27 1.27)) (justify right))
     )
@@
       (effects (font (size 1.27 1.27)) hide)
     )
-    (property "Value" "" (id 1) (at 132.08 31.75 0))
+    (property "Value" "GND" (id 1) (at 132.08 31.75 0))
     (property "Footprint" "" (id 2) (at 132.08 26.67 0)
       (effects (font (size 1.27 1.27)) hide)
@@
       (effects (font (size 1.27 1.27)) hide)
     )
-    (property "Value" "" (id 1) (at 248.92 93.9799 90)
+    (property "Value" "GND" (id 1) (at 248.92 93.9799 90)
       (effects (font (size 1.27 1.27)) (justify right))
     )
@@
     (in_bom yes) (on_board yes) (fields_autoplaced)
     (property "Reference" "C?" (id 0) (at 128.27 19.05 90))
-    (property "Value" "" (id 1) (at 128.27 21.59 90))
+    (property "Value" ".1uF" (id 1) (at 128.27 21.59 90))
     (property "Footprint" "" (id 2) (at 132.08 25.7048 0)
       (effects (font (size 1.27 1.27)) hide)
@@
       (effects (font (size 1.27 1.27)) hide)
     )
-    (property "Value" "" (id 1) (at 38.1 111.76 0))
+    (property "Value" "GND" (id 1) (at 38.1 111.76 0))
     (property "Footprint" "" (id 2) (at 38.1 106.68 0)
       (effects (font (size 1.27 1.27)) hide)

Commit message: final look
Parts:
- gave numbers to parts that had none: 7
Connections:
- no-connect marks 11 -> 25
Changed lines of the file:
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@@
   (no_connect (at 54.61 93.98))
   (no_connect (at 54.61 96.52))
+  (no_connect (at 172.72 54.61))
+  (no_connect (at 172.72 59.69))
+  (no_connect (at 172.72 64.77))
+  (no_connect (at 172.72 72.39))
+  (no_connect (at 172.72 76.2))
+  (no_connect (at 172.72 77.47))
+  (no_connect (at 238.76 57.15))
+  (no_connect (at 238.76 59.69))
+  (no_connect (at 238.76 67.31))
+  (no_connect (at 238.76 69.85))
+  (no_connect (at 238.76 72.39))
+  (no_connect (at 238.76 74.93))
+  (no_connect (at 238.76 80.01))
+  (no_connect (at 238.76 82.55))
   (no_connect (at 153.67 62.23))
   (no_connect (at 92.71 97.79))
@@
   (symbol (lib_id "max235cpg:max235cpg") (at 172.72 54.61 0) (unit 1)
     (in_bom yes) (on_board yes) (fields_autoplaced)
-    (property "Reference" "U?" (id 0) (at 205.74 43.18 0)
+    (property "Reference" "U903" (id 0) (at 205.74 43.18 0)
       (effects (font (size 1.524 1.524)))
     )
@@
   (symbol (lib_id "power:GND") (at 146.05 53.34 0) (unit 1)
     (in_bom yes) (on_board yes) (fields_autoplaced)
-    (property "Reference" "#PWR?" (id 0) (at 146.05 59.69 0)
+    (property "Reference" "#PWR0905" (id 0) (at 146.05 59.69 0)
       (effects (font (size 1.27 1.27)) hide)
     )
@@
   (symbol (lib_id "Logic_Programmable:PAL16L8") (at 38.1 91.44 0) (unit 1)
     (in_bom yes) (on_board yes) (fields_autoplaced)
-    (property "Reference" "U?" (id 0) (at 40.1194 72.39 0)
+    (property "Reference" "U901" (id 0) (at 40.1194 72.39 0)
       (effects (font (size 1.27 1.27)) (justify left))
     )
@@
   (symbol (lib_id "Interface_UART:16550") (at 118.11 74.93 0) (unit 1)
     (in_bom yes) (on_board yes) (fields_autoplaced)
-    (property "Reference" "U?" (id 0) (at 120.1294 30.48 0)
+    (property "Reference" "U902" (id 0) (at 120.1294 30.48 0)
       (effects (font (size 1.27 1.27)) (justify left))
     )
@@
   (symbol (lib_id "Device:R") (at 82.55 53.34 0) (unit 1)
     (in_bom yes) (on_board yes) (fields_autoplaced)
-    (property "Reference" "R?" (id 0) (at 85.09 52.0699 0)
+    (property "Reference" "R901" (id 0) (at 85.09 52.0699 0)
       (effects (font (size 1.27 1.27)) (justify left))
     )
@@
   (symbol (lib_id "power:GND") (at 118.11 118.11 0) (unit 1)
     (in_bom yes) (on_board yes) (fields_autoplaced)
-    (property "Reference" "#PWR?" (id 0) (at 118.11 124.46 0)
+    (property "Reference" "#PWR0903" (id 0) (at 118.11 124.46 0)
       (effects (font (size 1.27 1.27)) hide)
     )
@@
   (symbol (lib_id "power:GND") (at 92.71 105.41 270) (unit 1)
     (in_bom yes) (on_board yes) (fields_autoplaced)
-    (property "Reference" "#PWR?" (id 0) (at 86.36 105.41 0)
+    (property "Reference" "#PWR0902" (id 0) (at 86.36 105.41 0)
       (effects (font (size 1.27 1.27)) hide)
     )
@@
   (symbol (lib_id "DSUB-9:DSUB-9") (at 256.54 83.82 0) (unit 1)
     (in_bom yes) (on_board yes) (fields_autoplaced)
-    (property "Reference" "J?" (id 0) (at 278.13 92.71 0)
+    (property "Reference" "J901" (id 0) (at 278.13 92.71 0)
       (effects (font (size 1.524 1.524)) (justify left))
     )
@@
   (symbol (lib_id "power:GND") (at 248.92 63.5 90) (unit 1)
     (in_bom yes) (on_board yes) (fields_autoplaced)
-    (property "Reference" "#PWR?" (id 0) (at 255.27 63.5 0)
+    (property "Reference" "#PWR0907" (id 0) (at 255.27 63.5 0)
       (effects (font (size 1.27 1.27)) hide)
     )
@@
   (symbol (lib_id "Device:Crystal") (at 86.36 82.55 270) (unit 1)
     (in_bom yes) (on_board yes) (fields_autoplaced)
-    (property "Reference" "Y?" (id 0) (at 82.55 83.8201 90)
+    (property "Reference" "Y901" (id 0) (at 82.55 83.8201 90)
       (effects (font (size 1.27 1.27)) (justify right))
     )
@@
   (symbol (lib_id "power:GND") (at 132.08 26.67 0) (unit 1)
     (in_bom yes) (on_board yes) (fields_autoplaced)
-    (property "Reference" "#PWR?" (id 0) (at 132.08 33.02 0)
+    (property "Reference" "#PWR0904" (id 0) (at 132.08 33.02 0)
       (effects (font (size 1.27 1.27)) hide)
     )
@@
   (symbol (lib_id "power:GND") (at 252.73 93.98 270) (unit 1)
     (in_bom yes) (on_board yes) (fields_autoplaced)
-    (property "Reference" "#PWR?" (id 0) (at 246.38 93.98 0)
+    (property "Reference" "#PWR0908" (id 0) (at 246.38 93.98 0)
       (effects (font (size 1.27 1.27)) hide)
     )
@@
   (symbol (lib_id "Device:C") (at 128.27 26.67 90) (unit 1)
     (in_bom yes) (on_board yes) (fields_autoplaced)
-    (property "Reference" "C?" (id 0) (at 128.27 19.05 90))
+    (property "Reference" "C901" (id 0) (at 128.27 19.05 90))
     (property "Value" ".1uF" (id 1) (at 128.27 21.59 90))
     (property "Footprint" "" (id 2) (at 132.08 25.7048 0)
@@
   (symbol (lib_id "power:GND") (at 38.1 106.68 0) (unit 1)
     (in_bom yes) (on_board yes) (fields_autoplaced)
-    (property "Reference" "#PWR?" (id 0) (at 38.1 113.03 0)
+    (property "Reference" "#PWR0901" (id 0) (at 38.1 113.03 0)
       (effects (font (size 1.27 1.27)) hide)
     )
@@
   (symbol (lib_id "power:GND") (at 172.72 80.01 0) (unit 1)
     (in_bom yes) (on_board yes) (fields_autoplaced)
-    (property "Reference" "#PWR?" (id 0) (at 172.72 86.36 0)
-      (effects (font (size 1.27 1.27)) hide)
-    )
+    (property "Reference" "#PWR0906" (id 0) (at 172.72 86.36 0)
+      (effects (font (size 1.27 1.27)) hide)
+    )

Commit message: footprints
Parts:
- C901: footprint (none) -> Capacitor_SMD:CP_Elec_3x5.3
Changed lines of the file:
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@@
     (property "Reference" "C901" (id 0) (at 128.27 19.05 90))
     (property "Value" ".1uF" (id 1) (at 128.27 21.59 90))
-    (property "Footprint" "" (id 2) (at 132.08 25.7048 0)
+    (property "Footprint" "Capacitor_SMD:CP_Elec_3x5.3" (id 2) (at 132.08 25.7048 0)
       (effects (font (size 1.27 1.27)) hide)
     )

Commit message: pcb
Parts:
- J901: footprint DSUB-9 -> Connector_Dsub:DSUB-9_Female_Horizontal_P2.77x2.84mm_EdgePinOffset7.70mm_Housed_MountingHolesOffset9.12mm
- R901: footprint (none) -> Resistor_SMD:R_0201_0603Metric
- U901: footprint (none) -> Package_DIP:DIP-20_W7.62mm
- U903: footprint max235cpg -> Package_DIP:DIP-24_W10.16mm
Connections:
- net at U903.23 (R3OUT): now also J901.1 (DCD), J901.4 (DTR), J901.6 (DSR)
- no-connect marks 25 -> 24
Changed lines of the file:
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@@
   (no_connect (at 172.72 76.2))
   (no_connect (at 172.72 77.47))
-  (no_connect (at 238.76 57.15))
   (no_connect (at 238.76 59.69))
   (no_connect (at 238.76 67.31))
@@
     (stroke (width 0) (type default) (color 0 0 0 0))
   )
-  (wire (pts (xy 256.54 76.2) (xy 256.54 83.82))
+  (wire (pts (xy 256.54 57.15) (xy 256.54 83.82))
     (stroke (width 0) (type default) (color 0 0 0 0))
   )
@@
   )
   (wire (pts (xy 50.8 81.28) (xy 54.61 81.28))
+    (stroke (width 0) (type default) (color 0 0 0 0))
+  )
+  (wire (pts (xy 238.76 57.15) (xy 256.54 57.15))
     (stroke (width 0) (type default) (color 0 0 0 0))
   )
@@
       (effects (font (size 1.524 1.524)))
     )
-    (property "Footprint" "max235cpg" (id 2) (at 205.74 48.514 0)
+    (property "Footprint" "Package_DIP:DIP-24_W10.16mm" (id 2) (at 205.74 48.514 0)
       (effects (font (size 1.524 1.524)) hide)
     )
@@
       (effects (font (size 1.27 1.27)) (justify left))
     )
-    (property "Footprint" "" (id 2) (at 38.1 91.44 0)
+    (property "Footprint" "Package_DIP:DIP-20_W7.62mm" (id 2) (at 38.1 91.44 0)
       (effects (font (size 1.27 1.27)) hide)
     )
@@
       (effects (font (size 1.27 1.27)) (justify left))
     )
-    (property "Footprint" "" (id 2) (at 80.772 53.34 90)
+    (property "Footprint" "Resistor_SMD:R_0201_0603Metric" (id 2) (at 80.772 53.34 90)
       (effects (font (size 1.27 1.27)) hide)
     )
@@
       (effects (font (size 1.524 1.524)) (justify left))
     )
-    (property "Footprint" "DSUB-9" (id 2) (at 271.78 92.964 0)
+    (property "Footprint" "Connector_Dsub:DSUB-9_Female_Horizontal_P2.77x2.84mm_EdgePinOffset7.70mm_Housed_MountingHolesOffset9.12mm" (id 2) (at 271.78 92.964 0)
       (effects (font (size 1.524 1.524)) hide)
     )

Commit message: pcb update
Parts:
- Y901: footprint (none) -> Crystal:Crystal_AT310_D3.0mm_L10.0mm_Horizontal
Changed lines of the file:
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@@
       (effects (font (size 1.27 1.27)) (justify right))
     )
-    (property "Footprint" "" (id 2) (at 86.36 82.55 0)
+    (property "Footprint" "Crystal:Crystal_AT310_D3.0mm_L10.0mm_Horizontal" (id 2) (at 86.36 82.55 0)
       (effects (font (size 1.27 1.27)) hide)
     )

Commit message: pcb
Connections:
- net GND: no longer J901.3 (TDX), J901.7 (RTS), J901.8 (CTS), U903.24 (R3IN)
- new net: J901.3 (TDX), J901.7 (RTS), J901.8 (CTS), U903.24 (R3IN)
Changed lines of the file:
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@@
   (junction (at 156.21 21.59) (diameter 0) (color 0 0 0 0)
-  )
-  (junction (at 252.73 93.98) (diameter 0) (color 0 0 0 0)
   )
   (junction (at 118.11 21.59) (diameter 0) (color 0 0 0 0)
@@
     (stroke (width 0) (type default) (color 0 0 0 0))
   )
-  (wire (pts (xy 252.73 93.98) (xy 252.73 88.9))
+  (wire (pts (xy 252.73 88.9) (xy 252.73 101.6))
     (stroke (width 0) (type default) (color 0 0 0 0))
   )
@@
     (stroke (width 0) (type default) (color 0 0 0 0))
   )
-  (wire (pts (xy 252.73 101.6) (xy 252.73 93.98))
-    (stroke (width 0) (type default) (color 0 0 0 0))
-  )
