File: 8086proj/7seg.kicad_sch (KiCad schematic)
At the start: 20 parts, among them U1301 74AHC373, U1302 PAL16L8, U1303 D148K, U1304 74AHC373, U1305 D148K, U1306 74AHC373

Commit message: pcb
Parts:
- U1301, U1304, U1306: footprint (none) -> Package_DIP:DIP-14_W10.16mm
Changed lines of the file:
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@@
     (property "Reference" "U1306" (id 0) (at 236.22 112.8012 90))
     (property "Value" "74AHC373" (id 1) (at 236.22 115.3412 90))
-    (property "Footprint" "" (id 2) (at 214.63 119.38 0)
+    (property "Footprint" "Package_DIP:DIP-14_W10.16mm" (id 2) (at 214.63 119.38 0)
       (effects (font (size 1.27 1.27)) hide)
     )
@@
       (effects (font (size 1.27 1.27)) (justify left))
     )
-    (property "Footprint" "" (id 2) (at 173.99 87.63 0)
+    (property "Footprint" "Package_DIP:DIP-14_W10.16mm" (id 2) (at 173.99 87.63 0)
       (effects (font (size 1.27 1.27)) hide)
     )
@@
       (effects (font (size 1.27 1.27)) (justify left))
     )
-    (property "Footprint" "" (id 2) (at 48.26 86.36 0)
-      (effects (font (size 1.27 1.27)) hide)
-    )
+    (property "Footprint" "Package_DIP:DIP-14_W10.16mm" (id 2) (at 48.26 86.36 0)
+      (effects (font (size 1.27 1.27)) hide)
+    )

Commit message: pcb
Parts:
- U1301, U1304, U1306: footprint Package_DIP:DIP-14_W10.16mm -> (none)
Changed lines of the file:
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@@
     (property "Reference" "U1306" (id 0) (at 236.22 112.8012 90))
     (property "Value" "74AHC373" (id 1) (at 236.22 115.3412 90))
-    (property "Footprint" "Package_DIP:DIP-14_W10.16mm" (id 2) (at 214.63 119.38 0)
+    (property "Footprint" "" (id 2) (at 214.63 119.38 0)
       (effects (font (size 1.27 1.27)) hide)
     )
@@
       (effects (font (size 1.27 1.27)) (justify left))
     )
-    (property "Footprint" "Package_DIP:DIP-14_W10.16mm" (id 2) (at 173.99 87.63 0)
+    (property "Footprint" "" (id 2) (at 173.99 87.63 0)
       (effects (font (size 1.27 1.27)) hide)
     )
@@
       (effects (font (size 1.27 1.27)) (justify left))
     )
-    (property "Footprint" "Package_DIP:DIP-14_W10.16mm" (id 2) (at 48.26 86.36 0)
-      (effects (font (size 1.27 1.27)) hide)
-    )
+    (property "Footprint" "" (id 2) (at 48.26 86.36 0)
+      (effects (font (size 1.27 1.27)) hide)
+    )
