File: 8086proj/7seg.kicad_sch (KiCad schematic)
At the start: 20 parts

Commit message: 74244
Parts:
- C? (x3): value (none) -> .1uF
- D?: value (none) -> LED
- R?: value (none) -> R
- U?: value (none) -> PAL16L8
- U?: value (none) -> D148K; footprint (none) -> Display_7Segment:D1X8K
Changed lines of the file:
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@@
       (effects (font (size 1.27 1.27)) (justify left))
     )
-    (property "Value" "" (id 1) (at 70.5994 116.84 0)
+    (property "Value" "PAL16L8" (id 1) (at 70.5994 116.84 0)
       (effects (font (size 1.27 1.27)) (justify left))
     )
@@
     (in_bom yes) (on_board yes) (fields_autoplaced)
     (property "Reference" "C?" (id 0) (at 54.61 44.45 90))
-    (property "Value" "" (id 1) (at 54.61 46.99 90))
+    (property "Value" ".1uF" (id 1) (at 54.61 46.99 90))
     (property "Footprint" "" (id 2) (at 54.61 53.34 0)
       (effects (font (size 1.27 1.27)) hide)
@@
       (effects (font (size 1.27 1.27)) hide)
     )
-    (property "Value" "" (id 1) (at 60.96 58.42 0))
+    (property "Value" "GND" (id 1) (at 60.96 58.42 0))
     (property "Footprint" "" (id 2) (at 60.96 53.34 0)
       (effects (font (size 1.27 1.27)) hide)
@@
     (in_bom yes) (on_board yes) (fields_autoplaced)
     (property "Reference" "C?" (id 0) (at 180.34 46.99 90))
-    (property "Value" "" (id 1) (at 180.34 49.53 90))
+    (property "Value" ".1uF" (id 1) (at 180.34 49.53 90))
     (property "Footprint" "" (id 2) (at 180.34 55.88 0)
       (effects (font (size 1.27 1.27)) hide)
@@
     (in_bom yes) (on_board yes) (fields_autoplaced)
     (property "Reference" "R?" (id 0) (at 107.95 77.47 90))
-    (property "Value" "" (id 1) (at 107.95 80.01 90))
+    (property "Value" "R" (id 1) (at 107.95 80.01 90))
     (property "Footprint" "" (id 2) (at 107.95 85.598 90)
       (effects (font (size 1.27 1.27)) hide)
@@
       (effects (font (size 1.27 1.27)) hide)
     )
-    (property "Value" "" (id 1) (at 214.63 166.37 0))
+    (property "Value" "GND" (id 1) (at 214.63 166.37 0))
     (property "Footprint" "" (id 2) (at 214.63 161.29 0)
       (effects (font (size 1.27 1.27)) hide)
@@
     (in_bom yes) (on_board yes) (fields_autoplaced)
     (property "Reference" "U?" (id 0) (at 87.63 64.77 0))
-    (property "Value" "" (id 1) (at 87.63 67.31 0))
-    (property "Footprint" "" (id 2) (at 87.63 97.79 0)
+    (property "Value" "D148K" (id 1) (at 87.63 67.31 0))
+    (property "Footprint" "Display_7Segment:D1X8K" (id 2) (at 87.63 97.79 0)
       (effects (font (size 1.27 1.27)) hide)
     )
@@
       (effects (font (size 1.27 1.27)) hide)
     )
-    (property "Value" "" (id 1) (at 68.58 153.67 0))
+    (property "Value" "GND" (id 1) (at 68.58 153.67 0))
     (property "Footprint" "" (id 2) (at 68.58 148.59 0)
       (effects (font (size 1.27 1.27)) hide)
@@
     (in_bom yes) (on_board yes) (fields_autoplaced)
     (property "Reference" "D?" (id 0) (at 169.2275 143.51 0))
-    (property "Value" "" (id 1) (at 169.2275 146.05 0))
+    (property "Value" "LED" (id 1) (at 169.2275 146.05 0))
     (property "Footprint" "" (id 2) (at 167.64 151.13 0)
       (effects (font (size 1.27 1.27)) hide)
@@
       (effects (font (size 1.27 1.27)) hide)
     )
-    (property "Value" "" (id 1) (at 198.12 111.76 0))
+    (property "Value" "GND" (id 1) (at 198.12 111.76 0))
     (property "Footprint" "" (id 2) (at 198.12 106.68 0)
       (effects (font (size 1.27 1.27)) hide)
@@
     (in_bom yes) (on_board yes) (fields_autoplaced)
     (property "Reference" "C?" (id 0) (at 254 100.33 90))
-    (property "Value" "" (id 1) (at 254 102.87 90))
+    (property "Value" ".1uF" (id 1) (at 254 102.87 90))
     (property "Footprint" "" (id 2) (at 254 109.22 0)
       (effects (font (size 1.27 1.27)) hide)

Commit message: final look
Parts:
- gave numbers to parts that had none: 20

Commit message: footprints
Parts:
- C1301, C1302, C1303, C1304: footprint (none) -> Capacitor_SMD:CP_Elec_3x5.3
- D1301, D1302, D1303, D1304, D1305, D1306, D1307, D1308: footprint (none) -> LED_SMD:LED_0201_0603Metric
Changed lines of the file:
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@@
     (property "Reference" "C1301" (id 0) (at 54.61 44.45 90))
     (property "Value" ".1uF" (id 1) (at 54.61 46.99 90))
-    (property "Footprint" "" (id 2) (at 54.61 53.34 0)
+    (property "Footprint" "Capacitor_SMD:CP_Elec_3x5.3" (id 2) (at 54.61 53.34 0)
       (effects (font (size 1.27 1.27)) hide)
     )
@@
     (property "Reference" "D1303" (id 0) (at 193.3575 143.3526 0))
     (property "Value" "LED" (id 1) (at 193.3575 145.8926 0))
-    (property "Footprint" "" (id 2) (at 191.77 151.13 0)
+    (property "Footprint" "LED_SMD:LED_0201_0603Metric" (id 2) (at 191.77 151.13 0)
       (effects (font (size 1.27 1.27)) hide)
     )
@@
     (property "Reference" "D1305" (id 0) (at 218.7575 144.2906 0))
     (property "Value" "LED" (id 1) (at 218.7575 146.8306 0))
-    (property "Footprint" "" (id 2) (at 217.17 151.13 0)
+    (property "Footprint" "LED_SMD:LED_0201_0603Metric" (id 2) (at 217.17 151.13 0)
       (effects (font (size 1.27 1.27)) hide)
     )
@@
     (property "Reference" "D1304" (id 0) (at 206.0575 143.3526 0))
     (property "Value" "LED" (id 1) (at 206.0575 145.8926 0))
-    (property "Footprint" "" (id 2) (at 204.47 151.13 0)
+    (property "Footprint" "LED_SMD:LED_0201_0603Metric" (id 2) (at 204.47 151.13 0)
       (effects (font (size 1.27 1.27)) hide)
     )
@@
     (property "Reference" "C1302" (id 0) (at 118.11 87.63 90))
     (property "Value" ".1uF" (id 1) (at 118.11 90.17 90))
-    (property "Footprint" "" (id 2) (at 118.11 96.52 0)
+    (property "Footprint" "Capacitor_SMD:CP_Elec_3x5.3" (id 2) (at 118.11 96.52 0)
       (effects (font (size 1.27 1.27)) hide)
     )
@@
     (property "Reference" "C1303" (id 0) (at 180.34 46.99 90))
     (property "Value" ".1uF" (id 1) (at 180.34 49.53 90))
-    (property "Footprint" "" (id 2) (at 180.34 55.88 0)
+    (property "Footprint" "Capacitor_SMD:CP_Elec_3x5.3" (id 2) (at 180.34 55.88 0)
       (effects (font (size 1.27 1.27)) hide)
     )
@@
     (property "Reference" "D1308" (id 0) (at 258.1275 144.1799 0))
     (property "Value" "LED" (id 1) (at 258.1275 146.7199 0))
-    (property "Footprint" "" (id 2) (at 256.54 151.13 0)
+    (property "Footprint" "LED_SMD:LED_0201_0603Metric" (id 2) (at 256.54 151.13 0)
       (effects (font (size 1.27 1.27)) hide)
     )
@@
     (property "Reference" "D1307" (id 0) (at 245.4275 144.2906 0))
     (property "Value" "LED" (id 1) (at 245.4275 146.8306 0))
-    (property "Footprint" "" (id 2) (at 243.84 151.13 0)
+    (property "Footprint" "LED_SMD:LED_0201_0603Metric" (id 2) (at 243.84 151.13 0)
       (effects (font (size 1.27 1.27)) hide)
     )
@@
     (property "Reference" "D1301" (id 0) (at 169.2275 143.51 0))
     (property "Value" "LED" (id 1) (at 169.2275 146.05 0))
-    (property "Footprint" "" (id 2) (at 167.64 151.13 0)
+    (property "Footprint" "LED_SMD:LED_0201_0603Metric" (id 2) (at 167.64 151.13 0)
       (effects (font (size 1.27 1.27)) hide)
     )
@@
     (property "Reference" "D1306" (id 0) (at 231.4575 143.1313 0))
     (property "Value" "LED" (id 1) (at 231.4575 145.6713 0))
-    (property "Footprint" "" (id 2) (at 229.87 151.13 0)
+    (property "Footprint" "LED_SMD:LED_0201_0603Metric" (id 2) (at 229.87 151.13 0)
       (effects (font (size 1.27 1.27)) hide)
     )
@@
     (property "Reference" "D1302" (id 0) (at 181.9275 143.6847 0))
     (property "Value" "LED" (id 1) (at 181.9275 146.2247 0))
-    (property "Footprint" "" (id 2) (at 180.34 151.13 0)
+    (property "Footprint" "LED_SMD:LED_0201_0603Metric" (id 2) (at 180.34 151.13 0)
       (effects (font (size 1.27 1.27)) hide)
     )
@@
     (property "Reference" "C1304" (id 0) (at 254 100.33 90))
     (property "Value" ".1uF" (id 1) (at 254 102.87 90))
-    (property "Footprint" "" (id 2) (at 254 109.22 0)
-      (effects (font (size 1.27 1.27)) hide)
-    )
+    (property "Footprint" "Capacitor_SMD:CP_Elec_3x5.3" (id 2) (at 254 109.22 0)
+      (effects (font (size 1.27 1.27)) hide)
+    )

Commit message: pcb
Parts:
- R1301, R1302: footprint (none) -> Resistor_SMD:R_0201_0603Metric
- U1302: footprint (none) -> Package_DIP:DIP-20_W7.62mm
Changed lines of the file:
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@@
       (effects (font (size 1.27 1.27)) (justify left))
     )
-    (property "Footprint" "" (id 2) (at 68.58 133.35 0)
+    (property "Footprint" "Package_DIP:DIP-20_W7.62mm" (id 2) (at 68.58 133.35 0)
       (effects (font (size 1.27 1.27)) hide)
     )
@@
     (property "Reference" "R1301" (id 0) (at 107.95 77.47 90))
     (property "Value" "R" (id 1) (at 107.95 80.01 90))
-    (property "Footprint" "" (id 2) (at 107.95 85.598 90)
+    (property "Footprint" "Resistor_SMD:R_0201_0603Metric" (id 2) (at 107.95 85.598 90)
       (effects (font (size 1.27 1.27)) hide)
     )
@@
     (property "Reference" "R1302" (id 0) (at 224.79 77.47 90))
     (property "Value" "R" (id 1) (at 224.79 80.01 90))
-    (property "Footprint" "" (id 2) (at 224.79 85.598 90)
-      (effects (font (size 1.27 1.27)) hide)
-    )
+    (property "Footprint" "Resistor_SMD:R_0201_0603Metric" (id 2) (at 224.79 85.598 90)
+      (effects (font (size 1.27 1.27)) hide)
+    )

Commit message: PCB
Parts:
- U1301, U1304, U1306: footprint (none) -> Package_DIP:DIP-20_W7.62mm
Changed lines of the file:
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@@
+    (effects (font (size 1.27 1.27)) (justify left bottom))
+  )
+  (label "D[0..15]" (at 31.75 34.29 0)
     (effects (font (size 1.27 1.27)) (justify left bottom))
   )
@@
   )
   (label "A6" (at 49.53 135.89 0)
+    (effects (font (size 1.27 1.27)) (justify left bottom))
+  )
+  (label "A[0..19]" (at 39.37 30.48 0)
     (effects (font (size 1.27 1.27)) (justify left bottom))
   )
@@
     (property "Reference" "U1306" (id 0) (at 236.22 112.8012 90))
     (property "Value" "74AHC373" (id 1) (at 236.22 115.3412 90))
-    (property "Footprint" "" (id 2) (at 214.63 119.38 0)
+    (property "Footprint" "Package_DIP:DIP-20_W7.62mm" (id 2) (at 214.63 119.38 0)
       (effects (font (size 1.27 1.27)) hide)
     )
@@
       (effects (font (size 1.27 1.27)) (justify left))
     )
-    (property "Footprint" "" (id 2) (at 173.99 87.63 0)
+    (property "Footprint" "Package_DIP:DIP-20_W7.62mm" (id 2) (at 173.99 87.63 0)
       (effects (font (size 1.27 1.27)) hide)
     )
@@
       (effects (font (size 1.27 1.27)) (justify left))
     )
-    (property "Footprint" "" (id 2) (at 48.26 86.36 0)
-      (effects (font (size 1.27 1.27)) hide)
-    )
+    (property "Footprint" "Package_DIP:DIP-20_W7.62mm" (id 2) (at 48.26 86.36 0)
+      (effects (font (size 1.27 1.27)) hide)
+    )
