File: 8086proj/FinalProj.kicad_pcb (KiCad board)
At the start: 2 copper layers, 144 parts, among them J1001 Conn_01x03_Male, J1002 Conn_01x02_Male, J1003 Conn_01x03_Male, J201 Conn_01x15_Male, J202 Conn_01x20_Male, J203 Conn_01x16_Male, J601 Conn_01x08_Male, J602 Conn_01x08_Male, J603 Conn_01x08_Male, J604 Conn_01x08_Male, J605 Conn_01x08_Male, J606 Conn_01x08_Male, J607 Conn_01x08_Male, J608 Conn_01x08_Male, J609 Conn_01x08_Male, J701 Barrel_Jack, J801 Conn_01x04_Male, J901 DSUB-9, SW1101 SW_Push_45deg, SW1102 SW_Push_45deg, SW1103 SW_Push_45deg, SW1104 SW_Push_45deg, SW1105 SW_Push_45deg, SW1106 SW_Push_45deg, SW1107 SW_Push_45deg, SW1108 SW_Push_45deg, SW1109 SW_Push_45deg, SW1110 SW_Push_45deg, SW1111 SW_Push_45deg, SW1112 SW_Push_45deg, SW1113 SW_Push_45deg, SW1114 SW_Push_45deg, SW1115 SW_Push_45deg, SW1116 SW_Push_45deg, SW1117 SW_Push_45deg, SW1118 SW_Push_45deg, SW1119 SW_Push_45deg, SW1120 SW_Push_45deg, SW1121 SW_Push_45deg, SW1122 SW_Push_45deg, SW1123 SW_Push_45deg, SW1124 SW_Push_45deg, SW1125 SW_Push_45deg, SW1401 SW_DIP_x08, SW301 SW_DIP_x01, SW601 SW_DIP_x08, SW801 SW_Push, U1001 74LS04, U1002 74LS21, U1003 74LS21, U1004 PAL16L8, U1005 8254, U1101 74LS21, U1102 74LS21, U1103 PAL16L8, U1104 pkd8279, U1105 74LS138, U1201 PAL16L8, U1301 74AHC373, U1302 PAL16L8, U1303 D148K, U1304 74AHC373, U1305 D148K, U1306 74AHC373, U1401 74LS04, U1402 74LS21, U1403 74LS21, U1404 PAL16L8, U1405 74LS244, U201 8086_Min_Mode, U202 74AHC373, U203 74AHC373, U204 74AHC373, U401 PAL16L8, U402 28F010, U403 28F010, U501 PAL16L8, U502 CY7C199, U503 CY7C199, U504 CY7C199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

Commit message: pcb
Parts:
- moved C402 392.4 mm to (340.4, -99.1)
- moved U403 373.1 mm to (355.6, -95.2)
- moved U402 326.6 mm to (355.6, -47.0)
- moved C401 322.4 mm to (334.5, -3.12)
- moved U401 307.0 mm to (293.4, -90.2)
- moved J801 209.4 mm to (344.9, 290.4)
- moved U802 209.4 mm to (363.2, 275.9)
- moved C801 209.4 mm to (353.3, 286.4)
- moved C802 209.4 mm to (346.6, 286.4)
- moved R801 209.4 mm to (373.7, 267.9)
- moved R802 209.4 mm to (347.8, 289.7)
- moved SW801 209.4 mm to (385.1, 251.9)
- moved U801 209.4 mm to (376.5, 269.1)
- moved U803 209.4 mm to (363.2, 248.9)
- moved U804 209.4 mm to (344.8, 248.9)
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Connections:
- U201 pad 10: unconnected-(U201-Pad10) -> /16550/D6
- U201 pad 11: unconnected-(U201-Pad11) -> /16550/D5
- U201 pad 12: unconnected-(U201-Pad12) -> /16550/D4
- U201 pad 13: unconnected-(U201-Pad13) -> /16550/D3
- U201 pad 14: unconnected-(U201-Pad14) -> /16550/D2
- U201 pad 15: unconnected-(U201-Pad15) -> /16550/D1
- U201 pad 16: unconnected-(U201-Pad16) -> /16550/D0
- U201 pad 2: unconnected-(U201-Pad2) -> /16550/D14
- U201 pad 3: unconnected-(U201-Pad3) -> /16550/D13
- U201 pad 39: unconnected-(U201-Pad39) -> /16550/D15
- U201 pad 4: unconnected-(U201-Pad4) -> /16550/D12
- U201 pad 5: unconnected-(U201-Pad5) -> /16550/D11
- U201 pad 6: unconnected-(U201-Pad6) -> /16550/D10
- U201 pad 7: unconnected-(U201-Pad7) -> /16550/D9
- U201 pad 8: unconnected-(U201-Pad8) -> /16550/D8
- U201 pad 9: unconnected-(U201-Pad9) -> /16550/D7
- U202 pad 12: unconnected-(U202-Pad12) -> /16550/A4
- U202 pad 15: unconnected-(U202-Pad15) -> /16550/A5
- U202 pad 16: unconnected-(U202-Pad16) -> /16550/A6
- U202 pad 19: unconnected-(U202-Pad19) -> /16550/A7
- U202 pad 2: unconnected-(U202-Pad2) -> /16550/A0
- U202 pad 5: unconnected-(U202-Pad5) -> /16550/A1
- U202 pad 6: unconnected-(U202-Pad6) -> /16550/A2
- U202 pad 9: unconnected-(U202-Pad9) -> /16550/A3
- U203 pad 12: unconnected-(U203-Pad12) -> /16550/A12
- U203 pad 15: unconnected-(U203-Pad15) -> /16550/A13
- U203 pad 16: unconnected-(U203-Pad16) -> /16550/A14
- U203 pad 19: unconnected-(U203-Pad19) -> /16550/A15
- U203 pad 2: unconnected-(U203-Pad2) -> /16550/A8
- U203 pad 5: unconnected-(U203-Pad5) -> /16550/A9
- U203 pad 6: unconnected-(U203-Pad6) -> /16550/A10
- U203 pad 9: unconnected-(U203-Pad9) -> /16550/A11
- U204 pad 2: unconnected-(U204-Pad2) -> /8086/A16
- U204 pad 5: unconnected-(U204-Pad5) -> /8086/A17
- U204 pad 6: unconnected-(U204-Pad6) -> /8086/A18
- U204 pad 9: unconnected-(U204-Pad9) -> /8086/A19
Routing:
- net GND: track 0.92 -> 152.4 mm
- net /16550/D4: track 0.00 -> 115.9 mm
- net /16550/D5: track 0.00 -> 113.8 mm
- net Net-(U201-Pad25): track 0.00 -> 110.6 mm
- net /16550/D0: track 0.00 -> 100.1 mm
- net /16550/D6: track 0.00 -> 98.9 mm
- net /16550/D1: track 0.00 -> 95.0 mm
- net /16550/D8: track 0.00 -> 91.1 mm
- net /16550/D7: track 0.00 -> 88.9 mm
- net /16550/D9: track 0.00 -> 85.1 mm
- net /16550/D2: track 0.00 -> 84.9 mm
- net /16550/D12: track 0.00 -> 84.4 mm
- net /16550/D13: track 0.00 -> 84.0 mm
- net /16550/D14: track 0.00 -> 82.5 mm
- net /16550/D3: track 0.00 -> 79.0 mm
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Other:
- copper layers 2 -> 8

Commit message: pcb
Parts:
- added U301: ~, Package_DIP:DIP-18_W7.62mm, F.Cu at (14.0, -88.9)
- added Y301: ~, Crystal:Crystal_AT310_D3.0mm_L10.0mm_Horizontal, F.Cu at (31.4, -82.5)
- added Y901: ~, Crystal:Crystal_AT310_D3.0mm_L10.0mm_Horizontal, F.Cu at (278.1, 272.6)
- moved C302 365.4 mm to (32.0, -91.4)
- moved D301 357.8 mm to (25.4, -76.2), turned to 90 degrees
- moved R301 353.7 mm to (30.5, -76.2), turned to 90 degrees
- moved SW301 341.2 mm to (40.6, -71.1)
- moved C301 338.4 mm to (33.0, -61.0), turned to 90 degrees
- moved C401 52.4 mm to (368.3, -43.2)
- moved U401 30.5 mm to (322.6, -81.3)
- moved C402 27.9 mm to (368.3, -99.1)
- moved U402 12.7 mm to (345.4, -39.4)
- moved U403 7.72 mm to (348.0, -96.5)
Routing:
- net GND: track 152.4 -> 398.1 mm
- net /8086/READY: track 51.4 -> 236.3 mm
- net /8086/CLK: track 0.00 -> 174.4 mm
- net /16550/MR: track 59.4 -> 232.5 mm
- net /16550/A0: track 50.2 -> 170.4 mm
- net /28F010/_O2: track 0.00 -> 75.3 mm
- net /16550/M/_IO: track 67.6 -> 139.8 mm
- net Net-(C301-Pad2): track 0.00 -> 40.8 mm
- net /28F010/_O1: track 0.00 -> 39.0 mm
- net /16550/A1: track 67.5 -> 96.5 mm
- net /16550/A2: track 45.9 -> 73.4 mm
- net /16550/A3: track 43.2 -> 69.2 mm
- net /16550/A4: track 42.4 -> 66.8 mm
- net /16550/A5: track 44.1 -> 68.0 mm
- net /16550/A6: track 46.7 -> 70.1 mm
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
Commit message: pcb update
Parts:
- moved C1002 74.4 mm to (429.3, 132.1)
- moved R802 52.3 mm to (393.4, 264.2)
- moved J1003 45.9 mm to (393.7, 144.8)
- moved J1002 16.5 mm to (400.0, 144.8)
- moved C1401 3.57 mm to (405.4, 71.1)
- moved C1001 0.58 mm to (421.6, 132.1)
Routing:
- net GND: track 398.1 -> 707.5 mm
- net Net-(U1001-Pad2): track 0.00 -> 200.7 mm
- net Net-(U1004-Pad4): track 0.00 -> 195.6 mm
- net /8254/C2out: track 0.00 -> 153.8 mm
- net /16550/INTR: track 0.00 -> 145.1 mm
- net Net-(U1003-Pad6): track 0.00 -> 104.1 mm
- net Net-(U1402-Pad8): track 0.00 -> 57.8 mm
- net Net-(R802-Pad1): track 0.00 -> 54.0 mm
- net Net-(J801-Pad4): track 0.00 -> 47.4 mm
- net Net-(U1403-Pad8): track 0.00 -> 45.7 mm
- net Net-(J801-Pad3): track 0.00 -> 42.2 mm
- net Net-(J801-Pad2): track 0.00 -> 38.4 mm
- net Net-(U801-Pad8): track 0.00 -> 35.8 mm
- net Net-(J801-Pad1): track 0.00 -> 35.1 mm
- net Net-(U1001-Pad4): track 0.00 -> 34.4 mm
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
Commit message: pcb
Parts:
- U1405: footprint Package_DIP:DIP-14_W10.16mm -> Package_DIP:DIP-20_W7.62mm
Connections:
- SW1120 pad 1: /8279/8279 IRQ -> /8259/8279 IRQ

Commit message: pcb edit
Parts:
- moved C502 89.4 mm to (29.4, 223.5)
- moved C504 74.2 mm to (17.8, 223.5)
- moved C501 53.2 mm to (0.00, 223.5)
- moved C505 47.1 mm to (-17.8, 223.5)
- moved C503 42.6 mm to (-36.6, 223.5)
- moved U1401 7.61 mm to (415.9, 71.1)
Routing:
- net GND: track 707.5 -> 1016.9 mm
- net Net-(SW1106-Pad2): track 0.00 -> 182.1 mm
- net Net-(SW1111-Pad2): track 0.00 -> 181.9 mm
- net Net-(SW1101-Pad2): track 0.00 -> 178.1 mm
- net Net-(SW1121-Pad2): track 0.00 -> 157.7 mm
- net Net-(SW1116-Pad2): track 0.00 -> 154.9 mm
- net Net-(U1003-Pad1): track 0.00 -> 77.8 mm
- net /CY7C199/_CE1: track 0.00 -> 76.8 mm
- net /CY7C199/_CE0: track 0.00 -> 57.6 mm
- net /74374/_CS: track 0.00 -> 23.4 mm
- net Net-(SW1401-Pad12): track 0.00 -> 19.7 mm
- net Net-(SW1401-Pad9): track 0.00 -> 18.7 mm
- net Net-(SW1401-Pad11): track 0.00 -> 13.2 mm
- net Net-(SW1401-Pad10): track 0.00 -> 13.1 mm
- net Net-(SW1401-Pad13): track 0.00 -> 11.2 mm
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
Commit message: PCB
Parts:
- U1105: footprint Package_DIP:DIP-14_W10.16mm -> Package_DIP:DIP-16_W7.62mm
Changed lines of the file:
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@@
     )
   )
-  (footprint "Package_DIP:DIP-14_W10.16mm" (layer "F.Cu")
+  (footprint "Package_DIP:DIP-16_W7.62mm" (layer "F.Cu")
     (at 27.035 62.46)
-    (descr "14-lead though-hole mounted DIP package, row spacing 10.16 mm (400 mils)")
-    (tags "THT DIP DIL PDIP 2.54mm 10.16mm 400mil")
+    (descr "16-lead though-hole mounted DIP package, row spacing 7.62 mm (300 mils)")
+    (tags "THT DIP DIL PDIP 2.54mm 7.62mm 300mil")
     (property "Sheetfile" "8279.kicad_sch")
     (property "Sheetname" "8279")
     (attr through_hole)
-    (fp_text reference "U1105" (at 5.08 -2.33) (layer "F.SilkS")
+    (fp_text reference "U1105" (at 3.81 -2.33) (layer "F.SilkS")
       (effects (font (size 1 1) (thickness 0.15)))
     )
-    (fp_text value "74LS138" (at 5.08 17.57) (layer "F.Fab")
+    (fp_text value "74LS138" (at 3.81 20.11) (layer "F.Fab")
       (effects (font (size 1 1) (thickness 0.15)))
     )
-    (fp_text user "${REFERENCE}" (at 5.08 7.62) (layer "F.Fab")
+    (fp_text user "${REFERENCE}" (at 3.81 8.89) (layer "F.Fab")
       (effects (font (size 1 1) (thickness 0.15)))
     )
-    (fp_line (start 1.845 -1.33) (end 1.845 16.57) (layer "F.SilkS") (width 0.12))
-    (fp_line (start 8.315 -1.33) (end 6.08 -1.33) (layer "F.SilkS") (width 0.12))
-    (fp_line (start 8.315 16.57) (end 8.315 -1.33) (layer "F.SilkS") (width 0.12))
-    (fp_line (start 1.845 16.57) (end 8.315 16.57) (layer "F.SilkS") (width 0.12))
-    (fp_line (start 4.08 -1.33) (end 1.845 -1.33) (layer "F.SilkS") (width 0.12))
-    (fp_arc (start 6.08 -1.33) (mid 5.08 -0.33) (end 4.08 -1.33) (layer "F.SilkS") (width 0.12))
-    (fp_line (start -1.05 -1.55) (end -1.05 16.8) (layer "F.CrtYd") (width 0.05))
-    (fp_line (start 11.25 -1.55) (end -1.05 -1.55) (layer "F.CrtYd") (width 0.05))
-    (fp_line (start -1.05 16.8) (end 11.25 16.8) (layer "F.CrtYd") (width 0.05))
-    (fp_line (start 11.25 16.8) (end 11.25 -1.55) (layer "F.CrtYd") (width 0.05))
-    (fp_line (start 2.905 -1.27) (end 8.255 -1.27) (layer "F.Fab") (width 0.1))
-    (fp_line (start 1.905 16.51) (end 1.905 -0.27) (layer "F.Fab") (width 0.1))
-    (fp_line (start 8.255 -1.27) (end 8.255 16.51) (layer "F.Fab") (width 0.1))
-    (fp_line (start 1.905 -0.27) (end 2.905 -1.27) (layer "F.Fab") (width 0.1))
-    (fp_line (start 8.255 16.51) (end 1.905 16.51) (layer "F.Fab") (width 0.1))
+    (fp_line (start 6.46 19.11) (end 6.46 -1.33) (layer "F.SilkS") (width 0.12))
+    (fp_line (start 1.16 19.11) (end 6.46 19.11) (layer "F.SilkS") (width 0.12))
+    (fp_line (start 2.81 -1.33) (end 1.16 -1.33) (layer "F.SilkS") (width 0.12))
+    (fp_line (start 1.16 -1.33) (end 1.16 19.11) (layer "F.SilkS") (width 0.12))
+    (fp_line (start 6.46 -1.33) (end 4.81 -1.33) (layer "F.SilkS") (width 0.12))
+    (fp_arc (start 4.81 -1.33) (mid 3.81 -0.33) (end 2.81 -1.33) (layer "F.SilkS") (width 0.12))
+    (fp_line (start -1.1 -1.55) (end -1.1 19.3) (layer "F.CrtYd") (width 0.05))
+    (fp_line (start 8.7 -1.55) (end -1.1 -1.55) (layer "F.CrtYd") (width 0.05))
+    (fp_line (start 8.7 19.3) (end 8.7 -1.55) (layer "F.CrtYd") (width 0.05))
+    (fp_line (start -1.1 19.3) (end 8.7 19.3) (layer "F.CrtYd") (width 0.05))
+    (fp_line (start 0.635 19.05) (end 0.635 -0.27) (layer "F.Fab") (width 0.1))
+    (fp_line (start 1.635 -1.27) (end 6.985 -1.27) (layer "F.Fab") (width 0.1))
+    (fp_line (start 6.985 19.05) (end 0.635 19.05) (layer "F.Fab") (width 0.1))
+    (fp_line (start 0.635 -0.27) (end 1.635 -1.27) (layer "F.Fab") (width 0.1))
+    (fp_line (start 6.985 -1.27) (end 6.985 19.05) (layer "F.Fab") (width 0.1))
     (pad "1" thru_hole rect (at 0 0) (size 1.6 1.6) (drill 0.8) (layers *.Cu *.Mask)
       (net 316 "Net-(U1104-Pad32)") (pinfunction "A0") (pintype "input"))
@@
     (pad "7" thru_hole oval (at 0 15.24) (size 1.6 1.6) (drill 0.8) (layers *.Cu *.Mask)
       (net 319 "unconnected-(U1105-Pad7)") (pinfunction "O7") (pintype "output+no_connect"))
-    (pad "8" thru_hole oval (at 10.16 15.24) (size 1.6 1.6) (drill 0.8) (layers *.Cu *.Mask)
+    (pad "8" thru_hole oval (at 0 17.78) (size 1.6 1.6) (drill 0.8) (layers *.Cu *.Mask)
       (net 1 "GND") (pinfunction "GND") (pintype "power_in"))
-    (pad "9" thru_hole oval (at 10.16 12.7) (size 1.6 1.6) (drill 0.8) (layers *.Cu *.Mask)
+    (pad "9" thru_hole oval (at 7.62 17.78) (size 1.6 1.6) (drill 0.8) (layers *.Cu *.Mask)
       (net 320 "unconnected-(U1105-Pad9)") (pinfunction "O6") (pintype "output+no_connect"))
-    (pad "10" thru_hole oval (at 10.16 10.16) (size 1.6 1.6) (drill 0.8) (layers *.Cu *.Mask)
+    (pad "10" thru_hole oval (at 7.62 15.24) (size 1.6 1.6) (drill 0.8) (layers *.Cu *.Mask)
       (net 321 "unconnected-(U1105-Pad10)") (pinfunction "O5") (pintype "output+no_connect"))
-    (pad "11" thru_hole oval (at 10.16 7.62) (size 1.6 1.6) (drill 0.8) (layers *.Cu *.Mask)
+    (pad "11" thru_hole oval (at 7.62 12.7) (size 1.6 1.6) (drill 0.8) (layers *.Cu *.Mask)
       (net 162 "Net-(SW1121-Pad2)") (pinfunction "O4") (pintype "output"))
-    (pad "12" thru_hole oval (at 10.16 5.08) (size 1.6 1.6) (drill 0.8) (layers *.Cu *.Mask)
+    (pad "12" thru_hole oval (at 7.62 10.16) (size 1.6 1.6) (drill 0.8) (layers *.Cu *.Mask)
       (net 161 "Net-(SW1116-Pad2)") (pinfunction "O3") (pintype "output"))
-    (pad "13" thru_hole oval (at 10.16 2.54) (size 1.6 1.6) (drill 0.8) (layers *.Cu *.Mask)
+    (pad "13" thru_hole oval (at 7.62 7.62) (size 1.6 1.6) (drill 0.8) (layers *.Cu *.Mask)
       (net 160 "Net-(SW1111-Pad2)") (pinfunction "O2") (pintype "output"))
-    (pad "14" thru_hole oval (at 10.16 0) (size 1.6 1.6) (drill 0.8) (layers *.Cu *.Mask)
+    (pad "14" thru_hole oval (at 7.62 5.08) (size 1.6 1.6) (drill 0.8) (layers *.Cu *.Mask)
       (net 158 "Net-(SW1106-Pad2)") (pinfunction "O1") (pintype "output"))
-    (model "${KICAD6_3DMODEL_DIR}/Package_DIP.3dshapes/DIP-14_W10.16mm.wrl"
+    (pad "15" thru_hole oval (at 7.62 2.54) (size 1.6 1.6) (drill 0.8) (layers *.Cu *.Mask)
+      (net 153 "Net-(SW1101-Pad2)") (pinfunction "O0") (pintype "output"))
+    (pad "16" thru_hole oval (at 7.62 0) (size 1.6 1.6) (drill 0.8) (layers *.Cu *.Mask)
+      (net 1 "GND") (pinfunction "VCC") (pintype "power_in"))
+    (model "${KICAD6_3DMODEL_DIR}/Package_DIP.3dshapes/DIP-16_W7.62mm.wrl"
       (offset (xyz 0 0 0))
       (scale (xyz 1 1 1))

Commit message: pcb edits
Parts:
- moved U1104 184.9 mm to (73.7, 44.5)
- moved C1102 140.1 mm to (86.4, 38.1)
- moved U1103 130.6 mm to (41.9, 62.2)
- moved C1101 127.4 mm to (45.7, 91.4)
- moved C1103 82.5 mm to (30.5, 86.4)
Routing:
- net /8086/INTR: track 32.9 -> 572.6 mm
- net /8259/8279 IRQ: track 0.00 -> 450.6 mm
- net /8086/_INTA: track 45.9 -> 463.2 mm
- net Net-(U1002-Pad6): track 0.00 -> 414.3 mm
- net /8254/C2out: track 153.8 -> 532.0 mm
- net Net-(SW1101-Pad1): track 0.00 -> 291.0 mm
- net Net-(SW1104-Pad1): track 0.00 -> 261.9 mm
- net Net-(SW1102-Pad1): track 0.00 -> 217.0 mm
- net /8086/NMI: track 40.1 -> 231.1 mm, vias 0 -> 1
- net /16550/MR: track 232.5 -> 384.2 mm
- net Net-(SW1103-Pad1): track 0.00 -> 144.8 mm
- net Net-(U1102-Pad8): track 0.00 -> 117.7 mm
- net Net-(SW1105-Pad1): track 0.00 -> 110.8 mm
- net Net-(SW1110-Pad1): track 0.00 -> 107.0 mm
- net GND: track 1016.9 -> 1113.0 mm
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
Commit message: pcb
Parts:
- U1301, U1304, U1306: footprint Package_DIP:DIP-14_W10.16mm -> Package_DIP:DIP-20_W7.62mm
- moved D1301 379.5 mm to (-40.6, -94.0)
- moved D1302 377.8 mm to (-40.6, -91.4)
- moved D1303 371.2 mm to (-40.6, -88.9)
- moved D1304 370.7 mm to (-40.6, -86.4)
- moved D1305 367.4 mm to (-40.6, -83.8)
- moved D1306 367.4 mm to (-40.6, -81.3)
- moved C1303 367.1 mm to (-29.4, -91.4)
- moved D1307 364.3 mm to (-40.6, -78.7)
- moved D1308 361.0 mm to (-40.6, -76.2)
- moved U1306 355.4 mm to (-28.0, -86.4)
- moved U1301 350.9 mm to (-27.9, -61.0)
- moved C1302 350.4 mm to (-35.6, -71.1)
- moved R1301 348.5 mm to (-53.3, -53.3)
- moved R1302 327.2 mm to (-58.8, -27.9)
- moved C1304 323.8 mm to (-33.0, -40.6)
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Connections:
- J901 pad 3: GND -> Net-(J901-Pad3)
- J901 pad 7: GND -> Net-(J901-Pad3)
- J901 pad 8: GND -> Net-(J901-Pad3)
- U903 pad 24: GND -> Net-(J901-Pad3)
Routing:
- net /16550/_WR: track 47.4 -> 990.6 mm
- net /16550/_RD: track 57.9 -> 725.4 mm
- net /16550/M/_IO: track 139.8 -> 633.0 mm, vias 0 -> 2
- net /16550/MR: track 384.2 -> 805.9 mm
- net /16550/A6: track 70.1 -> 323.9 mm, vias 0 -> 1
- net /16550/A7: track 73.4 -> 321.1 mm, vias 0 -> 2
- net /16550/A11: track 64.6 -> 293.7 mm, vias 0 -> 3
- net /16550/A15: track 59.1 -> 269.8 mm, vias 0 -> 1
- net Net-(U1301-Pad12): track 0.00 -> 207.4 mm
- net /16550/A14: track 49.6 -> 253.1 mm, vias 0 -> 1
- net /16550/A9: track 62.5 -> 254.6 mm, vias 0 -> 2
- net /16550/A8: track 69.1 -> 259.7 mm, vias 0 -> 2
- net /16550/A3: track 69.2 -> 256.4 mm
- net /16550/A1: track 96.5 -> 278.3 mm
- net /16550/A2: track 73.4 -> 249.8 mm, vias 0 -> 1
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Other:
- copper layers 8 -> 10
