File: 8086proj/FinalProj.kicad_pcb (KiCad board)
At the start: 10 copper layers, 147 parts, among them J1001 Conn_01x03_Male, J1002 Conn_01x02_Male, J1003 Conn_01x03_Male, J201 Conn_01x15_Male, J202 Conn_01x20_Male, J203 Conn_01x16_Male, J601 Conn_01x08_Male, J602 Conn_01x08_Male, J603 Conn_01x08_Male, J604 Conn_01x08_Male, J605 Conn_01x08_Male, J606 Conn_01x08_Male, J607 Conn_01x08_Male, J608 Conn_01x08_Male, J609 Conn_01x08_Male, J701 Barrel_Jack, J801 Conn_01x04_Male, J901 DSUB-9, SW1101 SW_Push_45deg, SW1102 SW_Push_45deg, SW1103 SW_Push_45deg, SW1104 SW_Push_45deg, SW1105 SW_Push_45deg, SW1106 SW_Push_45deg, SW1107 SW_Push_45deg, SW1108 SW_Push_45deg, SW1109 SW_Push_45deg, SW1110 SW_Push_45deg, SW1111 SW_Push_45deg, SW1112 SW_Push_45deg, SW1113 SW_Push_45deg, SW1114 SW_Push_45deg, SW1115 SW_Push_45deg, SW1116 SW_Push_45deg, SW1117 SW_Push_45deg, SW1118 SW_Push_45deg, SW1119 SW_Push_45deg, SW1120 SW_Push_45deg, SW1121 SW_Push_45deg, SW1122 SW_Push_45deg, SW1123 SW_Push_45deg, SW1124 SW_Push_45deg, SW1125 SW_Push_45deg, SW1401 SW_DIP_x08, SW301 SW_DIP_x01, SW601 SW_DIP_x08, SW801 SW_Push, U1001 74LS04, U1002 74LS21, U1003 74LS21, U1004 PAL16L8, U1005 8254, U1101 74LS21, U1102 74LS21, U1103 PAL16L8, U1104 pkd8279, U1105 74LS138, U1201 PAL16L8, U1301 74AHC373, U1302 PAL16L8, U1303 D148K, U1304 74AHC373, U1305 D148K, U1306 74AHC373, U1401 74LS04, U1402 74LS21, U1403 74LS21, U1404 PAL16L8, U1405 74LS244, U201 8086_Min_Mode, U202 74AHC373, U203 74AHC373, U204 74AHC373, U401 PAL16L8, U402 28F010, U403 28F010, U501 PAL16L8, U502 CY7C199, U503 CY7C199, U504 CY7C199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

Commit message: pcb
Routing:
- net /16550/D5: track 113.8 -> 451.4 mm
- net /16550/D4: track 115.9 -> 404.8 mm
- net /16550/D3: track 79.0 -> 346.4 mm
- net /16550/D2: track 84.9 -> 329.0 mm
- net /16550/D1: track 95.0 -> 336.7 mm
- net /16550/D0: track 100.1 -> 336.4 mm
- net /16550/D15: track 60.5 -> 240.9 mm
- net /16550/D14: track 82.5 -> 212.7 mm
- net /16550/D13: track 84.0 -> 211.1 mm
- net /16550/D12: track 84.4 -> 207.2 mm
- net /16550/D11: track 77.3 -> 197.1 mm
- net /16550/D10: track 74.9 -> 191.8 mm
- net /16550/D9: track 85.1 -> 197.4 mm
- net /16550/D8: track 91.1 -> 200.6 mm
- net /16550/D7: track 88.9 -> 193.9 mm
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
Commit message: PCB
Connections:
- U1301 pad 11: /7seg/A15 -> /16550/A15
- U1301 pad 13: /7seg/D4 -> /16550/D4
- U1301 pad 14: /7seg/D5 -> /16550/D5
- U1301 pad 17: /7seg/D6 -> /16550/D6
- U1301 pad 18: /7seg/D7 -> /16550/D7
- U1301 pad 3: /7seg/D0 -> /16550/D0
- U1301 pad 4: /7seg/D1 -> /16550/D1
- U1301 pad 7: /7seg/D2 -> /16550/D2
- U1301 pad 8: /7seg/D3 -> /16550/D3
- U1302 pad 1: /7seg/A0 -> /16550/A0
- U1302 pad 11: /7seg/A9 -> /16550/A9
- U1302 pad 14: /7seg/A15 -> /16550/A15
- U1302 pad 15: /7seg/A14 -> /16550/A14
- U1302 pad 16: /7seg/A13 -> /16550/A13
- U1302 pad 17: /7seg/A12 -> /16550/A12
- U1302 pad 18: /7seg/A11 -> /16550/A11
- U1302 pad 19: /7seg/A10 -> /16550/A10
- U1302 pad 2: /7seg/A1 -> /16550/A1
- U1302 pad 3: /7seg/A2 -> /16550/A2
- U1302 pad 4: /7seg/A3 -> /16550/A3
- U1302 pad 5: /7seg/A4 -> /16550/A4
- U1302 pad 6: /7seg/A5 -> /16550/A5
- U1302 pad 7: /7seg/A6 -> /16550/A6
- U1302 pad 8: /7seg/A7 -> /16550/A7
- U1302 pad 9: /7seg/A8 -> /16550/A8
- U1304 pad 13: /7seg/D4 -> /16550/D4
- U1304 pad 14: /7seg/D5 -> /16550/D5
- U1304 pad 17: /7seg/D6 -> /16550/D6
- U1304 pad 18: /7seg/D7 -> /16550/D7
- U1304 pad 3: /7seg/D0 -> /16550/D0
- U1304 pad 4: /7seg/D1 -> /16550/D1
- U1304 pad 7: /7seg/D2 -> /16550/D2
- U1304 pad 8: /7seg/D3 -> /16550/D3
- U1306 pad 13: /7seg/D4 -> /16550/D4
- U1306 pad 14: /7seg/D5 -> /16550/D5
- U1306 pad 17: /7seg/D6 -> /16550/D6
- U1306 pad 18: /7seg/D7 -> /16550/D7
- U1306 pad 3: /7seg/D0 -> /16550/D0
- U1306 pad 4: /7seg/D1 -> /16550/D1
- U1306 pad 7: /7seg/D2 -> /16550/D2
- U1306 pad 8: /7seg/D3 -> /16550/D3
Routing:
- net /16550/A4: track 240.2 -> 1924.8 mm, vias 2 -> 7
- net /16550/A12: track 171.7 -> 1732.9 mm, vias 0 -> 1
- net /16550/A2: track 249.8 -> 1596.9 mm, vias 1 -> 6
- net GND: track 1169.1 -> 2296.9 mm, vias 0 -> 2
- net /16550/A13: track 218.9 -> 1271.9 mm
- net /16550/D6: track 200.9 -> 1060.6 mm, vias 0 -> 4
- net /16550/D2: track 329.0 -> 1160.7 mm, vias 0 -> 2
- net /16550/_RD: track 725.4 -> 1496.5 mm, vias 0 -> 2
- net /16550/D7: track 193.9 -> 957.7 mm, vias 0 -> 3
- net /16550/D3: track 346.4 -> 1081.2 mm, vias 0 -> 3
- net /16550/D0: track 336.4 -> 1023.4 mm, vias 0 -> 4
- net /16550/A0: track 170.4 -> 848.8 mm, vias 0 -> 1
- net /16550/A11: track 293.7 -> 970.3 mm
- net /16550/A3: track 256.4 -> 796.2 mm, vias 0 -> 2
- net /16550/A10: track 238.0 -> 727.4 mm
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
Commit message: pcb edits
Routing:
- net /16550/A8: track 724.0 -> 1677.0 mm, vias 3 -> 4
- net /16550/A6: track 655.7 -> 1414.0 mm, vias 2 -> 4
- net /16550/A1: track 707.5 -> 1417.7 mm, vias 0 -> 3
- net /16550/A7: track 656.5 -> 1215.6 mm
- net /16550/A9: track 724.0 -> 1116.5 mm
- net /16550/_WR: track 1012.6 -> 1338.5 mm
- net /16550/A10: track 727.4 -> 912.2 mm, vias 1 -> 2
- net /16550/_RD: track 1496.5 -> 1670.7 mm
- net /16550/A11: track 970.3 -> 1022.5 mm
- net /16550/A5: track 586.3 -> 606.7 mm
